File: HILTOP_motherboard/RETPower.sch (KiCad schematic (older format))
At the start: 90 parts, among them Q1 Q_NMOS_DS_POWERPAK, Q2 Q_NMOS_DS_POWERPAK, Q4 2N7002, U10 TLC271, U11 ADS1015, U12 MCP4725, U8 LM5118, U9 INA250A3

Commit message: Added new USB2.0 device
Parts:
- added C? (x2): 100uF, Capacitors_SMD:CP_Elec_6.3x7.7, symbol CP
- C179, C56, C58: value DNF -> 2.2uF; Devtank (none) -> 105-011
- C60: value 2200pF -> 100nF; Devtank 106-002 -> 105-002
- R58: value 29,4K -> 30K; Devtank 101-022 -> 101-021
- R59: value 18,2K -> 18K
- R75: value 4K7 -> 3K3; Devtank 101-009 -> 101-013
Connections:
- net +3V3: now also R60.1
- net GND: now also C?.2, C?.2
- net at C181.2, C182.2, C183.2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: now also C?.1, C?.1
- net at Q4.1 (G): now also R114.1, R116.1
Other:
- moved on the sheet: C117, C118, C179, C180, C181, C182, C183, C186, C187, C54, C56, C57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

Commit message: Added more detail to motherboard schemas
Connections:
- net RET_DC renamed VADJ_DC
Changed lines of the file:
@@
 $EndDescr
 Text HLabel 12450 3350 2    60   Output ~ 0
-RET_DC
+VADJ_DC
 Text HLabel 14850 3150 0    60   Input ~ 0
 PSU_SDA
@@
 $EndComp
 Text HLabel 12300 6300 2    60   Output ~ 0
-RET_GND
+VADJ_GND
 $Comp
 L TLC271 U10
