File: HILTOP_motherboard/HILTOP_Motherboard.kicad_pcb (KiCad board)
At the start: 4 copper layers, 170 x 170 mm, 1014 parts, among them J10 HDMI, J11 DISP_PWR, J12 DISPLAY_PORT, J13 DDR2_SODIMM_COMPUTE_MODULE_3, J14 PROG_PWR2, J15 PROG_PWR1, J16 SOFT_START_PWR, J17 PWR_LED, J18 RS232_DEBUG, J19 Micro_SD_Card, J2 ATX_MOLEX_02X12, J3 USB_A, J4 USB_A_DOUBLE, J5 SYSTEM_SPI_I2C, J6 USB_A, J7 USB_HEADER, J8 RS485_CONN, J9 RJ45-TRANS_SI-61001-F, Q1 Q_NMOS_DS_POWERPAK, Q2 Q_NMOS_DS_POWERPAK, Q3 2N7002, Q4 2N7002, U1 LM2664, U10 TLC271, U11 ADS1015, U12 MCP4725, U13 CME0303S3C, U14 ADuM1401, U15 ADuM1401, U16 CME0303S3C, U17 ISL83491, U18 ISL83491, U2 TPS2044B, U23 TPD12S016, U24 MAX16054, U25 STM6719SFWB6F, U27 TPS54394, U28 LP2985, U4 SN75240PWR, U6 SN75240PWR, U7 LAN7500, U8 LM5118, U9 INA250A3, Y1 6MHz Crystal, Y2 25MHz Crystal

Commit message: Fixed giabit LAN Schematic errors
Routing:
- net GND: track 519.7 -> 512.4 mm, vias 261 -> 256
- net (no net): track 14.3 -> 21.5 mm, vias 1 -> 6
Other:
- board text added: "DEVTANK/HILTOP/M'BOARD/001 P/N: 304-001 Rev: A"
- board text removed: "HILTOP MAIN BOARD"
- board text removed: "Part No. 304-001 Iss1.0"
Changed lines of the file:
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@@
 (kicad_pcb (version 4) (host pcbnew 4.0.7-e2-6376~58~ubuntu16.04.1)
   (general
-    (links 1839)
+    (links 1795)
     (no_connects 32)
     (area 45.057143 47.864999 225.292858 223.364286)
     (thickness 1.6)
-    (drawings 12)
+    (drawings 11)
     (tracks 6945)
     (zones 0)
@@
     (add_net "Net-(U27-Pad11)")
     (add_net "Net-(U27-Pad6)")
-    (add_net "Net-(U3-Pad11)")
-    (add_net "Net-(U3-Pad23)")
-    (add_net "Net-(U3-Pad28)")
-    (add_net "Net-(U3-Pad7)")
     (add_net "Net-(U7-Pad10)")
     (add_net "Net-(U7-Pad18)")
@@
       (solder_mask_margin 2.99974))
   )
-  (gr_text "HILTOP MAIN BOARD" (at 194.9 54.9) (layer F.SilkS)
-    (effects (font (size 1.4 1.4) (thickness 0.3)))
+  (gr_text "DEVTANK/HILTOP/M'BOARD/001\nP/N: 304-001\nRev: A" (at 184 54) (layer F.SilkS)
+    (effects (font (size 1 1) (thickness 0.15)) (justify left))
   )
   (gr_text USB2.0 (at 51.35 83.3 90) (layer F.SilkS)
@@
     (effects (font (size 1.2 1.2) (thickness 0.2)))
   )
-  (gr_text "Part No. 304-001 Iss1.0" (at 195.3 52.4) (layer F.SilkS)
-    (effects (font (size 1.4 1.4) (thickness 0.3)))
-  )
   (gr_line (start 220 50) (end 220 220) (angle 90) (layer Edge.Cuts) (width 0.15))
   (gr_line (start 220 220) (end 50 220) (angle 90) (layer Edge.Cuts) (width 0.15))
@@
   (via (at 139.5 187) (size 1) (drill 0.5) (layers F.Cu B.Cu) (net 0))
   (segment (start 139.065 84.455) (end 132.165001 91.355) (width 0.2) (layer F.Cu) (net 0))
+  (segment (start 95.649996 107.45) (end 95.6 107.499996) (width 0.25) (layer F.Cu) (net 0))
+  (segment (start 97.2 107.45) (end 95.649996 107.45) (width 0.25) (layer F.Cu) (net 0))
+  (via (at 95.6 107.499996) (size 0.8) (drill 0.4) (layers F.Cu B.Cu) (net 0))
+  (segment (start 90.1 102.35) (end 90.1 103.55) (width 0.25) (layer F.Cu) (net 0))
+  (segment (start 90.1 103.55) (end 90.5 103.95) (width 0.25) (layer F.Cu) (net 0))
+  (via (at 90.5 103.95) (size 0.8) (drill 0.4) (layers F.Cu B.Cu) (net 0))
+  (segment (start 93.1 111.05) (end 93.1 109.5) (width 0.25) (layer F.Cu) (net 0))
+  (segment (start 93.1 109.5) (end 93.05 109.45) (width 0.25) (layer F.Cu) (net 0))
+  (via (at 93.05 109.45) (size 0.8) (drill 0.4) (layers F.Cu B.Cu) (net 0))
+  (segment (start 95.6 111.05) (end 95.6 111.7) (width 0.25) (layer F.Cu) (net 0))
+  (segment (start 95.6 111.7) (end 96.2 112.3) (width 0.25) (layer F.Cu) (net 0))
+  (via (at 96.2 112.3) (size 0.8) (drill 0.4) (layers F.Cu B.Cu) (net 0))
+  (segment (start 97.2 109.45) (end 97.2 110.2) (width 0.25) (layer F.Cu) (net 0))
+  (via (at 97.2 110.2) (size 0.8) (drill 0.4) (layers F.Cu B.Cu) (net 0))
   (segment (start 137.5 195.5) (end 133.4 199.6) (width 2) (layer In2.Cu) (net 1))
   (segment (start 133.4 199.6) (end 119.1 199.6) (width 2) (layer In2.Cu) (net 1))
@@
   (segment (start 103.4 110.6) (end 104.6 110.6) (width 0.5) (layer F.Cu) (net 2))
   (via (at 104.6 110.6) (size 0.8) (drill 0.4) (layers F.Cu B.Cu) (net 2))
-  (segment (start 95.649996 107.45) (end 95.6 107.499996) (width 0.25) (layer F.Cu) (net 2))
-  (segment (start 97.2 107.45) (end 95.649996 107.45) (width 0.25) (layer F.Cu) (net 2))
-  (via (at 95.6 107.499996) (size 0.8) (drill 0.4) (layers F.Cu B.Cu) (net 2))
-  (segment (start 90.1 102.35) (end 90.1 103.55) (width 0.25) (layer F.Cu) (net 2))
-  (segment (start 90.1 103.55) (end 90.5 103.95) (width 0.25) (layer F.Cu) (net 2))
-  (via (at 90.5 103.95) (size 0.8) (drill 0.4) (layers F.Cu B.Cu) (net 2))
-  (segment (start 93.1 111.05) (end 93.1 109.5) (width 0.25) (layer F.Cu) (net 2))
-  (segment (start 93.1 109.5) (end 93.05 109.45) (width 0.25) (layer F.Cu) (net 2))
-  (via (at 93.05 109.45) (size 0.8) (drill 0.4) (layers F.Cu B.Cu) (net 2))
-  (segment (start 95.6 111.05) (end 95.6 111.7) (width 0.25) (layer F.Cu) (net 2))
-  (segment (start 95.6 111.7) (end 96.2 112.3) (width 0.25) (layer F.Cu) (net 2))
-  (via (at 96.2 112.3) (size 0.8) (drill 0.4) (layers F.Cu B.Cu) (net 2))
-  (segment (start 97.2 109.45) (end 97.2 110.2) (width 0.25) (layer F.Cu) (net 2))
-  (via (at 97.2 110.2) (size 0.8) (drill 0.4) (layers F.Cu B.Cu) (net 2))
   (segment (start 84.05 78.9) (end 83.7 78.9) (width 0.5) (layer F.Cu) (net 2))
   (via (at 83.2 78.4) (size 0.8) (drill 0.4) (layers F.Cu B.Cu) (net 2))

Commit message: Furthe progress on Schematics, assigned all main footprints using latest libraries, removed unwanted tracking and parts from original PCB layout
Parts:
- removed JP1: Jumper_NO_Small, Pin_Headers:Pin_Header_Straight_1x02_Pitch2.54mm
- removed the REF** at (204.0, 119.0)
- removed the REF** at (189.0, 116.0)
- removed the REF** at (87.7, 150.9)
- removed the REF** at (87.7, 148.1)
- removed the REF** at (100.5, 144.0)
- removed the REF** at (98.0, 144.0)
- removed the REF** at (95.5, 144.0)
- removed the REF** at (93.4, 144.4)
- removed the REF** at (88.4, 159.3)
- removed the REF** at (91.9, 159.9)
- removed the REF** at (89.6, 158.4)
- removed the REF** at (93.8, 156.4)
- removed the REF** at (101.1, 159.6)
- removed the REF** at (99.0, 159.5)
- removed the REF** at (94.0, 159.5)
- removed the REF** at (155.0, 98.0)
- removed the REF** at (152.0, 98.0)
- removed the REF** at (155.0, 95.0)
- removed the REF** at (149.0, 95.0) (x2)
- removed the REF** at (149.0, 101.0)
- removed the REF** at (143.0, 101.0)
- removed the REF** at (143.0, 98.0)
- removed the REF** at (91.8, 157.9)
- removed the REF** at (146.0, 101.0)
- removed the REF** at (146.0, 95.0)
- removed the REF** at (152.0, 95.0)
- removed the REF** at (146.0, 98.0)
- removed the REF** at (149.0, 98.0)
- removed the REF** at (143.0, 61.0)
- added C100: 4.7uF, Capacitor_SMD:C_0805_2012Metric, F.Cu at (171.3, 338.2)
- added C101: 470pF, Capacitor_SMD:C_0603_1608Metric, F.Cu at (191.5, 330.6)
- added C102: 2.2uF, Capacitor_SMD:C_0805_2012Metric, F.Cu at (186.4, 325.5)
- added C103: 9pF, Capacitor_SMD:C_0603_1608Metric, F.Cu at (202.4, 321.6)
- added C104: 9pF, Capacitor_SMD:C_0603_1608Metric, F.Cu at (184.2, 336.2)
- added C122: 100nF, Capacitor_SMD:C_0603_1608Metric, F.Cu at (168.4, 347.8)
- added C129: 100nF, Capacitor_SMD:C_0603_1608Metric, F.Cu at (186.6, 331.0)
- added C153: 4.7uF, Capacitor_SMD:C_0805_2012Metric, F.Cu at (194.0, 316.6)
- added C154: 470pF, Capacitor_SMD:C_0603_1608Metric, F.Cu at (191.1, 325.3)
- added C155: 100nF, Capacitor_SMD:C_0603_1608Metric, F.Cu at (188.7, 336.2)
- added C156: 100nF, Capacitor_SMD:C_0603_1608Metric, F.Cu at (186.5, 346.7)
- added C157: 100nF, Capacitor_SMD:C_0603_1608Metric, F.Cu at (177.5, 345.7)
- added C158: 47pF, Capacitor_SMD:C_0603_1608Metric, F.Cu at (193.3, 337.4)
- added C159: 47pF, Capacitor_SMD:C_0603_1608Metric, F.Cu at (196.1, 326.9)
- added C160: 100nF, Capacitor_SMD:C_0603_1608Metric, F.Cu at (184.6, 341.5)
- added C161: 47pF, Capacitor_SMD:C_0603_1608Metric, F.Cu at (200.2, 326.9)
- added C162: 47pF, Capacitor_SMD:C_0603_1608Metric, F.Cu at (196.1, 332.1)
- added C163: 47pF, Capacitor_SMD:C_0603_1608Metric, F.Cu at (182.0, 346.7)
- added C164: 47pF, Capacitor_SMD:C_0603_1608Metric, F.Cu at (189.1, 341.5)
- added C165: 47pF, Capacitor_SMD:C_0603_1608Metric, F.Cu at (200.2, 332.1)
- added C166: 47pF, Capacitor_SMD:C_0603_1608Metric, F.Cu at (204.4, 326.9)
- added C195: 1uF, Capacitor_SMD:C_0603_1608Metric, F.Cu at (244.3, 301.6)
- added C196: 22uF, Capacitor_SMD:C_0805_2012Metric, F.Cu at (239.1, 290.9)
- added C197: 10nF, Resistor_SMD:R_0402_1005Metric, F.Cu at (249.0, 306.3)
- added C198: 10nF, Resistor_SMD:R_0402_1005Metric, F.Cu at (259.0, 295.8)
- added C199: 10nF, Resistor_SMD:R_0402_1005Metric, F.Cu at (259.0, 300.8)
- added C200: 10nF, Resistor_SMD:R_0402_1005Metric, F.Cu at (253.1, 306.3)
- added C201: 100nF, Capacitor_SMD:C_0603_1608Metric, F.Cu at (249.6, 296.0)
- added C202: 100nF, Capacitor_SMD:C_0603_1608Metric, F.Cu at (234.6, 312.5)
- added C203: 100nF, Capacitor_SMD:C_0603_1608Metric, F.Cu at (239.6, 307.3)
- added C204: 100nF, Capacitor_SMD:C_0603_1608Metric, F.Cu at (257.6, 290.7)
- added C205: 100nF, Capacitor_SMD:C_0603_1608Metric, F.Cu at (244.5, 306.9)
- added C206: 100nF, Capacitor_SMD:C_0603_1608Metric, F.Cu at (254.5, 296.0)
- added C207: 100nF, Capacitor_SMD:C_0603_1608Metric, F.Cu at (249.6, 301.2)
- added C208: 1uF, Capacitor_SMD:C_0603_1608Metric, F.Cu at (239.2, 312.5)
- added C209: 100nF, Capacitor_SMD:C_0603_1608Metric, F.Cu at (244.5, 312.1)
- added C210: 22uF, Capacitor_SMD:C_0805_2012Metric, F.Cu at (235.0, 290.9)
- added C211: 100nF, Capacitor_SMD:C_0603_1608Metric, F.Cu at (254.5, 301.2)
- added C212: 100nF, Capacitor_SMD:C_0603_1608Metric, F.Cu at (247.8, 290.7)
- added C213: 100nF, Capacitor_SMD:C_0603_1608Metric, F.Cu at (252.7, 290.7)
- added C214: 100nF, Capacitor_SMD:C_0603_1608Metric, F.Cu at (244.7, 296.4)
- added C215: 100nF, Capacitor_SMD:C_0603_1608Metric, F.Cu at (229.7, 311.7)
- added C216: 100nF, Capacitor_SMD:C_0603_1608Metric, F.Cu at (234.6, 307.3)
- added C217: 22uF, Capacitor_SMD:C_0805_2012Metric, F.Cu at (224.4, 306.7)
- added C218: 100nF, Capacitor_SMD:C_0603_1608Metric, F.Cu at (235.6, 302.0)
- added C219: 100nF, Capacitor_SMD:C_0603_1608Metric, F.Cu at (239.7, 296.4)
- added C220: 100nF, Capacitor_SMD:C_0603_1608Metric, F.Cu at (229.0, 306.5)
- added C221: 22uF, Capacitor_SMD:C_0805_2012Metric, F.Cu at (235.2, 296.6)
- added C222: 22uF, Capacitor_SMD:C_0805_2012Metric, F.Cu at (243.3, 290.9)
- added C223: 100nF, Capacitor_SMD:C_0603_1608Metric, F.Cu at (224.8, 312.1)
- added C224: 100nF, Capacitor_SMD:C_0603_1608Metric, F.Cu at (193.2, 248.1)
- added C225: 100nF, Capacitor_SMD:C_0603_1608Metric, F.Cu at (178.5, 248.1)
- added C226: 100nF, Capacitor_SMD:C_0603_1608Metric, F.Cu at (266.3, 235.3)
- added C227: 100nF, Capacitor_SMD:C_0603_1608Metric, F.Cu at (183.4, 248.1)
- added C228: 100nF, Capacitor_SMD:C_0603_1608Metric, F.Cu at (178.5, 253.4)
- added C229: 100nF, Capacitor_SMD:C_0603_1608Metric, F.Cu at (266.3, 240.5)
- added C230: 100nF, Capacitor_SMD:C_0603_1608Metric, F.Cu at (183.4, 253.4)
- added C231: 100nF, Capacitor_SMD:C_0603_1608Metric, F.Cu at (178.5, 258.6)
- added C232: 100nF, Capacitor_SMD:C_0603_1608Metric, F.Cu at (188.3, 248.1)
- added C99: 100nF, Capacitor_SMD:C_0603_1608Metric, F.Cu at (198.7, 316.4)
- added D11: GRN, LED_SMD:LED_0603_1608Metric, F.Cu at (173.4, 369.2)
- added D12: YEL, LED_SMD:LED_0603_1608Metric, F.Cu at (151.4, 384.2)
- added D13: GRN, LED_SMD:LED_0603_1608Metric, F.Cu at (158.2, 379.0)
- added D14: YEL, LED_SMD:LED_0603_1608Metric, F.Cu at (179.7, 374.4)
- added D15: GRN, LED_SMD:LED_0603_1608Metric, F.Cu at (151.6, 373.7)
- added D16: YEL, LED_SMD:LED_0603_1608Metric, F.Cu at (166.5, 370.9)
- added D17: GRN, LED_SMD:LED_0603_1608Metric, F.Cu at (183.1, 374.4)
- added D25: YEL, LED_SMD:LED_0603_1608Metric, F.Cu at (176.4, 374.4)
- added D26: GRN, LED_SMD:LED_0603_1608Metric, F.Cu at (180.1, 369.2)
- added D27: YEL, LED_SMD:LED_0603_1608Metric, F.Cu at (180.4, 358.7)
- added D28: GRN, LED_SMD:LED_0603_1608Metric, F.Cu at (176.8, 369.2)
- added D29: YEL, LED_SMD:LED_0603_1608Metric, F.Cu at (173.4, 363.9)
- added D30: GRN, LED_SMD:LED_0603_1608Metric, F.Cu at (164.8, 381.4)
- added D31: YEL, LED_SMD:LED_0603_1608Metric, F.Cu at (169.0, 376.2)
- added D32: RED_LED, LED_SMD:LED_0603_1608Metric, F.Cu at (283.4, 258.7)
- added D33: RED_LED, LED_SMD:LED_0603_1608Metric, F.Cu at (314.0, 235.3)
- added D34: RED_LED, LED_SMD:LED_0603_1608Metric, F.Cu at (290.0, 258.7)
- added D35: RED_LED, LED_SMD:LED_0603_1608Metric, F.Cu at (294.5, 252.0)
- added D36: NUP2105L, Package_TO_SOT_SMD:SOT-23, F.Cu at (165.1, 341.7)
- added D37: NUP2105L, Package_TO_SOT_SMD:SOT-23, F.Cu at (180.2, 326.2)
- added FB10: 120R_100MHz, Resistor_SMD:R_0603_1608Metric, F.Cu at (227.5, 296.0)
- added FB11: 120R_100MHz, Resistor_SMD:R_0603_1608Metric, F.Cu at (227.8, 301.2)
- added FB6: 120R_100MHz, Resistor_SMD:R_0603_1608Metric, F.Cu at (217.0, 309.6)
- added FB7: 120R_100MHz, Resistor_SMD:R_0603_1608Metric, F.Cu at (217.0, 304.4)
- added FB9: 120R_100MHz, Resistor_SMD:R_0603_1608Metric, F.Cu at (227.5, 290.7)
- added FL1: PE-1812ACC510STS, Devtank_PCB_Lib:Inductor_PE-1812ACCXXXSTS, F.Cu at (137.2, 158.5)
- added FL2: PE-1812ACC510STS, Devtank_PCB_Lib:Inductor_PE-1812ACCXXXSTS, F.Cu at (148.1, 158.8)
- added J1: Conn_02x10_Odd_Even, Connector_PinHeader_2.54mm:PinHeader_2x10_P2.54mm_Vertical, F.Cu at (53.4, 94.5)
- added J20: CAMERA_PORT, Devtank_PCB_Lib:DSI_SFW15R-2STE1LF, F.Cu at (169.0, 129.6)
- added J21: EXT_FAN, Connector_Molex:Molex_KK-254_AE-6410-04A_1x04_P2.54mm_Vertical, F.Cu at (213.8, 92.9)
- added J22: SO-DIMM, Devtank_PCB_Lib:Conn_TE-DDR2-SODIMM-0.6-200P-ComputeModule, F.Cu at (91.8, 126.3)
- added J23: 1-5145154-2, Devtank_PCB_Lib:TE_1-5145154-2_PCI_120, F.Cu at (177.1, 114.3)
- added J24: Conn_02x10_Odd_Even, Connector_PinHeader_2.54mm:PinHeader_2x10_P2.54mm_Vertical, F.Cu at (60.3, 94.4)
- added L11: 15uH, Devtank_PCB_Lib:Inductor_MuRata_82103C, F.Cu at (163.5, 349.2)
- added L7: 15uH, Devtank_PCB_Lib:Inductor_MuRata_82103C, F.Cu at (178.6, 333.6)
- added Q5: ZXMN6A07F, Package_TO_SOT_SMD:SOT-23, F.Cu at (233.4, 98.0)
- added R157: 1K, Resistor_SMD:R_0603_1608Metric, F.Cu at (321.3, 245.8)
- added R158: 1K, Resistor_SMD:R_0603_1608Metric, F.Cu at (315.8, 251.4)
- added R159: 0R, Resistor_SMD:R_0603_1608Metric, F.Cu at (142.8, 38.2)
- added R167: 10K, Resistor_SMD:R_0603_1608Metric, F.Cu at (146.1, 27.3)
- added R168: DNF, Resistor_SMD:R_0402_1005Metric, F.Cu at (175.7, 31.9)
- added R169: DNF, Resistor_SMD:R_0402_1005Metric, F.Cu at (183.0, 31.8)
- added R170: DNF, Resistor_SMD:R_0402_1005Metric, F.Cu at (187.0, 28.8)
- added R171: DNF, Resistor_SMD:R_0402_1005Metric, F.Cu at (187.0, 30.8)
- added R172: DNF, Resistor_SMD:R_0402_1005Metric, F.Cu at (186.5, 26.3)
- added R173: DNF, Resistor_SMD:R_0402_1005Metric, F.Cu at (185.6, 32.6)
- added R174: 0R, Resistor_SMD:R_0603_1608Metric, F.Cu at (71.2, 374.5)
- added R175: DNF, Resistor_SMD:R_0603_1608Metric, F.Cu at (172.9, 345.7)
- added R176: DNF, Resistor_SMD:R_0603_1608Metric, F.Cu at (203.2, 316.4)
- added R177: R, Resistor_SMD:R_0603_1608Metric, F.Cu at (240.1, 301.6)
- added REF**: Via-0.6mm, KiCAD_PCB_Lib:Via-0.6mm, F.Cu at (138.4, 55.4)
- added U19: USB6B1, Package_SOIC:SOIC-8_3.9x4.9mm_P1.27mm, F.Cu at (73.8, 158.9)
- added U20: USB6B1, Package_SOIC:SOIC-8_3.9x4.9mm_P1.27mm, F.Cu at (95.3, 158.9)
- added U21: USB6B1, Package_SOIC:SOIC-8_3.9x4.9mm_P1.27mm, F.Cu at (89.3, 158.9)
- added U22: BQ32000, Package_SOIC:SOIC-8_3.9x4.9mm_P1.27mm, F.Cu at (136.3, 34.7)
- added U26: AT30TS75, Package_SOIC:SOIC-8_3.9x4.9mm_P1.27mm, F.Cu at (180.2, 27.5)
- added U29: AM1S-0505SZ, Devtank_PCB_Lib:CME_XXXX_S3C_PSU_MODULE, F.Cu at (131.8, 161.8)
- added U3: USB2517, Devtank_PCB_Lib:QFN-64-1EP_9x9mm_P0.5mm_EP4.7x4.7mm, F.Cu at (119.4, 84.4)
- added U30: MCP2517FD, Package_SOIC:SOIC-14_3.9x8.7mm_P1.27mm, F.Cu at (138.8, 129.3)
- added U31: MCP2517FD, Package_SOIC:SOIC-14_3.9x8.7mm_P1.27mm, F.Cu at (150.3, 129.6)
- added U32: AM1S-0505SZ, Devtank_PCB_Lib:CME_XXXX_S3C_PSU_MODULE, F.Cu at (157.4, 160.7)
- added U33: ADuM1201, Package_SOIC:SOIC-8_3.9x4.9mm_P1.27mm, F.Cu at (137.7, 139.5)
- added U34: ADuM1201, Package_SOIC:SOIC-8_3.9x4.9mm_P1.27mm, F.Cu at (149.7, 140.8)
- added U35: MCP2561FD, Package_SOIC:SOIC-8_3.9x4.9mm_P1.27mm, F.Cu at (137.5, 149.6)
- added U36: MCP2561FD, Package_SOIC:SOIC-8_3.9x4.9mm_P1.27mm, F.Cu at (149.3, 150.0)
- added U37: TUSB9260, Devtank_PCB_Lib:PQFP-64_7x7mm_P0.4mm_EP, F.Cu at (65.4, 85.8)
- added U5: SP3003-02XJ, Devtank_PCB_Lib:SC70-5, F.Cu at (114.0, 72.8)
- added Y3: 0.22F, Devtank_PCB_Lib:Battery_SD_V_SuperCap, F.Cu at (138.3, 29.2)
- added Y4: 32.768kHz, Crystal:Crystal_SMD_EuroQuartz_EQ161-2Pin_3.2x1.5mm, F.Cu at (144.1, 34.1)
- added Y5: 40MHz Crystal, Crystal:Crystal_SMD_SeikoEpson_FA238V-4Pin_3.2x2.5mm, F.Cu at (155.5, 345.5)
- added Y6: 40MHz Crystal, Crystal:Crystal_SMD_SeikoEpson_FA238V-4Pin_3.2x2.5mm, F.Cu at (144.4, 348.3)
- C1: value 10uF -> 100nF; footprint Capacitors_SMD:C_0805 -> Capacitor_SMD:C_1210_3225Metric; moved to F.Cu
- C10, C119, C4, C6: footprint Capacitors_SMD:CP_Elec_6.3x5.3 -> Capacitor_SMD:CP_Elec_6.3x5.3
- C105: value 4.7uF -> 9pF; footprint Capacitors_SMD:C_0805 -> Capacitor_SMD:C_0603_1608Metric
- C106, C109, C110, C112, C117, C118, C12, C121, C123, C124, C125, C126, C127, C128, C130, C131, C135, C136, C137, C138, C139, C14, C140, C141, C142, C143, C144, C145, C146, C147, C148, C149, C15, C150, C151, C152, C167, C169, C17, C173, C175, C176, C177, C180, C187, C188, C189, C19, C190, C191, C192, C20, C22, C23, C24, C25, C26, C5, C57, C61, C62, C8, C80, C81, C82, C83, C85, C86, C87, C88, C89, C90, C91, C92, C93, C94, C95, C96, C97: footprint Capacitors_SMD:C_0603 -> Capacitor_SMD:C_0603_1608Metric
- C107, C111, C113, C114, C115, C116, C170, C171, C172, C178, C184, C185, C193, C194, C27, C50, C63, C64, C69, C76, C78: footprint Capacitors_SMD:C_0805 -> Capacitor_SMD:C_0805_2012Metric
- C108: value 100nF -> 9pF; footprint Capacitors_SMD:C_0603 -> Capacitor_SMD:C_0603_1608Metric
- C11, C120, C16, C9: footprint Capacitors_SMD:CP_Elec_5x5.3 -> Capacitor_SMD:CP_Elec_5x5.3
- C13, C18, C3, C7: value 10uF -> 100uF; footprint Capacitors_SMD:C_0805 -> Capacitor_SMD:CP_Elec_6.3x7.7
- C132: footprint Capacitors_SMD:C_0603 -> Capacitor_SMD:C_0603_1608Metric_Pad0.84x1.00mm_HandSolder
- C133, C134, C168, C174: footprint Capacitors_SMD:C_1206 -> Capacitor_SMD:C_1206_3216Metric
- C179, C56, C58: value DNF -> 2.2uF; footprint Capacitors_SMD:C_1206 -> Capacitor_SMD:C_1206_3216Metric
- C181, C182, C183, C65: footprint Capacitors_SMD:C_1210 -> Capacitor_SMD:C_1210_3225Metric
- C186, C67: footprint Capacitors_SMD:CP_Elec_6.3x7.7 -> Capacitor_SMD:CP_Elec_6.3x7.7
- C2, C70: value 100nF -> 100uF; footprint Capacitors_SMD:C_0603 -> Capacitor_SMD:CP_Elec_6.3x7.7; moved to F.Cu
- C21: value 10uF -> 1uF; footprint Capacitors_SMD:C_0805 -> Capacitor_SMD:C_0603_1608Metric; moved to F.Cu
- C28, C36, C38, C39, C40, C41: value 22pF -> 100nF; footprint Capacitors_SMD:C_0603 -> Capacitor_SMD:C_0201_0603Metric
- C29, C37, C42: value 22pF -> 1uF; footprint Capacitors_SMD:C_0603 -> Capacitor_SMD:C_0201_0603Metric
- C30, C31, C33, C34, C51, C52, C54: footprint Capacitors_SMD:C_0603 -> Capacitor_SMD:C_0201_0603Metric
- C32: value 1nF -> 100nF; footprint Capacitors_SMD:C_0603 -> Capacitor_SMD:C_0201_0603Metric
- C35, C53, C55, C77: footprint Capacitors_SMD:C_0603 -> Capacitor_SMD:C_0201_0603Metric; moved to F.Cu
- C43, C46: value 22pF -> 470pF; footprint Capacitors_SMD:C_0603 -> Capacitor_SMD:C_0603_1608Metric
- C44: value 22pF -> 2.2uF; footprint Capacitors_SMD:C_0603 -> Capacitor_SMD:C_0805_2012Metric
- C45: value 22pF -> 4.7uF; footprint Capacitors_SMD:C_0603 -> Capacitor_SMD:C_0805_2012Metric
- C47, C48: value 22pF -> 12pF; footprint Capacitors_SMD:C_0603 -> Resistor_SMD:R_0603_1608Metric
- C49: value 22pF -> 100nF; footprint Capacitors_SMD:C_0603 -> Resistor_SMD:R_0603_1608Metric
- C59, C66, C71, C72, C73, C74, C75, C98: footprint Capacitors_SMD:C_0603 -> Capacitor_SMD:C_0603_1608Metric; moved to F.Cu
- C60: value 2200pF -> 100nF; footprint Capacitors_SMD:C_0603 -> Capacitor_SMD:C_0603_1608Metric
- C68: value 100nF -> 4.7uF; footprint Capacitors_SMD:C_0603 -> Capacitor_SMD:C_0805_2012Metric; moved to F.Cu
- C79: value 2.2uF -> 100uF; footprint Capacitors_SMD:C_0805 -> Capacitor_SMD:CP_Elec_6.3x7.7
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Connections:
- net /Ethernet/LEDG_K renamed /LEDG_K
- net /Ethernet/LEDY_K renamed /LEDY_K
- net /Ethernet/TR0_N renamed /TR0_N
- net /Ethernet/TR0_P renamed /TR0_P
- net /Ethernet/TR1_P renamed /TR1_P
- net /Ethernet/TR3_N renamed /TR3_N
- net /Ethernet/TR3_P renamed /TR3_P
- net /Processor/DISP1_CK_N renamed /DISP1_CK_N
- net /Processor/DISP1_CK_P renamed /DISP1_CK_P
- net /Processor/DISP1_D0_N renamed /DISP1_D0_N
- net /Processor/DISP1_D0_P renamed /DISP1_D0_P
- net /Processor/DISP1_D1_N renamed /DISP1_D1_N
- net /Processor/DISP1_D1_P renamed /DISP1_D1_P
- net /RETPower/PSU_ADC_ADDR renamed /AdjPower/PSU_ADC_ADDR
- net /RETPower/PSU_DAC_ADDR renamed /AdjPower/PSU_DAC_ADDR
- net /RETPower/VMON_1 renamed /AdjPower/VMON_1
- net /RETPower/VMON_2 renamed /AdjPower/VMON_2
- C1 pad 1: +5V -> GND
- C1 pad 2: GND -> Earth
- C105 pad 1: +3V3_ISO4 -> Net-(C105-Pad1)
- C105 pad 2: GND_ISO4 -> GND
- C108 pad 1: +3V3_ISO3 -> Net-(C108-Pad1)
- C108 pad 2: GND_ISO3 -> GND
- C13 pad 1: /USBHub/D7_5V -> /USBHub/PWR2_5V
- C15 pad 1: /USBHub/D7_5V -> +5V_ISO3
- C18 pad 1: /USBHub/D3_5V -> /USBHub/PWR2_5V
- C19 pad 1: /USBHub/D3_5V -> /USBHub/PWR2_5V
- C2 pad 1: +5V -> /USBHub/PWR1_5V
- C20 pad 1: /USBHub/D6_5V -> +5V_ISO4
- C21 pad 1: /USBHub/D6_5V -> Net-(C21-Pad1)
- C23 pad 1: GND -> +3V3
- C23 pad 2: +3V3 -> GND
- C28 pad 1: /USBHub/USB0_N -> Net-(C21-Pad1)
- C29 pad 1: /USBHub/USB0_P -> Net-(C29-Pad1)
- C3 pad 1: +5V -> /FR_PANEL_USB_PWR
- C30 pad 1: Net-(C30-Pad1) -> GND
- C30 pad 2: GND -> Net-(C30-Pad2)
- C31 pad 1: GND -> +3V3
- C31 pad 2: +5V -> GND
- C35 pad 1: +3V3 -> Net-(C29-Pad1)
- C36 pad 1: /LAN_USB_P -> +3V3
- C37 pad 1: /LAN_USB_N -> +3V3
- C38 pad 1: /FPGA_USB_P -> +3V3
- C39 pad 1: /FPGA_USB_N -> +3V3
- C40 pad 1: /USBHub/USB2_P -> +3V3
- C41 pad 1: /USBHub/USB3_P -> +3V3
- C42 pad 1: /USBHub/USB2_N -> +3V3
- C43 pad 1: /USBHub/USB3_N -> +5V_ISO3
- C43 pad 2: GND -> GND_ISO3
- C44 pad 1: /USBHub/USB6_P -> GND
- C44 pad 2: GND -> Net-(C44-Pad2)
- C45 pad 1: /USBHub/USB7_P -> +5V_ISO4
- C45 pad 2: GND -> GND_ISO4
- C46 pad 1: /USBHub/USB1_P -> +5V_ISO4
- C46 pad 2: GND -> GND_ISO4
- C47 pad 1: /USBHub/USB6_N -> Net-(C47-Pad1)
- C48 pad 1: /USBHub/USB7_N -> Net-(C48-Pad1)
- C49 pad 1: /USBHub/USB1_N -> +3V3
- C5 pad 1: +5V -> /FR_PANEL_USB_PWR
- C66 pad 2: -5V -> +3V3
- C68 pad 1: GND -> +CM_5V
- C68 pad 2: -5V -> GND
- C7 pad 1: /USBHub/D2_5V -> /USBHub/PWR1_5V
- C70 pad 1: GND -> Net-(C181-Pad2)
- C70 pad 2: -5V -> GND
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Routing:
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- added copper zone on In2.Cu, net ADJ_DC
- removed copper zone on In2.Cu, net +3V3
- removed copper zone on In2.Cu, net -5V
- removed copper zone on In1.Cu, net GND_ISO3
- removed copper zone on In1.Cu, net GND_ISO4
- removed copper zone on In2.Cu, net RET_DC
Other:
- board text removed: "USB2.0"

Commit message: Schematics complete - 1st draft
Parts:
- removed D34, D35: RED_LED, LED_SMD:LED_0603_1608Metric
- removed FID1, FID2: Fiducial_classic_Small_SilkscreenTop_Type1, Fiducials:Fiducial_classic_Small_SilkscreenTop_Type1
- removed G***: LOGO, KiCAD_PCB_Lib:Devtank_Rev2_Logo_Small
- removed JP2: Jumper_NO_Small, Pin_Headers:Pin_Header_Straight_1x02_Pitch2.54mm
- removed the REF** at (116.9, 195.2)
- removed the REF** at (194.0, 156.0)
- removed the REF** at (53.0, 53.5)
- removed the REF** at (51.5, 52.0)
- removed the REF** at (53.0, 52.0)
- removed the REF** at (54.5, 52.0)
- removed the REF** at (94.5, 59.0)
- removed the REF** at (93.0, 57.5)
- removed the REF** at (93.0, 59.0)
- removed the REF** at (93.0, 56.0)
- removed the REF** at (94.5, 57.5)
- removed the REF** at (94.5, 56.0)
- removed the REF** at (189.5, 158.5)
- removed the REF** at (93.0, 54.5)
- removed the REF** at (93.0, 53.0)
- removed the REF** at (94.5, 54.5)
- removed the REF** at (94.5, 53.0)
- removed the REF** at (91.5, 59.0)
- removed the REF** at (91.5, 57.5)
- removed the REF** at (91.5, 56.0)
- removed the REF** at (91.5, 54.5)
- removed the REF** at (91.5, 53.0)
- removed the REF** at (97.5, 51.5)
- removed the REF** at (186.5, 158.5)
- removed the REF** at (100.5, 51.5)
- removed the REF** at (99.0, 51.5)
- removed the REF** at (103.5, 51.5)
- removed the REF** at (102.0, 51.5)
- removed the REF** at (106.5, 51.5)
- removed the REF** at (105.0, 51.5)
- removed the REF** at (93.0, 51.5)
- removed the REF** at (91.5, 51.5)
- removed the REF** at (82.5, 51.5)
- removed the REF** at (84.0, 51.5)
- removed the REF** at (176.5, 159.5)
- removed the REF** at (85.5, 51.5)
- removed the REF** at (90.0, 51.5)
- removed the REF** at (88.5, 51.5)
- removed the REF** at (87.0, 51.5)
- removed the REF** at (96.0, 51.5)
- removed the REF** at (94.5, 51.5)
- removed the REF** at (142.4, 51.9)
- removed the REF** at (140.9, 51.9)
- removed the REF** at (139.4, 51.9)
- removed the REF** at (133.4, 51.9)
- removed the REF** at (183.0, 158.5)
- removed the REF** at (131.9, 51.9)
- removed the REF** at (148.4, 51.9)
- removed the REF** at (152.9, 51.9)
- removed the REF** at (149.9, 51.9)
- removed the REF** at (151.4, 51.9)
- removed the REF** at (155.9, 51.9)
- removed the REF** at (154.4, 51.9)
- removed the REF** at (146.9, 51.9)
- removed the REF** at (145.4, 51.9)
- removed the REF** at (143.9, 51.9)
- removed the REF** at (179.5, 158.5)
- removed the REF** at (137.9, 51.9)
- removed the REF** at (134.9, 51.9)
- removed the REF** at (136.4, 51.9)
- removed the REF** at (130.4, 51.9)
- removed the REF** at (128.9, 51.9)
- removed the REF** at (127.4, 51.9)
- removed the REF** at (127.5, 57.5)
- removed the REF** at (130.5, 57.5)
- removed the REF** at (129.0, 57.5)
- removed the REF** at (142.4, 50.4)
- removed the REF** at (183.0, 156.5)
- removed the REF** at (140.9, 50.4)
- removed the REF** at (139.4, 50.4)
- removed the REF** at (133.4, 50.4)
- removed the REF** at (131.9, 50.4)
- removed the REF** at (148.4, 50.4)
- removed the REF** at (152.9, 50.4)
- removed the REF** at (149.9, 50.4)
- removed the REF** at (151.4, 50.4)
- removed the REF** at (155.9, 50.4)
- removed the REF** at (154.4, 50.4)
- removed the REF** at (179.5, 156.5)
- removed the REF** at (146.9, 50.4)
- removed the REF** at (145.4, 50.4)
- removed the REF** at (143.9, 50.4)
- removed the REF** at (137.9, 50.4)
- removed the REF** at (134.9, 50.4)
- removed the REF** at (136.4, 50.4)
- removed the REF** at (130.4, 50.4)
- removed the REF** at (128.9, 50.4)
- removed the REF** at (127.4, 50.4)
- removed the REF** at (127.5, 56.0)
- removed the REF** at (164.5, 155.5)
- removed the REF** at (130.5, 56.0)
- removed the REF** at (129.0, 56.0)
- removed the REF** at (202.4, 51.9)
- removed the REF** at (200.9, 51.9)
- removed the REF** at (199.4, 51.9)
- removed the REF** at (197.9, 51.9)
- removed the REF** at (196.4, 51.9)
- removed the REF** at (194.9, 51.9)
- removed the REF** at (193.4, 51.9)
- removed the REF** at (191.9, 51.9)
- removed the REF** at (170.0, 155.5)
- removed the REF** at (190.4, 51.9)
- removed the REF** at (188.9, 51.9)
- removed the REF** at (187.4, 51.9)
- removed the REF** at (185.9, 51.9)
- removed the REF** at (184.4, 51.9)
- removed the REF** at (182.9, 51.9)
- removed the REF** at (181.4, 51.9)
- removed the REF** at (179.9, 51.9)
- removed the REF** at (178.4, 51.9)
- removed the REF** at (202.4, 50.4)
- removed the REF** at (116.9, 197.3)
- removed the REF** at (173.0, 156.5)
- removed the REF** at (200.9, 50.4)
- removed the REF** at (199.4, 50.4)
- removed the REF** at (197.9, 50.4)
- removed the REF** at (196.4, 50.4)
- removed the REF** at (194.9, 50.4)
- removed the REF** at (193.4, 50.4)
- removed the REF** at (191.9, 50.4)
- removed the REF** at (190.4, 50.4)
- removed the REF** at (188.9, 50.4)
- removed the REF** at (187.4, 50.4)
- removed the REF** at (175.5, 180.5)
- removed the REF** at (185.9, 50.4)
- removed the REF** at (184.4, 50.4)
- removed the REF** at (182.9, 50.4)
- removed the REF** at (181.4, 50.4)
- removed the REF** at (179.9, 50.4)
- removed the REF** at (178.4, 50.4)
- removed the REF** at (202.4, 48.9)
- removed the REF** at (200.9, 48.9)
- removed the REF** at (199.4, 48.9)
- removed the REF** at (197.9, 48.9)
- removed the REF** at (175.5, 177.5)
- removed the REF** at (196.4, 48.9)
- removed the REF** at (194.9, 48.9)
- removed the REF** at (193.4, 48.9)
- removed the REF** at (191.9, 48.9)
- removed the REF** at (190.4, 48.9)
- removed the REF** at (188.9, 48.9)
- removed the REF** at (187.4, 48.9)
- removed the REF** at (185.9, 48.9)
- removed the REF** at (184.4, 48.9)
- removed the REF** at (182.9, 48.9)
- removed the REF** at (172.5, 177.5)
- removed the REF** at (181.4, 48.9)
- removed the REF** at (179.9, 48.9)
- removed the REF** at (178.4, 48.9)
- removed the REF** at (202.4, 47.4)
- removed the REF** at (200.9, 47.4)
- removed the REF** at (199.4, 47.4)
- removed the REF** at (197.9, 47.4)
- removed the REF** at (196.4, 47.4)
- removed the REF** at (194.9, 47.4)
- removed the REF** at (193.4, 47.4)
- removed the REF** at (175.5, 174.0)
- removed the REF** at (191.9, 47.4)
- removed the REF** at (190.4, 47.4)
- removed the REF** at (188.9, 47.4)
- removed the REF** at (187.4, 47.4)
- removed the REF** at (185.9, 47.4)
- removed the REF** at (184.4, 47.4)
- removed the REF** at (182.9, 47.4)
- removed the REF** at (181.4, 47.4)
- removed the REF** at (179.9, 47.4)
- removed the REF** at (178.4, 47.4)
- removed the REF** at (172.5, 174.0)
- removed the REF** at (202.4, 45.9)
- removed the REF** at (200.9, 45.9)
- removed the REF** at (199.4, 45.9)
- removed the REF** at (197.9, 45.9)
- removed the REF** at (196.4, 45.9)
- removed the REF** at (194.9, 45.9)
- removed the REF** at (193.4, 45.9)
- removed the REF** at (191.9, 45.9)
- removed the REF** at (190.4, 45.9)
- removed the REF** at (188.9, 45.9)
- removed the REF** at (175.5, 171.0)
- removed the REF** at (187.4, 45.9)
- removed the REF** at (185.9, 45.9)
- removed the REF** at (184.4, 45.9)
- removed the REF** at (182.9, 45.9)
- removed the REF** at (181.4, 45.9)
- removed the REF** at (179.9, 45.9)
- removed the REF** at (178.4, 45.9)
- removed the REF** at (168.7, 48.4)
- removed the REF** at (167.2, 48.4)
- removed the REF** at (165.7, 48.4)
- removed the REF** at (198.4, 96.4)
- removed the REF** at (164.2, 48.4)
- removed the REF** at (162.7, 48.4)
- removed the REF** at (161.2, 48.4)
- removed the REF** at (159.7, 48.4)
- removed the REF** at (168.7, 46.9)
- removed the REF** at (167.2, 46.9)
- removed the REF** at (165.7, 46.9)
- removed the REF** at (164.2, 46.9)
- removed the REF** at (162.7, 46.9)
- removed the REF** at (161.2, 46.9)
- removed the REF** at (216.5, 122.0)
- removed the REF** at (159.7, 46.9)
- removed the REF** at (155.9, 48.9)
- removed the REF** at (154.4, 48.9)
- removed the REF** at (152.9, 48.9)
- removed the REF** at (151.4, 48.9)
- removed the REF** at (149.9, 48.9)
- removed the REF** at (148.4, 48.9)
- removed the REF** at (146.9, 48.9)
- removed the REF** at (145.4, 48.9)
- removed the REF** at (143.9, 48.9)
- removed the REF** at (213.9, 63.9)
- removed the REF** at (142.4, 48.9)
- removed the REF** at (140.9, 48.9)
- removed the REF** at (139.4, 48.9)
- removed the REF** at (137.9, 48.9)
- removed the REF** at (136.4, 48.9)
- removed the REF** at (134.9, 48.9)
- removed the REF** at (133.4, 48.9)
- removed the REF** at (131.9, 48.9)
- removed the REF** at (130.4, 48.9)
- removed the REF** at (128.9, 48.9)
- removed the REF** at (115.7, 195.2)
- removed the REF** at (213.9, 68.4)
- removed the REF** at (127.4, 48.9)
- removed the REF** at (130.5, 54.5)
- removed the REF** at (129.0, 54.5)
- removed the REF** at (127.5, 54.5)
- removed the REF** at (126.0, 54.5)
- removed the REF** at (124.5, 54.5)
- removed the REF** at (123.0, 54.5)
- removed the REF** at (121.5, 54.5)
- removed the REF** at (120.0, 54.5)
- removed the REF** at (118.5, 54.5)
- removed the REF** at (210.9, 68.4)
- removed the REF** at (117.0, 54.5)
- removed the REF** at (115.5, 54.5)
- removed the REF** at (114.0, 54.5)
- removed the REF** at (112.5, 54.5)
- removed the REF** at (111.0, 54.5)
- removed the REF** at (109.5, 54.5)
- removed the REF** at (155.9, 47.4)
- removed the REF** at (154.4, 47.4)
- removed the REF** at (152.9, 47.4)
- removed the REF** at (151.4, 47.4)
- removed the REF** at (210.9, 63.9)
- removed the REF** at (149.9, 47.4)
- removed the REF** at (148.4, 47.4)
- removed the REF** at (146.9, 47.4)
- removed the REF** at (145.4, 47.4)
- removed the REF** at (143.9, 47.4)
- removed the REF** at (142.4, 47.4)
- removed the REF** at (140.9, 47.4)
- removed the REF** at (139.4, 47.4)
- removed the REF** at (137.9, 47.4)
- removed the REF** at (136.4, 47.4)
- removed the REF** at (207.4, 68.4)
- removed the REF** at (134.9, 47.4)
- removed the REF** at (133.4, 47.4)
- removed the REF** at (131.9, 47.4)
- removed the REF** at (130.4, 47.4)
- removed the REF** at (128.9, 47.4)
- removed the REF** at (127.4, 47.4)
- removed the REF** at (130.5, 53.0)
- removed the REF** at (129.0, 53.0)
- removed the REF** at (127.5, 53.0)
- removed the REF** at (126.0, 53.0)
- removed the REF** at (207.4, 63.9)
- removed the REF** at (124.5, 53.0)
- removed the REF** at (123.0, 53.0)
- removed the REF** at (121.5, 53.0)
- removed the REF** at (120.0, 53.0)
- removed the REF** at (118.5, 53.0)
- removed the REF** at (117.0, 53.0)
- removed the REF** at (115.5, 53.0)
- removed the REF** at (114.0, 53.0)
- removed the REF** at (112.5, 53.0)
- removed the REF** at (111.0, 53.0)
- removed the REF** at (195.0, 113.5)
- removed the REF** at (109.5, 53.0)
- removed the REF** at (155.9, 45.9)
- removed the REF** at (154.4, 45.9)
- removed the REF** at (152.9, 45.9)
- removed the REF** at (151.4, 45.9)
- removed the REF** at (149.9, 45.9)
- removed the REF** at (148.4, 45.9)
- removed the REF** at (146.9, 45.9)
- removed the REF** at (145.4, 45.9)
- removed the REF** at (143.9, 45.9)
- removed the REF** at (190.4, 104.9)
- removed the REF** at (142.4, 45.9)
- removed the REF** at (140.9, 45.9)
- removed the REF** at (139.4, 45.9)
- removed the REF** at (137.9, 45.9)
- removed the REF** at (136.4, 45.9)
- removed the REF** at (134.9, 45.9)
- removed the REF** at (133.4, 45.9)
- removed the REF** at (131.9, 45.9)
- removed the REF** at (130.4, 45.9)
- removed the REF** at (128.9, 45.9)
- removed the REF** at (190.4, 101.4)
- removed the REF** at (127.4, 45.9)
- removed the REF** at (130.5, 51.5)
- removed the REF** at (129.0, 51.5)
- removed the REF** at (127.5, 51.5)
- removed the REF** at (126.0, 51.5)
- removed the REF** at (124.5, 51.5)
- removed the REF** at (123.0, 51.5)
- removed the REF** at (121.5, 51.5)
- removed the REF** at (120.0, 51.5)
- removed the REF** at (118.5, 51.5)
- removed the REF** at (190.4, 97.9)
- removed the REF** at (117.0, 51.5)
- removed the REF** at (115.5, 51.5)
- removed the REF** at (114.0, 51.5)
- removed the REF** at (112.5, 51.5)
- removed the REF** at (111.0, 51.5)
- removed the REF** at (89.2, 69.7)
- removed the REF** at (94.2, 69.9)
- removed the REF** at (188.0, 188.5)
- removed the REF** at (186.0, 188.5)
- removed the REF** at (184.0, 188.5)
- removed the REF** at (184.4, 106.9)
- removed the REF** at (182.0, 188.5)
- removed the REF** at (188.0, 186.5)
- removed the REF** at (186.0, 186.5)
- removed the REF** at (184.0, 186.5)
- removed the REF** at (182.0, 186.5)
- removed the REF** at (188.0, 184.5)
- removed the REF** at (186.0, 184.5)
- removed the REF** at (184.0, 184.5)
- removed the REF** at (182.0, 184.5)
- removed the REF** at (188.0, 182.5)
- removed the REF** at (115.7, 197.2)
- removed the REF** at (181.9, 104.4)
- removed the REF** at (186.0, 182.5)
- removed the REF** at (184.0, 182.5)
- removed the REF** at (182.0, 182.5)
- removed the REF** at (188.0, 180.5)
- removed the REF** at (186.0, 180.5)
- removed the REF** at (184.0, 180.5)
- removed the REF** at (182.0, 180.5)
- removed the REF** at (188.0, 178.5)
- removed the REF** at (186.0, 178.5)
- removed the REF** at (184.0, 178.5)
- removed the REF** at (161.9, 103.4)
- removed the REF** at (182.0, 178.5)
- removed the REF** at (193.5, 170.0)
- removed the REF** at (191.5, 170.0)
- removed the REF** at (189.5, 170.0)
- removed the REF** at (187.5, 170.0)
- removed the REF** at (191.0, 172.0)
- removed the REF** at (193.5, 168.0)
- removed the REF** at (191.5, 168.0)
- removed the REF** at (189.5, 168.0)
- removed the REF** at (187.5, 168.0)
- removed the REF** at (178.4, 87.4)
- removed the REF** at (185.5, 168.0)
- removed the REF** at (193.5, 166.0)
- removed the REF** at (191.5, 166.0)
- removed the REF** at (189.5, 166.0)
- removed the REF** at (187.5, 166.0)
- removed the REF** at (185.5, 166.0)
- removed the REF** at (216.0, 204.5)
- removed the REF** at (214.0, 204.5)
- removed the REF** at (212.0, 204.5)
- removed the REF** at (210.0, 204.5)
- removed the REF** at (185.4, 77.4)
- removed the REF** at (208.0, 204.5)
- removed the REF** at (216.0, 202.5)
- removed the REF** at (214.0, 202.5)
- removed the REF** at (212.0, 202.5)
- removed the REF** at (210.0, 202.5)
- removed the REF** at (208.0, 202.5)
- removed the REF** at (216.0, 200.5)
- removed the REF** at (214.0, 200.5)
- removed the REF** at (212.0, 200.5)
- removed the REF** at (210.0, 200.5)
- removed the REF** at (185.4, 90.9)
- removed the REF** at (208.0, 200.5)
- removed the REF** at (202.0, 204.5)
- removed the REF** at (200.0, 204.5)
- removed the REF** at (198.0, 204.5)
- removed the REF** at (196.0, 204.5)
- removed the REF** at (194.0, 203.0)
- removed the REF** at (192.5, 204.5)
- removed the REF** at (202.0, 202.5)
- removed the REF** at (200.0, 202.5)
- removed the REF** at (198.0, 202.5)
- removed the REF** at (181.9, 94.9)
- removed the REF** at (190.5, 199.0)
- removed the REF** at (189.5, 201.0)
- removed the REF** at (192.0, 202.0)
- removed the REF** at (202.0, 200.5)
- removed the REF** at (200.0, 200.5)
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Connections:
- net /AdjPower/PSU_ADC_ADDR renamed Net-(R123-Pad1)
- net /AdjPower/PSU_DAC_ADDR renamed Net-(R118-Pad1)
- net /PWR_ENABLE renamed Net-(D66-Pad3)
- net /RS485/RS485_CH1_DE renamed Net-(R81-Pad1)
- C195 pad 1: +1V2_SATA -> +1V1_SATA
- C196 pad 1: +1V2_SATA -> +1V1_SATA
- C197 pad 1: (no net) -> Net-(C197-Pad1)
- C197 pad 2: (no net) -> /SATA_Bridge/CAP_SATATXM
- C198 pad 1: (no net) -> Net-(C198-Pad1)
- C198 pad 2: (no net) -> /SATA_Bridge/CAP_SATATXP
- C199 pad 1: (no net) -> Net-(C199-Pad1)
- C199 pad 2: (no net) -> /SATA_Bridge/CAP_SATARXM
- C200 pad 1: (no net) -> Net-(C200-Pad1)
- C200 pad 2: (no net) -> /SATA_Bridge/CAP_SATARXP
- C201 pad 1: +1V2_SATA -> +1V1_SATA
- C202 pad 1: +1V2_SATA -> +1V1_SATA
- C203 pad 1: +1V2_SATA -> +1V1_SATA
- C204 pad 1: +1V8_SATA -> Net-(C204-Pad1)
- C204 pad 2: GND -> Net-(C204-Pad2)
- C205 pad 1: +1V2_SATA -> +1V1_SATA
- C206 pad 1: +1V8_SATA -> Net-(C206-Pad1)
- C206 pad 2: GND -> Net-(C204-Pad2)
- C207 pad 1: +1V2_SATA -> +1V1_SATA
- C208 pad 1: +1V8_SATA -> +3V3
- C209 pad 1: +1V2_SATA -> +1V1_SATA
- C210 pad 1: +1V8_SATA -> Net-(C210-Pad1)
- C211 pad 1: +1V2_SATA -> +1V1_SATA
- C212 pad 1: +1V2_SATA -> +1V1_SATA
- C213 pad 1: +1V2_SATA -> +1V1_SATA
- C214 pad 1: +1V2_SATA -> +1V1_SATA
- C217 pad 1: +1V2_USB2_SATA -> +3V3
- C219 pad 1: +1V2_USB2_SATA -> +3V3
- C226 pad 1: +5V -> GND
- C226 pad 2: GND -> +3V3
- C227 pad 1: +5V -> GND
- C227 pad 2: GND -> Net-(C227-Pad2)
- C228 pad 2: -5V -> +3V3
- C229 pad 1: +12V -> GND
- C229 pad 2: GND -> Net-(C229-Pad2)
- C230 pad 1: +12V -> GND
- C230 pad 2: GND -> Net-(C230-Pad2)
- C231 pad 1: ADJ_DC -> GND
- C231 pad 2: GND -> Net-(C231-Pad2)
- C232 pad 1: ADJ_DC -> +3V3
- C50 pad 1: Net-(C50-Pad1) -> GND
- C74 pad 1: +12V -> GND
- C74 pad 2: GND -> Net-(C50-Pad2)
- C75 pad 1: +12V -> GND
- C75 pad 2: GND -> Net-(C119-Pad2)
- C77 pad 1: +12V -> GND
- C77 pad 2: GND -> +3V3
- D32 pad 1: GND -> Net-(D32-Pad1)
- D32 pad 2: Net-(D32-Pad2) -> +3V3
- D33 pad 1: GND -> Net-(D33-Pad1)
- D33 pad 2: Net-(D33-Pad2) -> +3V3
- EXP2 pad 1: +5V -> +3V3
- EXP2 pad 10: /SYS_CLK1 -> /DEBUG_RX
- EXP2 pad 11: GND -> /SPI1_CS1_CAM_IO0
- EXP2 pad 12: /SYS_PWM1 -> /SPI1_CS0
- EXP2 pad 13: GND -> /PR_GPIO27
- EXP2 pad 14: (no net) -> GND
- EXP2 pad 15: (no net) -> /PR_GPIO22
- EXP2 pad 16: (no net) -> /PR_GPIO23
- EXP2 pad 17: (no net) -> +3V3
- EXP2 pad 18: GND -> /PR_GPIO24
- EXP2 pad 19: (no net) -> /SPI0_MOSI
- EXP2 pad 20: (no net) -> GND
- EXP2 pad 21: (no net) -> /SPI0_MISO
- EXP2 pad 22: (no net) -> /PR_GPIO25
- EXP2 pad 23: GND -> /SPI0_SCLK
- EXP2 pad 24: (no net) -> /SPI0_CS0
- EXP2 pad 25: (no net) -> GND
- EXP2 pad 26: (no net) -> /SPI0_CS1
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Routing:
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