File: HILTOP_motherboard/HILTOP_Motherboard.kicad_pcb (KiCad board)
At the start: 6 copper layers, 170 x 170 mm, 758 parts, among them J1 BACKPLANE_PWR, J10 HDMI, J11 DISP_PWR, J12 DISPLAY_PORT, J13 DDR2_SODIMM_COMPUTE_MODULE_3, J14 VADJ_B, J15 VADJ_A, J16 SOFT_START_PWR, J17 PWR_LED, J18 USB_B, J19 Micro_SD_Card, J2 ATX_MOLEX_02X12, J20 CAMERA_PORT, J21 EXT_FAN, J22 BACKPLANE_LV_PWR, J23 EXT_FAN, J24 HILTOP_PCIE-64_CONN, J25 DEBUG, J26 IO_EXP, J3 SATA, J4 USB_A_DOUBLE, J5 USB FRONT PANEL, J6 CAN, J7 RS485, J8 EXT_TEMP_MON, J9 RJ45-TRANS_SI-61001-F, Q1 Si7148DP-T1-E3, Q2 Si7148DP-T1-E3, Q3 2N7002, Q4 2N7002, Q5 ZXMN6A07F, Q6 ZXMN6A07F, Q7 ZXMN6A07F, Q8 SSM3J328R, U1 LM337BD2TG, U10 TLC271, U11 ADS1015, U12 MCP4725, U13 CME0505S3C, U14 SP3003-02XJ, U15 ISO3080, U16 ISO3080, U17 CME0505S3C, U18 USB6B1, U19 USB6B1, U2 MIC2026-1YM, U20 USB6B1, U21 USB6B1, U22 BQ32000, U23 TPD12S016, U24 MAX16054, U25 STM6719SFWB6F, U26 LM75B, U27 TPS54394, U28 LP2985, U29 CME0505S3C, U3 USB2517, U30 MCP2517FD, U31 MCP2517FD, U32 CME0505S3C, U33 ADuM1201, U34 ADuM1201, U35 MCP2561FD, U36 MCP2561FD, U37 TUSB9261, U38 AT25DN512CSSHF-B, U39 MCP23017, U4 MIC2026-1YM, U40 SP3003-02XJ, U41 CP2102N-A01-GQFN24, U43 MAX3107, U44 MAX3107, U45 93AAxxA, U5 SP3003-02XJ, U6 SP3003-02XJ, U7 LAN7500, U8 LM5118, U9 INA250A3, Y1 24MHz Crystal, Y2 25MHz Crystal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

Commit message: DRC checks complete, all errors and warnings cleared. BOM created and parts rationalised.
Parts:
- C132: footprint Capacitor_SMD:C_0603_1608Metric_Pad0.84x1.00mm_HandSolder -> Capacitor_SMD:C_0402_1005Metric
- C151: footprint Capacitor_SMD:C_0603_1608Metric -> Capacitor_SMD:C_0402_1005Metric
- C29, C37, C42: footprint Capacitor_SMD:C_0201_0603Metric -> Capacitor_SMD:C_0603_1608Metric
- C30, C31, C32, C33, C34, C35, C36, C38, C39, C40, C41, C51, C52, C54: footprint Capacitor_SMD:C_0201_0603Metric -> Capacitor_SMD:C_0402_1005Metric
- moved C67 7.40 mm to (201.9, 159.4)
- moved C186 7.03 mm to (209.2, 159.4)
- moved C18 0.07 mm to (144.3, 64.7)
Routing:
- net GND: track 383.7 -> 385.0 mm, vias 204 -> 205
- net (no net): track 21.9 -> 20.6 mm, vias 2 -> 1

Commit message: tracking updates
Parts:
- C117, C118, C180, C187, C188, C189, C190, C191, C192, C57: value 100n -> 100nF
- C184, C185, C193, C194, C64: footprint Capacitor_SMD:C_0805_2012Metric -> Capacitor_SMD:C_0603_1608Metric
- C196, C221, C222: footprint Capacitor_SMD:C_0805_2012Metric -> Capacitor_SMD:C_1206_3216Metric
- R65, R66, R67, R68: footprint Resistor_SMD:R_0603_1608Metric_Pad0.84x1.00mm_HandSolder -> Resistor_SMD:R_0603_1608Metric
- moved TP24 5.18 mm to (76.9, 141.1)
- moved TP61 1.67 mm to (82.2, 130.8)
- moved R221 1.19 mm to (81.9, 132.6)
- moved TP62 1.03 mm to (56.1, 129.8)
- moved R222 1.01 mm to (55.3, 132.1)
- moved C199 0.71 mm to (61.2, 78.3)
- moved TP94 0.71 mm to (76.1, 131.1)
- moved C200 0.64 mm to (60.0, 78.3)
- moved TP81 0.51 mm to (67.2, 127.7)
- moved TP85 0.49 mm to (80.3, 127.9)
- moved C197 0.48 mm to (64.5, 78.2)
- moved C198 0.46 mm to (63.3, 78.3)
- moved TP77 0.39 mm to (62.2, 127.7)
- moved C228 0.25 mm to (59.2, 131.7)
- moved C229 0.25 mm to (60.9, 131.7)
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Connections:
- net /SATA_Bridge/CAP_SATARXM renamed /SATA_Bridge/CAP_SATARX_N
- net /SATA_Bridge/CAP_SATARXP renamed /SATA_Bridge/CAP_SATARX_P
- net Net-(C197-Pad1) renamed /SATA_Bridge/TX_N
- net Net-(C198-Pad1) renamed /SATA_Bridge/TX_P
- net Net-(C199-Pad1) renamed /SATA_Bridge/RX_N
- net Net-(C200-Pad1) renamed /SATA_Bridge/RX_P
- C197 pad 2: /SATA_Bridge/CAP_SATATXM -> /SATA_Bridge/CAP_SATATX_P
- C198 pad 2: /SATA_Bridge/CAP_SATATXP -> /SATA_Bridge/CAP_SATATX_N
- J3 pad 2: /SATA_Bridge/CAP_SATATXP -> /SATA_Bridge/CAP_SATATX_P
- J3 pad 3: /SATA_Bridge/CAP_SATATXM -> /SATA_Bridge/CAP_SATATX_N
Routing:
- net /SPI0_MISO: track 0.00 -> 65.4 mm, vias 0 -> 1
- net /SPI0_MOSI: track 0.00 -> 56.5 mm, vias 0 -> 2
- net /UART_CH2_IRQ: track 0.00 -> 54.8 mm, vias 0 -> 1
- net /SPI0_SCLK: track 0.00 -> 49.6 mm
- net +3V3: track 195.3 -> 240.4 mm, vias 44 -> 51
- net GND: track 385.0 -> 421.3 mm, vias 205 -> 224
- net /UART_CH1_IRQ: track 0.00 -> 35.2 mm, vias 0 -> 1
- net Net-(R223-Pad1): track 0.00 -> 33.9 mm, vias 0 -> 2
- net Net-(U16-Pad6): track 0.00 -> 10.3 mm, vias 0 -> 2
- net Net-(U15-Pad6): track 0.00 -> 10.2 mm, vias 0 -> 2
- net Net-(U43-Pad24): track 0.00 -> 8.36 mm
- net Net-(U44-Pad24): track 0.00 -> 8.27 mm
- net /~MASTER_RESET: track 9.25 -> 17.4 mm
- net Net-(U43-Pad1): track 0.00 -> 7.79 mm
- net Net-(U44-Pad1): track 0.00 -> 7.72 mm
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