File: HILTOP_motherboard/ice40_FPGA.sch (KiCad schematic (older format))
At the start: 15 parts, among them J1 Lattice_ice40-HX8KBreakoutBoa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

Commit message: Added new USB2.0 device
Changed lines of the file:
@@
 LIBS:regul
 LIBS:references
-LIBS:pspice
 LIBS:Power_Management
 LIBS:powerint
@@
 LIBS:Diode
 LIBS:digital-audio
-LIBS:device
 LIBS:Decawave
 LIBS:dc-dc
@@
 LIBS:adc-dac
 LIBS:ac-dc
+LIBS:device
 LIBS:HILTOP_Motherboard-cache
 EELAYER 25 0
@@
 $Descr A3 16535 11693
 encoding utf-8
-Sheet 5 8
+Sheet 5 9
 Title "HILTOP Motherboard"
 Date "26th January 2018"
@@
 Wire Wire Line
 	6300 4150 6850 4150
+Text HLabel 3500 2750 0    60   Input ~ 0
+USB_N
+Text HLabel 3500 2900 0    60   Input ~ 0
+USB_P
 $EndSCHEMATC

Commit message: Added more detail to motherboard schemas
Parts:
- removed unit 1 of J1
- removed unit 2 of J1
- added J?: SO-DIMM, symbol SO-DIMM
Other:
- moved on the sheet: J1C, J1D, R140, R141, R84, R86, R87, R88, R89, R90, R92, R93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

Commit message: Updated pinouts for Backplane and Compute Module
Connections:
- net labels removed: PWR_LED
Changed lines of the file:
@@
 $Descr A3 16535 11693
 encoding utf-8
-Sheet 5 11
+Sheet 5 12
 Title "HILTOP Motherboard"
 Date "26th January 2018"
@@
 Text HLabel 18425 15375 0    60   Output ~ 0
 PWR_ENABLE
-Text HLabel 18425 15275 0    60   Output ~ 0
-PWR_LED
 Text HLabel 25075 19125 2    60   Output ~ 0
 FP_GPIO_1

Commit message: Furthe progress on Schematics, assigned all main footprints using latest libraries, removed unwanted tracking and parts from original PCB layout
Parts:
- removed J1: Lattice_ice40-HX8KBreakoutBoard, KiCAD_PCB_Lib:ice40HX8KDevBrd_Header_2.54mm, symbol Lattice_ice40-HX8KBreakoutBoard
- J22: renamed from J?; footprint (none) -> Devtank_PCB_Lib:Conn_TE-DDR2-SODIMM-0.6-200P-ComputeModule
- R140, R141, R84, R86, R87, R88, R89, R90, R92, R93, R94, R95, R96, R97: footprint Resistors_SMD:R_0603 -> Resistor_SMD:R_0603_1608Metric

Commit message: Schematics complete - 1st draft
Parts:
- J22: symbol SO-DIMM -> Devtank:SO-DIMM
- R140, R141, R84, R86, R87, R88, R89, R90, R92, R93, R94, R95, R96, R97: symbol R -> device:R
Changed lines of the file:
@@
-EESchema Schematic File Version 2
-LIBS:HILTOP_Motherboard-rescue
-LIBS:Devtank
-LIBS:Zilog
-LIBS:zetex
-LIBS:xilinx
-LIBS:Xicor
-LIBS:Worldsemi
-LIBS:wiznet
-LIBS:video
-LIBS:Valve
-LIBS:triac_thyristor
-LIBS:Transistor
-LIBS:Transformer
-LIBS:texas
-LIBS:Switch
-LIBS:supertex
-LIBS:siliconi
-LIBS:silabs
-LIBS:sensors
-LIBS:Sensor_Humidity
-LIBS:Sensor_Current
-LIBS:RFSolutions
-LIBS:rfcom
-LIBS:RF_Bluetooth
-LIBS:Relay
-LIBS:regul
-LIBS:references
-LIBS:Power_Management
-LIBS:powerint
-LIBS:power
-LIBS:philips
-LIBS:Oscillators
-LIBS:opto
-LIBS:onsemi
-LIBS:nxp
-LIBS:nordicsemi
-LIBS:motorola
-LIBS:motor_drivers
-LIBS:Motor
-LIBS:modules
-LIBS:microcontrollers
-LIBS:microchip
-LIBS:memory
-LIBS:Mechanical
-LIBS:MCU_Texas_MSP430
-LIBS:MCU_ST_STM32
-LIBS:MCU_ST_STM8
-LIBS:MCU_Parallax
-LIBS:MCU_NXP_S08
-LIBS:MCU_NXP_LPC
-LIBS:MCU_NXP_Kinetis
-LIBS:MCU_Microchip_PIC32
-LIBS:MCU_Microchip_PIC24
-LIBS:MCU_Microchip_PIC18
-LIBS:MCU_Microchip_PIC16
-LIBS:MCU_Microchip_PIC12
-LIBS:MCU_Microchip_PIC10
-LIBS:maxim
-LIBS:Logic_TTL_IEEE
-LIBS:logic_programmable
-LIBS:Logic_CMOS_IEEE
-LIBS:Logic_CMOS_4000
-LIBS:Logic_74xx
-LIBS:Logic_74xgxx
-LIBS:linear
-LIBS:LEM
-LIBS:LED
-LIBS:Lattice
-LIBS:ir
-LIBS:intersil
-LIBS:interface
-LIBS:intel
-LIBS:infineon
-LIBS:hc11
-LIBS:Graphic
-LIBS:gennum
-LIBS:ftdi
-LIBS:FPGA_Actel
-LIBS:Espressif
-LIBS:ESD_Protection
-LIBS:elec-unifil
-LIBS:DSP_Microchip_DSPIC33
-LIBS:dsp
-LIBS:driver_gate
-LIBS:Display
-LIBS:Diode
-LIBS:digital-audio
-LIBS:Decawave
-LIBS:dc-dc
-LIBS:cypress
-LIBS:contrib
-LIBS:Connector
-LIBS:brooktre
-LIBS:Bosch
-LIBS:bbd
-LIBS:Battery_Management
-LIBS:audio
-LIBS:atmel
-LIBS:analog_switches
-LIBS:analog_devices
-LIBS:Altera
-LIBS:adc-dac
-LIBS:ac-dc
-LIBS:device
+EESchema Schematic File Version 4
 LIBS:HILTOP_Motherboard-cache
-EELAYER 25 0
+EELAYER 26 0
 EELAYER END
 $Descr A3 16535 11693
@@
 $EndDescr
 $Comp
-L +3V3 #PWR0214
+L power:+3V3 #PWR213
 U 1 1 589A308F
 P 21025 14075
-F 0 "#PWR0214" H 21025 13925 50  0001 C CNN
+F 0 "#PWR213" H 21025 13925 50  0001 C CNN
 F 1 "+3V3" V 21025 14275 50  0000 C CNN
 F 2 "" H 21025 14075 50  0000 C CNN
@@
 $EndComp
 $Comp
-L +1V2 #PWR0215
+L power:+1V2 #PWR210
 U 1 1 589A3092
 P 20825 14075
-F 0 "#PWR0215" H 20825 13925 50  0001 C CNN
+F 0 "#PWR210" H 20825 13925 50  0001 C CNN
 F 1 "+1V2" V 20825 14275 50  0000 C CNN
 F 2 "" H 20825 14075 50  0000 C CNN
@@
 $EndComp
 $Comp
-L GND #PWR0216
+L power:GND #PWR220
 U 1 1 589A30AC
 P 24575 16575
-F 0 "#PWR0216" H 24575 16325 50  0001 C CNN
+F 0 "#PWR220" H 24575 16325 50  0001 C CNN
 F 1 "GND" H 24575 16425 50  0000 C CNN
 F 2 "" H 24575 16575 50  0000 C CNN
@@
 SYS_CLK1
 $Comp
-L +2V5 #PWR0217
+L power:+2V5 #PWR211
 U 1 1 5911AE45
 P 20925 14075
-F 0 "#PWR0217" H 20925 13925 50  0001 C CNN
+F 0 "#PWR211" H 20925 13925 50  0001 C CNN
 F 1 "+2V5" V 20925 14275 50  0000 C CNN
 F 2 "" H 20925 14075 50  0000 C CNN
@@
 I2C_SDA_PI
 $Comp
-L R R87
+L device:R R87
 U 1 1 591DED47
 P 20475 14375
@@
 $EndComp
 $Comp
-L R R86
+L device:R R86
 U 1 1 591DF05A
 P 20475 14275
@@
 $EndComp
 $Comp
-L R R84
+L device:R R84
 U 1 1 591DF1B0
 P 20475 14175
@@
 $EndComp
 $Comp
-L +3V3 #PWR0218
+L power:+3V3 #PWR226
 U 1 1 591E0007
 P 25425 14075
-F 0 "#PWR0218" H 25425 13925 50  0001 C CNN
+F 0 "#PWR226" H 25425 13925 50  0001 C CNN
 F 1 "+3V3" V 25425 14275 50  0000 C CNN
 F 2 "" H 25425 14075 50  0000 C CNN
@@
 $EndComp
 $Comp
-L +1V2 #PWR0219
+L power:+1V2 #PWR217
 U 1 1 591E000D
 P 22725 14125
-F 0 "#PWR0219" H 22725 13975 50  0001 C CNN
+F 0 "#PWR217" H 22725 13975 50  0001 C CNN
 F 1 "+1V2" V 22725 14325 50  0000 C CNN
 F 2 "" H 22725 14125 50  0000 C CNN
@@
 $EndComp
 $Comp
-L +2V5 #PWR0220
+L power:+2V5 #PWR224
 U 1 1 591E0014
 P 25325 14075
-F 0 "#PWR0220" H 25325 13925 50  0001 C CNN
+F 0 "#PWR224" H 25325 13925 50  0001 C CNN
 F 1 "+2V5" V 25325 14275 50  0000 C CNN
 F 2 "" H 25325 14075 50  0000 C CNN
@@
 $EndComp
 $Comp
-L R R96
+L device:R R96
 U 1 1 591E001A
 P 24875 14375
@@
 $EndComp
 $Comp
-L R R95
+L device:R R95
 U 1 1 591E0022
 P 24875 14275
@@
 $EndComp
 $Comp
-L R R94
+L device:R R94
 U 1 1 591E0028
 P 24875 14175
@@
 $EndComp
 $Comp
-L +3V3 #PWR0221
+L power:+3V3 #PWR215
 U 1 1 591E0245
 P 21125 17575
-F 0 "#PWR0221" H 21125 17425 50  0001 C CNN
+F 0 "#PWR215" H 21125 17425 50  0001 C CNN
 F 1 "+3V3" V 21125 17775 50  0000 C CNN
 F 2 "" H 21125 17575 50  0000 C CNN
@@
 $EndComp
 $Comp
-L +1V2 #PWR0222
+L power:+1V2 #PWR212
 U 1 1 591E024B
 P 20925 17575
-F 0 "#PWR0222" H 20925 17425 50  0001 C CNN
+F 0 "#PWR212" H 20925 17425 50  0001 C CNN
 F 1 "+1V2" V 20925 17775 50  0000 C CNN
 F 2 "" H 20925 17575 50  0000 C CNN
@@
 $EndComp
 $Comp
-L +2V5 #PWR0223
+L power:+2V5 #PWR214
 U 1 1 591E0252
 P 21025 17575
-F 0 "#PWR0223" H 21025 17425 50  0001 C CNN
+F 0 "#PWR214" H 21025 17425 50  0001 C CNN
 F 1 "+2V5" V 21025 17775 50  0000 C CNN
 F 2 "" H 21025 17575 50  0000 C CNN
@@
 $EndComp
 $Comp
-L R R90
+L device:R R90
 U 1 1 591E0258
 P 20575 17875
@@
 $EndComp
 $Comp
-L R R89
+L device:R R89
 U 1 1 591E0260
 P 20575 17775
@@
 $EndComp
 $Comp
-L R R88
+L device:R R88
 U 1 1 591E0266
 P 20575 17675
@@
 $EndComp
 $Comp
-L +3V3 #PWR0224
+L power:+3V3 #PWR227
 U 1 1 591E042D
 P 25475 17525
-F 0 "#PWR0224" H 25475 17375 50  0001 C CNN
+F 0 "#PWR227" H 25475 17375 50  0001 C CNN
 F 1 "+3V3" V 25475 17725 50  0000 C CNN
 F 2 "" H 25475 17525 50  0000 C CNN
@@
 $EndComp
 $Comp
-L +1V2 #PWR0225
+L power:+1V2 #PWR223
 U 1 1 591E0433
 P 25275 17525
-F 0 "#PWR0225" H 25275 17375 50  0001 C CNN
+F 0 "#PWR223" H 25275 17375 50  0001 C CNN
 F 1 "+1V2" V 25275 17725 50  0000 C CNN
 F 2 "" H 25275 17525 50  0000 C CNN
@@
 $EndComp
 $Comp
-L +2V5 #PWR0226
+L power:+2V5 #PWR225
 U 1 1 591E043A
 P 25375 17525
-F 0 "#PWR0226" H 25375 17375 50  0001 C CNN
+F 0 "#PWR225" H 25375 17375 50  0001 C CNN
 F 1 "+2V5" V 25375 17725 50  0000 C CNN
 F 2 "" H 25375 17525 50  0000 C CNN
@@
 $EndComp
 $Comp
-L R R141
+L device:R R141
 U 1 1 591E0440
 P 24925 17825
@@
 $EndComp
 $Comp
-L R R140
+L device:R R140
 U 1 1 591E0448
 P 24925 17725
@@
 $EndComp
 $Comp
-L R R97
+L device:R R97
 U 1 1 591E044E
 P 24925 17625
@@
 $EndComp
 $Comp
-L R R92
+L device:R R92
 U 1 1 591E1509
 P 23025 14375
@@
 $EndComp
 $Comp
-L +3V3 #PWR0227
+L power:+3V3 #PWR216
 U 1 1 591E1949
 P 22625 17525
-F 0 "#PWR0227" H 22625 17375 50  0001 C CNN
+F 0 "#PWR216" H 22625 17375 50  0001 C CNN
 F 1 "+3V3" V 22625 17725 50  0000 C CNN
 F 2 "" H 22625 17525 50  0000 C CNN
@@
 $EndComp
 $Comp
-L R R93
+L device:R R93
 U 1 1 591E19E0
 P 23025 17825
@@
 $EndComp
 $Comp
-L GND #PWR0228
+L power:GND #PWR219
 U 1 1 591E2746
 P 23275 16575
-F 0 "#PWR0228" H 23275 16325 50  0001 C CNN
+F 0 "#PWR219" H 23275 16325 50  0001 C CNN
 F 1 "GND" H 23275 16425 50  0000 C CNN
 F 2 "" H 23275 16575 50  0000 C CNN
@@
 $EndComp
 $Comp
-L +1V2 #PWR0229
+L power:+1V2 #PWR222
 U 1 1 591E36B7
 P 25225 14075
-F 0 "#PWR0229" H 25225 13925 50  0001 C CNN
+F 0 "#PWR222" H 25225 13925 50  0001 C CNN
 F 1 "+1V2" V 25225 14275 50  0000 C CNN
 F 2 "" H 25225 14075 50  0000 C CNN
@@
 NOTE: \nPower supply rail resistors should \nnot be fitted with ice40 eval board.
 $Comp
-L GND #PWR0230
+L power:GND #PWR208
 U 1 1 591E4259
 P 20225 16575
-F 0 "#PWR0230" H 20225 16325 50  0001 C CNN
+F 0 "#PWR208" H 20225 16325 50  0001 C CNN
 F 1 "GND" H 20225 16425 50  0000 C CNN
 F 2 "" H 20225 16575 50  0000 C CNN
@@
 $EndComp
 $Comp
-L GND #PWR0231
+L power:GND #PWR206
 U 1 1 591E429D
 P 18925 16575
-F 0 "#PWR0231" H 18925 16325 50  0001 C CNN
+F 0 "#PWR206" H 18925 16325 50  0001 C CNN
 F 1 "GND" H 18925 16425 50  0000 C CNN
 F 2 "" H 18925 16575 50  0000 C CNN
@@
 Connection ~ 18925 15075
 $Comp
-L GND #PWR0232
+L power:GND #PWR207
 U 1 1 591E4B93
 P 18975 20125
-F 0 "#PWR0232" H 18975 19875 50  0001 C CNN
+F 0 "#PWR207" H 18975 19875 50  0001 C CNN
 F 1 "GND" H 18975 19975 50  0000 C CNN
 F 2 "" H 18975 20125 50  0000 C CNN
@@
 $EndComp
 $Comp
-L GND #PWR0233
+L power:GND #PWR209
 U 1 1 591E4CA8
 P 20325 20125
-F 0 "#PWR0233" H 20325 19875 50  0001 C CNN
+F 0 "#PWR209" H 20325 19875 50  0001 C CNN
 F 1 "GND" H 20325 19975 50  0000 C CNN
 F 2 "" H 20325 20125 50  0000 C CNN
@@
 Connection ~ 20325 19775
 $Comp
-L GND #PWR0234
+L power:GND #PWR218
 U 1 1 591E5514
 P 23225 20125
-F 0 "#PWR0234" H 23225 19875 50  0001 C CNN
+F 0 "#PWR218" H 23225 19875 50  0001 C CNN
 F 1 "GND" H 23225 19975 50  0000 C CNN
 F 2 "" H 23225 20125 50  0000 C CNN
@@
 $EndComp
 $Comp
-L GND #PWR0235
+L power:GND #PWR221
 U 1 1 591E5558
 P 24625 20125
-F 0 "#PWR0235" H 24625 19875 50  0001 C CNN
+F 0 "#PWR221" H 24625 19875 50  0001 C CNN
 F 1 "GND" H 24625 19975 50  0000 C CNN
 F 2 "" H 24625 20125 50  0000 C CNN
@@
 USB_P
 $Comp
-L SO-DIMM J22
+L Devtank:SO-DIMM J22
 U 1 1 5AD2CF1C
 P 7750 575
