File: HILTOP_motherboard/CAN.sch (KiCad schematic (older format))
At the start: 22 parts

Commit message: Added RTC and Temp Sensor
Parts:
- FL?: symbol EMI_Filter_CommonMode -> EMI_Filter_CommonMode-RESCUE-HILTOP_Motherboard
Changed lines of the file:
@@
 EESchema Schematic File Version 2
+LIBS:HILTOP_Motherboard-rescue
 LIBS:Devtank
 LIBS:Zilog
@@
 $Descr A4 11693 8268
 encoding utf-8
-Sheet 9 9
+Sheet 9 10
 Title ""
 Date ""
@@
 Connection ~ 7300 5800
 $Comp
-L EMI_Filter_CommonMode FL?
+L EMI_Filter_CommonMode-RESCUE-HILTOP_Motherboard FL?
 U 1 1 5A730278
 P 8500 2000
+AR Path="/5A730278" Ref="FL?"  Part="1"
+AR Path="/5A7BC033/5A730278" Ref="FL?"  Part="1"
 F 0 "FL?" H 8500 2175 50  0000 C CNN
 F 1 "PE-1812ACC510STS" H 8500 1825 50  0000 C CNN

Commit message: Added more detail to motherboard schemas
Parts:
- added C? (x4): 47pF, Capacitors_SMD:C_0603, symbol C
- added C?: 100nF, Capacitor_SMD:C_0603_1608Metric, symbol C
- added C? (x2): 100nF, Capacitors_SMD:C_0603, symbol C
- added D?: NUP2105L, TO_SOT_Packages_SMD:SOT-23, symbol NUP2105L
- added FL?: PE-1812ACC510STS, symbol EMI_Filter_CommonMode-RESCUE-HILTOP_Motherboard
- added JP?: Jumper_NO_Small, Pin_Headers:Pin_Header_Straight_1x02_Pitch2.54mm, symbol Jumper_NO_Small
- added R?: 120R, Resistors_SMD:R_0603, symbol R
- added U?: MCP2561FD, MODULE, symbol MCP2561FD
- added U?: ADuM1201, Package_SOIC:SOIC-8_3.9x4.9mm_P1.27mm, symbol ADuM1201
- added U?: MCP2517FD, symbol MCP2517FD
Connections:
- net labels added: CAN_CH2_H, CAN_CH2_L
- wire segments 82 -> 184
Other:
- moved on the sheet: C?

Commit message: Finished CAN nd RS485 interface circuits
Parts:
- removed C? (x2): 4.7uF, Capacitors_SMD:C_0805, symbol C
- removed C? (x2): 2.2uF, Capacitors_SMD:C_0805, symbol C
- removed JP? (x2): Jumper_NO_Small, Pin_Headers:Pin_Header_Straight_1x02_Pitch2.54mm, symbol Jumper_NO_Small
- removed L? (x2): 10uH, KiCAD_PCB_Lib:Inductor_MuRata_82103C, symbol L
- removed R?: 120R, Resistors_SMD:R_0603, symbol R
- removed U? (x2): CME0303S3C, KiCAD_PCB_Lib:CME_XXXX_S3C_PSU_MODULE, symbol CME0303S3C
- added C? (x4): 9pF, Capacitors_SMD:C_0603, symbol C
- added C? (x2): 100nF, Capacitor_SMD:C_0603_1608Metric, symbol C
- added C? (x2): 4.7uF, Capacitors_SMD:C_0805, symbol C
- added C? (x2): 2.2uF, Capacitors_SMD:C_0805, symbol C
- added C? (x2): 470pF, Capacitor_SMD:C_0603_1608Metric, symbol C
- added L? (x2): 15uH, KiCAD_PCB_Lib:Inductor_MuRata_82103C, symbol L
- added R?: DNF, Resistors_SMD:R_0603, symbol R
- added U? (x2): AM1S-0505SZ, KiCAD_PCB_Lib:CME_XXXX_S3C_PSU_MODULE, symbol CME0303S3C
- added Y? (x2): 40MHz Crystal, Crystals:Crystal_SMD_SeikoEpson_FA238V-4pin_3.2x2.5mm, symbol Crystal_GND24
- R?: value 120R -> DNF; Devtank 101-018 -> (none)
Connections:
- net labels added: +5V, CAN_CH1_INT, CAN_CH1_INT0, CAN_CH1_INT1, CAN_CH2_INT, CAN_CH2_INT0, CAN_CH2_INT1
- wire segments 184 -> 248
Other:
- note removed: "OPTIONAL: \nLine Termination\n"
- moved on the sheet: C?, D?, FL?, R?, U?

Commit message: Furthe progress on Schematics, assigned all main footprints using latest libraries, removed unwanted tracking and parts from original PCB layout
Parts:
- C100, C102, C153, C84: renamed from C?; footprint Capacitors_SMD:C_0805 -> Capacitor_SMD:C_0805_2012Metric
- C103, C104, C105, C108, C155, C156, C157, C158, C159, C160, C161, C162, C163, C164, C165, C166: renamed from C?; footprint Capacitors_SMD:C_0603 -> Capacitor_SMD:C_0603_1608Metric
- D36, D37: renamed from D?; footprint TO_SOT_Packages_SMD:SOT-23 -> Package_TO_SOT_SMD:SOT-23
- FL1, FL2: renamed from FL?; footprint (none) -> Devtank_PCB_Lib:Inductor_PE-1812ACCXXXSTS
- L11, L7: renamed from L?; footprint KiCAD_PCB_Lib:Inductor_MuRata_82103C -> Devtank_PCB_Lib:Inductor_MuRata_82103C
- R175, R176: renamed from R?; footprint Resistors_SMD:R_0603 -> Resistor_SMD:R_0603_1608Metric
- U29, U32: renamed from U?; footprint KiCAD_PCB_Lib:CME_XXXX_S3C_PSU_MODULE -> Devtank_PCB_Lib:CME_XXXX_S3C_PSU_MODULE
- U30, U31: renamed from U?; footprint (none) -> Package_SOIC:SOIC-14_3.9x8.7mm_P1.27mm
- U35, U36: renamed from U?; footprint MODULE -> Package_SOIC:SOIC-8_3.9x4.9mm_P1.27mm
- Y5, Y6: renamed from Y?; footprint Crystals:Crystal_SMD_SeikoEpson_FA238V-4pin_3.2x2.5mm -> Crystal:Crystal_SMD_SeikoEpson_FA238V-4Pin_3.2x2.5mm
- gave numbers to parts that had none: 8

Commit message: Schematics complete - 1st draft
Parts:
- added R199, R200: 10K, Resistor_SMD:R_0603_1608Metric, symbol device:R
- C100, C101, C102, C103, C104, C105, C108, C122, C129, C153, C154, C155, C156, C157, C158, C159, C160, C161, C162, C163, C164, C165, C166, C84, C98, C99: symbol C -> device:C
- D36, D37: symbol NUP2105L -> ESD_Protection:NUP2105L
- FL1, FL2: symbol EMI_Filter_CommonMode-RESCUE-HILTOP_Motherboard -> HILTOP_Motherboard-rescue:EMI_Filter_CommonMode-RESCUE-HILTOP_Motherboard
- L11, L7: symbol L -> device:L
- R175, R176: symbol R -> device:R
- U29, U32: symbol CME0303S3C -> Devtank:CME0303S3C
- U30, U31: symbol MCP2517FD -> Devtank:MCP2517FD
- U33, U34: symbol ADuM1201 -> Devtank:ADuM1201
- U35, U36: symbol MCP2561FD -> Devtank:MCP2561FD
- Y5, Y6: symbol Crystal_GND24 -> device:Crystal_GND24
Connections:
- net +3V3: now also R199.1, R200.1
- net CAN_CH1_CS: now also R199.2
- net CAN_CH2_CS: now also R200.2

Commit message: BOM nearly complete!
Parts:
- D36, D37: Devtank (none) -> 136-002
- FL1, FL2: Devtank (none) -> 114-001
- U30, U31: Devtank (none) -> 118-006
- U33, U34: Devtank (none) -> 117-002
- U35, U36: Devtank (none) -> 118-005
Connections:
- no-connect marks 0 -> 7
Changed lines of the file:
@@
 F 2 "Package_SOIC:SOIC-8_3.9x4.9mm_P1.27mm" H 9250 2075 50  0001 C CNN
 F 3 "DOCUMENTATION" H 9400 1975 50  0001 C CNN
+F 4 "118-005" H 9550 2575 50  0001 C CNN "Devtank"
 	1    9550 2575
 	1    0    0    -1
@@
 F 2 "Package_SOIC:SOIC-8_3.9x4.9mm_P1.27mm" H 7550 2825 50  0001 L CIN
 F 3 "" H 7500 3375 50  0000 C CNN
+F 4 "117-002" H 7500 2875 50  0001 C CNN "Devtank"
 	1    7500 2875
 	1    0    0    -1
@@
 F 2 "Devtank_PCB_Lib:Inductor_PE-1812ACCXXXSTS" V 11200 2615 50  0001 C CNN
 F 3 "" V 11200 2615 50  0000 C CNN
+F 4 "114-001" H 11200 2575 50  0001 C CNN "Devtank"
 	1    11200 2575
 	1    0    0    -1
@@
 F 2 "Package_TO_SOT_SMD:SOT-23" H 12475 2925 50  0001 L CNN
 F 3 "" H 12375 3100 50  0001 C CNN
+F 4 "136-002" H 12250 2975 50  0001 C CNN "Devtank"
 	1    12250 2975
 	1    0    0    -1
@@
 F 2 "Package_SOIC:SOIC-14_3.9x8.7mm_P1.27mm" H 6025 7175 60  0001 C CNN
 F 3 "" H 6025 7175 60  0000 C CNN
+F 4 "118-006" H 4975 5675 50  0001 C CNN "Devtank"
 	1    4975 5675
 	-1   0    0    -1
@@
 F 2 "Package_SOIC:SOIC-8_3.9x4.9mm_P1.27mm" H 9225 4875 50  0001 C CNN
 F 3 "DOCUMENTATION" H 9375 4775 50  0001 C CNN
+F 4 "118-005" H 9525 5375 50  0001 C CNN "Devtank"
 	1    9525 5375
 	1    0    0    -1
@@
 F 2 "Package_SOIC:SOIC-8_3.9x4.9mm_P1.27mm" H 7525 5625 50  0001 L CIN
 F 3 "" H 7475 6175 50  0000 C CNN
+F 4 "117-002" H 7475 5675 50  0001 C CNN "Devtank"
 	1    7475 5675
 	1    0    0    -1
@@
 F 2 "Devtank_PCB_Lib:Inductor_PE-1812ACCXXXSTS" V 11175 5415 50  0001 C CNN
 F 3 "" V 11175 5415 50  0000 C CNN
+F 4 "114-001" H 11175 5375 50  0001 C CNN "Devtank"
 	1    11175 5375
 	1    0    0    -1
@@
 F 2 "Package_TO_SOT_SMD:SOT-23" H 12450 5725 50  0001 L CNN
 F 3 "" H 12350 5900 50  0001 C CNN
+F 4 "136-002" H 12225 5775 50  0001 C CNN "Devtank"
 	1    12225 5775
 	1    0    0    -1
@@
 F 2 "Package_SOIC:SOIC-14_3.9x8.7mm_P1.27mm" H 6000 9975 60  0001 C CNN
 F 3 "" H 6000 9975 60  0000 C CNN
+F 4 "118-006" H 4950 8475 50  0001 C CNN "Devtank"
 	1    4950 8475
 	-1   0    0    -1
@@
 Wire Wire Line
 	2025 5325 3550 5325
+NoConn ~ 7425 5800
+NoConn ~ 5275 2675
+NoConn ~ 5250 5475
+NoConn ~ 10300 2425
+NoConn ~ 10300 2725
+NoConn ~ 10275 5225
+NoConn ~ 10275 5525
 $EndSCHEMATC
