File: HILTOP_motherboard/CAN.sch (KiCad schematic (older format))
At the start: 46 parts, among them U29 AM1S-0505SZ, U30 MCP2517FD, U31 MCP2517FD, U32 AM1S-0505SZ, U33 ADuM1201, U34 ADuM1201, U35 MCP2561FD, U36 MCP2561FD, Y5 40MHz Crystal, Y6 40MHz Crystal

Commit message: nearly finished placing all parts!
Parts:
- FL1, FL2: symbol HILTOP_Motherboard-rescue:EMI_Filter_CommonMode-RESCUE-HILTOP_Motherboard -> Devtank:CAN_Filter_Choke
- L11, L7: value 15uH -> 10uH; Devtank 112-007 -> 112-004
- U29, U32: value AM1S-0505SZ -> CME0505S3C; Devtank 131-002 -> 131-003
Other:
- moved on the sheet: U29, U32

Commit message: DRC checks complete, all errors and warnings cleared. BOM created and parts rationalised.
Parts:
- C158, C159, C161, C162, C163, C164, C165, C166: Devtank 105-002 -> 106-011
Connections:
- wire segments 266 -> 274
Other:
- moved on the sheet: U32

Commit message: finished new tracking for RS485 signals and general house keeping
Connections:
- wire segments 274 -> 282
- no-connect marks 7 -> 5
Changed lines of the file:
@@
 Sheet 7 12
 Title "HILTOP Motherboard"
-Date "2019-01-10"
-Rev "Issue 1"
+Date "2019-07-03"
+Rev "Rev B"
 Comp "Devtank Ltd"
 Comment1 ""
@@
 	10800 3225 10550 3225
 Wire Wire Line
-	10550 3125 10550 3225
+	10550 3125 10550 3175
 Connection ~ 10550 3225
 $Comp
@@
 	10775 6025 10525 6025
 Wire Wire Line
-	10525 5925 10525 6025
+	10525 5925 10525 5950
 Connection ~ 10525 6025
 Wire Wire Line
@@
 NoConn ~ 5275 2675
 NoConn ~ 5250 5475
-NoConn ~ 10300 2425
 NoConn ~ 10300 2725
-NoConn ~ 10275 5225
 NoConn ~ 10275 5525
 Wire Wire Line
@@
 Wire Wire Line
 	4550 9325 4550 9400
+Wire Wire Line
+	10275 5225 10375 5225
+Wire Wire Line
+	10375 5225 10375 5950
+Wire Wire Line
+	10375 5950 10525 5950
+Connection ~ 10525 5950
+Wire Wire Line
+	10525 5950 10525 6025
+Wire Wire Line
+	10300 2425 10425 2425
+Wire Wire Line
+	10425 2425 10425 3175
+Wire Wire Line
+	10425 3175 10550 3175
+Connection ~ 10550 3175
+Wire Wire Line
+	10550 3175 10550 3225
 $EndSCHEMATC

Commit message: Rev C - pre-release
Parts:
- C100, C101, C102, C103, C104, C105, C108, C122, C129, C153, C154, C155, C156, C157, C158, C159, C160, C161, C162, C163, C164, C165, C166, C84, C98, C99: symbol device:C -> HILTOP_Motherboard-rescue:C-device
- D36, D37: symbol ESD_Protection:NUP2105L -> HILTOP_Motherboard-rescue:NUP2105L-ESD_Protection
- L11, L7: symbol device:L -> HILTOP_Motherboard-rescue:L-device
- R175, R176, R199, R200: symbol device:R -> HILTOP_Motherboard-rescue:R-device
- Y5, Y6: symbol device:Crystal_GND24 -> HILTOP_Motherboard-rescue:Crystal_GND24-device
Changed lines of the file:
@@
 $Descr A3 16535 11693
 encoding utf-8
-Sheet 7 12
+Sheet 6 12
 Title "HILTOP Motherboard"
 Date "2019-07-03"
@@
 	2875 2025 2875 2125
 $Comp
-L device:C C162
+L HILTOP_Motherboard-rescue:C-device C162
 U 1 1 5A71D94F
 P 10800 2975
@@
 $EndComp
 $Comp
-L device:C C155
+L HILTOP_Motherboard-rescue:C-device C155
 U 1 1 5A71D957
 P 9500 8025
@@
 $EndComp
 $Comp
-L device:C C98
+L HILTOP_Motherboard-rescue:C-device C98
 U 1 1 5A71D95F
 P 3125 2025
@@
 	8250 2775 8000 2775
 $Comp
-L device:C C156
+L HILTOP_Motherboard-rescue:C-device C156
 U 1 1 5A72DCA3
 P 9850 8025
@@
 CAN_CH1_L
 $Comp
-L device:R R176
+L HILTOP_Motherboard-rescue:R-device R176
 U 1 1 5A7330B3
 P 12850 2475
@@
 	12850 2250 12850 2325
 $Comp
-L ESD_Protection:NUP2105L D37
+L HILTOP_Motherboard-rescue:NUP2105L-ESD_Protection D37
 U 1 1 5A733232
 P 12250 2975
@@
 $EndComp
 $Comp
-L device:C C159
+L HILTOP_Motherboard-rescue:C-device C159
 U 1 1 5A733494
 P 10550 2975
@@
 $EndComp
 $Comp
-L device:C C164
+L HILTOP_Motherboard-rescue:C-device C164
 U 1 1 5A7336A0
 P 11600 2975
@@
 $EndComp
 $Comp
-L device:C C166
+L HILTOP_Motherboard-rescue:C-device C166
 U 1 1 5A73397E
 P 11850 2975
@@
 	3950 4600 3950 4700
 $Comp
-L device:C C161
+L HILTOP_Motherboard-rescue:C-device C161
 U 1 1 5AC9B9B6
 P 10775 5775
@@
 $EndComp
 $Comp
-L device:C C99
+L HILTOP_Motherboard-rescue:C-device C99
 U 1 1 5AC9B9BD
 P 3700 4600
@@
 Connection ~ 12825 5475
 $Comp
-L ESD_Protection:NUP2105L D36
+L HILTOP_Motherboard-rescue:NUP2105L-ESD_Protection D36
 U 1 1 5AC9BA13
 P 12225 5775
@@
 $EndComp
 $Comp
-L device:C C158
+L HILTOP_Motherboard-rescue:C-device C158
 U 1 1 5AC9BA1A
 P 10525 5775
@@
 $EndComp
 $Comp
-L device:C C163
+L HILTOP_Motherboard-rescue:C-device C163
 U 1 1 5AC9BA21
 P 11575 5775
@@
 $EndComp
 $Comp
-L device:C C165
+L HILTOP_Motherboard-rescue:C-device C165
 U 1 1 5AC9BA28
 P 11825 5775
@@
 	9850 8175 9850 8275
 $Comp
-L device:C C157
+L HILTOP_Motherboard-rescue:C-device C157
 U 1 1 5AC9D355
 P 10325 8025
@@
 $EndComp
 $Comp
-L device:C C160
+L HILTOP_Motherboard-rescue:C-device C160
 U 1 1 5AC9D35C
 P 10675 8025
@@
 Connection ~ 2875 2975
 $Comp
-L device:R R175
+L HILTOP_Motherboard-rescue:R-device R175
 U 1 1 5AE7E2F5
 P 12825 5250
@@
 	12825 5400 12825 5475
 $Comp
-L device:Crystal_GND24 Y5
+L HILTOP_Motherboard-rescue:Crystal_GND24-device Y5
 U 1 1 5AFAB522
 P 5950 6075
@@
 $EndComp
 $Comp
-L device:C C103
+L HILTOP_Motherboard-rescue:C-device C103
 U 1 1 5AFAB52A
 P 5600 6325
@@
 $EndComp
 $Comp
-L device:C C105
+L HILTOP_Motherboard-rescue:C-device C105
 U 1 1 5AFAB538
 P 6300 6325
@@
 	5275 2825 5675 2825
 $Comp
-L device:Crystal_GND24 Y6
+L HILTOP_Motherboard-rescue:Crystal_GND24-device Y6
 U 1 1 5AFB1B89
 P 5975 3275
@@
 $EndComp
 $Comp
-L device:C C104
+L HILTOP_Motherboard-rescue:C-device C104
 U 1 1 5AFB1B90
 P 5625 3525
@@
 $EndComp
 $Comp
-L device:C C108
+L HILTOP_Motherboard-rescue:C-device C108
 U 1 1 5AFB1B9D
 P 6325 3525
@@
 	6150 2025 6150 2125
 $Comp
-L device:C C129
+L HILTOP_Motherboard-rescue:C-device C129
 U 1 1 5AFB6124
 P 6400 2025
@@
 	6100 4825 6100 4925
 $Comp
-L device:C C122
+L HILTOP_Motherboard-rescue:C-device C122
 U 1 1 5AFB68CC
 P 6350 4825
@@
 Connection ~ 6675 4825
 $Comp
-L device:C C100
+L HILTOP_Motherboard-rescue:C-device C100
 U 1 1 5AFC0572
 P 4225 9000
@@
 $EndComp
 $Comp
-L device:L L7
+L HILTOP_Motherboard-rescue:L-device L7
 U 1 1 5AFC057A
 P 3825 8750
@@
 $EndComp
 $Comp
-L device:C C84
+L HILTOP_Motherboard-rescue:C-device C84
 U 1 1 5AFC0588
 P 1900 8975
@@
 $EndComp
 $Comp
-L device:C C101
+L HILTOP_Motherboard-rescue:C-device C101
 U 1 1 5AFC05BE
 P 4550 9000
@@
 Connection ~ 4550 8750
 $Comp
-L device:C C153
+L HILTOP_Motherboard-rescue:C-device C153
 U 1 1 5AFC05CD
 P 8150 9000
@@
 $EndComp
 $Comp
-L device:L L11
+L HILTOP_Motherboard-rescue:L-device L11
 U 1 1 5AFC05D5
 P 7700 8750
@@
 $EndComp
 $Comp
-L device:C C102
+L HILTOP_Motherboard-rescue:C-device C102
 U 1 1 5AFC05DD
 P 5725 8975
@@
 $EndComp
 $Comp
-L device:C C154
+L HILTOP_Motherboard-rescue:C-device C154
 U 1 1 5AFC0607
 P 8475 9000
@@
 	8475 8750 8475 8850
 $Comp
-L device:R R?
+L HILTOP_Motherboard-rescue:R-device R?
 U 1 1 5C47457C
 P 2000 1975
@@
 	2000 2525 3575 2525
 $Comp
-L device:R R?
+L HILTOP_Motherboard-rescue:R-device R?
 U 1 1 5C4B087B
 P 2025 4775

Commit message: changed silkscreen to revD and updated sheet information
Parts:
- FL1, FL2: symbol Devtank:CAN_Filter_Choke -> HILTOP_Motherboard-rescue:CAN_Filter_Choke-Devtank
- U29, U32: symbol Devtank:CME0303S3C -> HILTOP_Motherboard-rescue:CME0303S3C-Devtank
- U30, U31: symbol Devtank:MCP2517FD -> HILTOP_Motherboard-rescue:MCP2517FD-Devtank
- U33, U34: symbol Devtank:ADuM1201 -> HILTOP_Motherboard-rescue:ADuM1201-Devtank
- U35, U36: symbol Devtank:MCP2561FD -> HILTOP_Motherboard-rescue:MCP2561FD-Devtank
Changed lines of the file:
@@
 Sheet 6 12
 Title "HILTOP Motherboard"
-Date "2020-04-28"
-Rev "Rev C"
+Date "2021-02-17"
+Rev "Rev D"
 Comp "Devtank Ltd"
-Comment1 ""
+Comment1 "Part No: 304-001"
 Comment2 ""
 Comment3 ""
@@
 $EndComp
 $Comp
-L Devtank:MCP2561FD U36
+L HILTOP_Motherboard-rescue:MCP2561FD-Devtank U36
 U 1 1 5A724F50
 P 9550 2575
@@
 Isolation Options:\n(Pin Compatible)\nADuM1201\nISO7221
 $Comp
-L Devtank:ADuM1201 U34
+L HILTOP_Motherboard-rescue:ADuM1201-Devtank U34
 U 1 1 5A72CF9F
 P 7500 2875
@@
 $EndComp
 $Comp
-L Devtank:+5V_ISO1 #PWR0376
+L HILTOP_Motherboard-rescue:+5V_ISO1-Devtank #PWR0376
 U 1 1 5A72D1D4
 P 8500 1925
@@
 	6700 2775 7000 2775
 $Comp
-L Devtank:GND_ISO1 #PWR0374
+L HILTOP_Motherboard-rescue:GND_ISO1-Devtank #PWR0374
 U 1 1 5A72D8C5
 P 8250 3475
@@
 Connection ~ 8250 2975
 $Comp
-L Devtank:+5V_ISO1 #PWR0377
+L HILTOP_Motherboard-rescue:+5V_ISO1-Devtank #PWR0377
 U 1 1 5A72F267
 P 9500 7725
@@
 Connection ~ 9500 7775
 $Comp
-L Devtank:GND_ISO1 #PWR0378
+L HILTOP_Motherboard-rescue:GND_ISO1-Devtank #PWR0378
 U 1 1 5A72F44A
 P 9500 8375
@@
 Connection ~ 9500 8275
 $Comp
-L Devtank:CAN_Filter_Choke FL?
+L HILTOP_Motherboard-rescue:CAN_Filter_Choke-Devtank FL?
 U 1 1 5A730278
 P 11200 2575
@@
 Connection ~ 11850 2475
 $Comp
-L Devtank:GND_ISO1 #PWR0382
+L HILTOP_Motherboard-rescue:GND_ISO1-Devtank #PWR0382
 U 1 1 5A73402C
 P 10550 3275
@@
 $EndComp
 $Comp
-L Devtank:GND_ISO1 #PWR0384
+L HILTOP_Motherboard-rescue:GND_ISO1-Devtank #PWR0384
 U 1 1 5A734109
 P 11600 3275
@@
 Connection ~ 10550 3225
 $Comp
-L Devtank:GND_ISO1 #PWR0386
+L HILTOP_Motherboard-rescue:GND_ISO1-Devtank #PWR0386
 U 1 1 5A734385
 P 12250 3275
@@
 Connection ~ 12350 2675
 $Comp
-L Devtank:MCP2517FD U31
+L HILTOP_Motherboard-rescue:MCP2517FD-Devtank U31
 U 1 1 5A735F1E
 P 4975 5675
@@
 $EndComp
 $Comp
-L Devtank:MCP2561FD U35
+L HILTOP_Motherboard-rescue:MCP2561FD-Devtank U35
 U 1 1 5AC9B9C3
 P 9525 5375
@@
 Isolation Options:\n(Pin Compatible)\nADuM1201\nISO7221
 $Comp
-L Devtank:ADuM1201 U33
+L HILTOP_Motherboard-rescue:ADuM1201-Devtank U33
 U 1 1 5AC9B9CA
 P 7475 5675
@@
 Connection ~ 8225 5775
 $Comp
-L Devtank:CAN_Filter_Choke FL1
+L HILTOP_Motherboard-rescue:CAN_Filter_Choke-Devtank FL1
 U 1 1 5AC9B9EF
 P 11175 5375
@@
 Connection ~ 12325 5475
 $Comp
-L Devtank:MCP2517FD U30
+L HILTOP_Motherboard-rescue:MCP2517FD-Devtank U30
 U 1 1 5AC9BA59
 P 4950 8475
@@
 	10675 8175 10675 8275
 $Comp
-L Devtank:+5V_ISO2 #PWR0379
+L HILTOP_Motherboard-rescue:+5V_ISO2-Devtank #PWR0379
 U 1 1 5AC9D4BC
 P 10325 7725
@@
 $EndComp
 $Comp
-L Devtank:GND_ISO2 #PWR0380
+L HILTOP_Motherboard-rescue:GND_ISO2-Devtank #PWR0380
 U 1 1 5AC9D533
 P 10325 8375
@@
 $EndComp
 $Comp
-L Devtank:+5V_ISO2 #PWR0375
+L HILTOP_Motherboard-rescue:+5V_ISO2-Devtank #PWR0375
 U 1 1 5ACA9D31
 P 8475 4725
@@
 $EndComp
 $Comp
-L Devtank:GND_ISO2 #PWR0373
+L HILTOP_Motherboard-rescue:GND_ISO2-Devtank #PWR0373
 U 1 1 5ACAA030
 P 8225 6275
@@
 $EndComp
 $Comp
-L Devtank:GND_ISO2 #PWR0381
+L HILTOP_Motherboard-rescue:GND_ISO2-Devtank #PWR0381
 U 1 1 5ACAA233
 P 10525 6075
@@
 $EndComp
 $Comp
-L Devtank:GND_ISO2 #PWR0383
+L HILTOP_Motherboard-rescue:GND_ISO2-Devtank #PWR0383
 U 1 1 5ACAA33A
 P 11575 6075
@@
 $EndComp
 $Comp
-L Devtank:GND_ISO2 #PWR0385
+L HILTOP_Motherboard-rescue:GND_ISO2-Devtank #PWR0385
 U 1 1 5ACAA4F5
 P 12225 6075
@@
 Connection ~ 4225 9225
 $Comp
-L Devtank:CME0303S3C U29
+L HILTOP_Motherboard-rescue:CME0303S3C-Devtank U29
 U 1 1 5AFC05A8
 P 2875 9075
@@
 Connection ~ 8150 9225
 $Comp
-L Devtank:CME0303S3C U32
+L HILTOP_Motherboard-rescue:CME0303S3C-Devtank U32
 U 1 1 5AFC05F7
 P 6700 9075
@@
 Connection ~ 8475 8750
 $Comp
-L Devtank:+5V_ISO1 #PWR0355
+L HILTOP_Motherboard-rescue:+5V_ISO1-Devtank #PWR0355
 U 1 1 5AFC07F3
 P 4550 8575
@@
 $EndComp
 $Comp
-L Devtank:GND_ISO1 #PWR0356
+L HILTOP_Motherboard-rescue:GND_ISO1-Devtank #PWR0356
 U 1 1 5AFC0A3A
 P 4550 9400
@@
 $EndComp
 $Comp
-L Devtank:+5V_ISO2 #PWR0371
+L HILTOP_Motherboard-rescue:+5V_ISO2-Devtank #PWR0371
 U 1 1 5AFC0CE9
 P 8475 8575
@@
 $EndComp
 $Comp
-L Devtank:GND_ISO2 #PWR0372
+L HILTOP_Motherboard-rescue:GND_ISO2-Devtank #PWR0372
 U 1 1 5AFC1068
 P 8475 9400
