File: HILTOP_motherboard/Processor.sch (KiCad schematic (older format))
At the start: 22 parts, among them J13 DDR2_SODIMM_COMPUTE_MODULE_3, U23 TPD12S016

Commit message: Added new USB2.0 device
Parts:
- added C?: 4.7uF, Capacitors_SMD:C_0805, symbol C
- added R?: 0R, Resistors_SMD:R_0603, symbol R
Connections:
- net labels added: +CM_5V
- wire segments 235 -> 242
Changed lines of the file:
@@
 LIBS:regul
 LIBS:references
-LIBS:pspice
 LIBS:Power_Management
 LIBS:powerint
@@
 LIBS:Diode
 LIBS:digital-audio
-LIBS:device
 LIBS:Decawave
 LIBS:dc-dc
@@
 LIBS:adc-dac
 LIBS:ac-dc
+LIBS:device
 LIBS:HILTOP_Motherboard-cache
 EELAYER 25 0
@@
 $Descr A3 11693 16535 portrait
 encoding utf-8
-Sheet 6 8
+Sheet 6 9
 Title "HILTOP Motherboard"
 Date "26th January 2018"
@@
 	10050 13850 10500 13850
 Wire Wire Line
-	7750 12100 7750 12600
-Wire Wire Line
 	7000 12200 7750 12200
 Wire Wire Line
-	7000 12300 7750 12300
+	7750 12300 7000 12300
 Connection ~ 7750 12200
 Wire Wire Line
-	7000 12500 7750 12500
+	7000 12500 8050 12500
 Connection ~ 7750 12300
 Wire Wire Line
-	7750 12600 7000 12600
-Connection ~ 7750 12500
+	8050 12600 7000 12600
 Wire Wire Line
 	7600 11850 7600 12100
@@
 Connection ~ 7400 11800
 Wire Wire Line
-	4100 12100 4100 12600
-Wire Wire Line
-	4100 12600 4850 12600
-Wire Wire Line
-	4850 12500 4100 12500
-Connection ~ 4100 12500
-Wire Wire Line
-	4850 12300 4100 12300
-Connection ~ 4100 12300
+	3800 12600 4850 12600
+Wire Wire Line
+	3800 12500 4850 12500
+Wire Wire Line
+	4100 12300 4850 12300
 Wire Wire Line
 	4850 12200 4100 12200
-Connection ~ 4100 12200
 Wire Wire Line
 	4300 11900 4300 12100
@@
 Text HLabel 3700 4300 0    60   Output ~ 0
 PI_SPIO_MOSI
+$Comp
+L GND #PWR?
+U 1 1 5A76E65E
+P 10500 12400
+F 0 "#PWR?" H 10500 12150 50  0001 C CNN
+F 1 "GND" H 10500 12250 50  0000 C CNN
+F 2 "" H 10500 12400 50  0000 C CNN
+F 3 "" H 10500 12400 50  0000 C CNN
+	1    10500 12400
+	1    0    0    -1
+$EndComp
+$Comp
+L R R?
+U 1 1 5A76E671
+P 10500 11600
+F 0 "R?" H 10650 11650 50  0000 C CNN
+F 1 "0R" H 10600 11550 50  0000 C CNN
+F 2 "Resistors_SMD:R_0603" V 10430 11600 50  0001 C CNN
+F 3 "" H 10500 11600 50  0000 C CNN
+F 4 "101-005" H 10500 11600 60  0001 C CNN "Devtank"
+	1    10500 11600
+	1    0    0    -1
+$EndComp
+$Comp
+L C C?
+U 1 1 5A76E678
+P 10500 12200
+F 0 "C?" H 10600 12250 50  0000 L CNN
+F 1 "4.7uF" H 10600 12150 50  0000 L CNN
+F 2 "Capacitors_SMD:C_0805" H 10538 12050 50  0001 C CNN
+F 3 "" H 10500 12200 50  0000 C CNN
+F 4 "105-007" H 10500 12200 60  0001 C CNN "Devtank"
+	1    10500 12200
+	1    0    0    -1
+$EndComp
+Wire Wire Line
+	10500 11750 10500 12050
+Connection ~ 10500 11950
+Wire Wire Line
+	10500 12400 10500 12350
+Wire Wire Line
+	10500 11250 10500 11450
+Wire Wire Line
+	10050 11950 10500 11950
+Wire Wire Line
+	10050 11850 10050 11950
+$Comp
+L +CM_5V #PWR?
+U 1 1 5A76E760
+P 10050 11850
+F 0 "#PWR?" H 10050 11700 50  0001 C CNN
+F 1 "+CM_5V" H 10050 11990 50  0000 C CNN
+F 2 "" H 10050 11850 50  0000 C CNN
+F 3 "" H 10050 11850 50  0000 C CNN
+	1    10050 11850
+	1    0    0    -1
+$EndComp
+$Comp
+L +5V #PWR?
+U 1 1 5A76EAEC
+P 10500 11250
+F 0 "#PWR?" H 10500 11100 50  0001 C CNN
+F 1 "+5V" H 10500 11390 50  0000 C CNN
+F 2 "" H 10500 11250 50  0001 C CNN
+F 3 "" H 10500 11250 50  0001 C CNN
+	1    10500 11250
+	1    0    0    -1
+$EndComp
+$Comp
+L +CM_5V #PWR?
+U 1 1 5A76EDE6
+P 8050 12450
+F 0 "#PWR?" H 8050 12300 50  0001 C CNN
+F 1 "+CM_5V" H 8050 12590 50  0000 C CNN
+F 2 "" H 8050 12450 50  0000 C CNN
+F 3 "" H 8050 12450 50  0000 C CNN
+	1    8050 12450
+	1    0    0    -1
+$EndComp
+Wire Wire Line
+	7750 12100 7750 12300
+Wire Wire Line
+	8050 12450 8050 12600
+Connection ~ 8050 12500
+Wire Wire Line
+	4100 12100 4100 12300
+Connection ~ 4100 12200
+$Comp
+L +CM_5V #PWR?
+U 1 1 5A76FB57
+P 3800 12450
+F 0 "#PWR?" H 3800 12300 50  0001 C CNN
+F 1 "+CM_5V" H 3800 12590 50  0000 C CNN
+F 2 "" H 3800 12450 50  0000 C CNN
+F 3 "" H 3800 12450 50  0000 C CNN
+	1    3800 12450
+	1    0    0    -1
+$EndComp
+Wire Wire Line
+	3800 12450 3800 12600
+Connection ~ 3800 12500
 $EndSCHEMATC

Commit message: Added RTC and Temp Sensor
Parts:
- added C? (x2): 100nF, Resistor_SMD:R_0603_1608Metric, symbol C
- added C? (x2): 12pF, Resistor_SMD:R_0603_1608Metric, symbol C
- added R? (x6): DNF, Resistor_SMD:R_0402_1005Metric, symbol R
- added R?: 10K, Resistor_SMD:R_0603_1608Metric, symbol R
- added R?: 0R, Resistor_SMD:R_0603_1608Metric, symbol R
- added U?: AT30TS75, Package_DFN_QFN:DFN-8-1EP_3x2mm_P0.5mm, symbol AT30TS75
- added U?: BQ32000, Package_SOIC:SOIC-8_3.9x4.9mm_P1.27mm, symbol BQ32000
- added Y?: Crystal, symbol Crystal
- added Y?: 0.22F, Devtank_PCB_Lib:Battery_SD_V_SuperCap, symbol SuperCap
Connections:
- net labels added: SCL1, SDA1
- wire segments 242 -> 293

Commit message: Updated pinouts for Backplane and Compute Module
Connections:
- net labels added: CAM1_CK_N, CAM1_CK_P, CAM1_D0_N, CAM1_D0_P, CAM1_D1_N, CAM1_D1_P, PI_GPIO0_I2C0_SDA, PI_GPIO10_SPIO_MOSI, PI_GPIO11_SPI0_SCLK, PI_GPIO14_RS232_TX, PI_GPIO15_RS232_RX, PI_GPIO16_SPI1_CS2, PI_GPIO17_SPI1_CS1, PI_GPIO18_SPI1_CS0, PI_GPIO19_SPI1_MISO, PI_GPIO1_I2C0_SCL, PI_GPIO20_SPI1_MOSI, PI_GPIO21_SPI1_CLK, PI_GPIO2_I2C1_SDA, PI_GPIO3_I2C1_SCL, PI_GPIO4_GPCLK0, PI_GPIO5_GPCLK1, PI_GPIO6_GPCLK2, PI_GPIO7_SPI0_CS1, PI_GPIO8_SPI0_CS0, PI_GPIO9_SPI0_MISO
- net labels removed: PI_GPCLK0, PI_GPCLK1, PI_GPCLK2, PI_GPIO16, PI_GPIO17, PI_GPIO18_PCMCLK, PI_GPIO19_PCMFS, PI_GPIO20_PCMDIN, PI_GPIO21_PCMDOUT, PI_RS232_RX, PI_RS232_TX, PI_SCL0_DISP, PI_SCL1, PI_SDA0_DISP, PI_SDA1, PI_SPI0_CE0_N, PI_SPI0_CE1_N, PI_SPI0_MISO, PI_SPI0_SCLK, PI_SPIO_MOSI
- wire segments 293 -> 299
Changed lines of the file:
@@
 $Descr A3 11693 16535 portrait
 encoding utf-8
-Sheet 6 11
+Sheet 6 12
 Title "HILTOP Motherboard"
 Date "26th January 2018"
@@
 $EndComp
 Text HLabel 3700 5300 0    60   Output ~ 0
-PI_RS232_RX
+PI_GPIO15_RS232_RX
 Text HLabel 3700 5200 0    60   Output ~ 0
-PI_RS232_TX
+PI_GPIO14_RS232_TX
 Text HLabel 3700 3100 0    60   Output ~ 0
-PI_SDA1
+PI_GPIO2_I2C1_SDA
 Text HLabel 3700 3200 0    60   Output ~ 0
-PI_SCL1
+PI_GPIO3_I2C1_SCL
 Text HLabel 3700 3400 0    60   Output ~ 0
-PI_GPCLK0
+PI_GPIO4_GPCLK0
 Text HLabel 3700 3500 0    60   Output ~ 0
-PI_GPCLK1
+PI_GPIO5_GPCLK1
 Text HLabel 3700 3700 0    60   Output ~ 0
-PI_GPCLK2
+PI_GPIO6_GPCLK2
 Text HLabel 3700 3800 0    60   Output ~ 0
-PI_SPI0_CE1_N
+PI_GPIO7_SPI0_CS1
 Text HLabel 3700 4000 0    60   Output ~ 0
-PI_SPI0_CE0_N
+PI_GPIO8_SPI0_CS0
 Text HLabel 3700 4100 0    60   Output ~ 0
-PI_SPI0_MISO
+PI_GPIO9_SPI0_MISO
 Text HLabel 3700 4400 0    60   Output ~ 0
-PI_SPI0_SCLK
+PI_GPIO11_SPI0_SCLK
 Text HLabel 3700 2800 0    60   Output ~ 0
-PI_SDA0_DISP
+PI_GPIO0_I2C0_SDA
 Text HLabel 3700 2900 0    60   Output ~ 0
-PI_SCL0_DISP
+PI_GPIO1_I2C0_SCL
 Text HLabel 3700 4900 0    60   Output ~ 0
 PI_GPIO12_PWM0
@@
 PI_GPIO13_PWM1
 Text HLabel 3700 5500 0    60   Output ~ 0
-PI_GPIO16
+PI_GPIO16_SPI1_CS2
 Text HLabel 3700 5600 0    60   Output ~ 0
-PI_GPIO17
+PI_GPIO17_SPI1_CS1
 Text HLabel 3700 5800 0    60   Output ~ 0
-PI_GPIO18_PCMCLK
+PI_GPIO18_SPI1_CS0
 Text HLabel 3700 5900 0    60   Output ~ 0
-PI_GPIO19_PCMFS
+PI_GPIO19_SPI1_MISO
 Text HLabel 3700 6100 0    60   Output ~ 0
-PI_GPIO20_PCMDIN
+PI_GPIO20_SPI1_MOSI
 Text HLabel 3700 6200 0    60   Output ~ 0
-PI_GPIO21_PCMDOUT
+PI_GPIO21_SPI1_CLK
 Text HLabel 3700 6400 0    60   Output ~ 0
 PI_GPIO22
@@
 Wire Wire Line
 	2600 13400 2450 13400
-Text Notes 2700 10700 0    60   ~ 0
+Text Notes 1575 10975 0    60   ~ 0
 *USB Signals to be tracked as \nmatched length 90R differential pairs
 Text Notes 4750 14200 0    60   ~ 0
@@
 	4850 4300 3700 4300
 Text HLabel 3700 4300 0    60   Output ~ 0
-PI_SPIO_MOSI
+PI_GPIO10_SPIO_MOSI
 $Comp
 L GND #PWR?
@@
 Text Label 11000 1825 2    60   ~ 0
 SDA1
+Text HLabel 4125 10700 0    60   Output ~ 0
+CAM1_D0_N
+Text HLabel 4125 10600 0    60   Output ~ 0
+CAM1_D0_P
+Text HLabel 4125 10300 0    60   Output ~ 0
+CAM1_D1_P
+Text HLabel 4125 10400 0    60   Output ~ 0
+CAM1_D1_N
+Text HLabel 4125 10100 0    60   Output ~ 0
+CAM1_CK_N
+Text HLabel 4125 10000 0    60   Output ~ 0
+CAM1_CK_P
+Wire Wire Line
+	4850 10000 4125 10000
+Wire Wire Line
+	4850 10100 4125 10100
+Wire Wire Line
+	4850 10300 4125 10300
+Wire Wire Line
+	4850 10400 4125 10400
+Wire Wire Line
+	4850 10600 4125 10600
+Wire Wire Line
+	4850 10700 4125 10700
 $EndSCHEMATC

Commit message: Furthe progress on Schematics, assigned all main footprints using latest libraries, removed unwanted tracking and parts from original PCB layout
Parts:
- C106, C109, C96, C97: footprint Capacitors_SMD:C_0603 -> Capacitor_SMD:C_0603_1608Metric
- C107, C113, C114, C116: footprint Capacitors_SMD:C_0805 -> Capacitor_SMD:C_0805_2012Metric
- C66: renamed from C?; footprint Resistor_SMD:R_0603_1608Metric -> Capacitor_SMD:C_0603_1608Metric
- C68: renamed from C?; footprint Capacitors_SMD:C_0805 -> Capacitor_SMD:C_0805_2012Metric
- FB8, R100, R101, R102, R103, R104, R73, R77, R79, R91, R98, R99: footprint Resistors_SMD:R_0603 -> Resistor_SMD:R_0603_1608Metric
- J13: footprint KiCAD_PCB_Lib:Conn_TE-DDR2-SODIMM-0.6-200P-ComputeModule -> Devtank_PCB_Lib:Conn_TE-DDR2-SODIMM-0.6-200P-ComputeModule
- R174: renamed from R?; footprint Resistors_SMD:R_0603 -> Resistor_SMD:R_0603_1608Metric
- U23: footprint Housings_SSOP:TSSOP-24_4.4x7.8mm_Pitch0.65mm -> Package_SSOP:TSSOP-24_4.4x7.8mm_P0.65mm
- U26: renamed from U?; footprint Package_DFN_QFN:DFN-8-1EP_3x2mm_P0.5mm -> Package_SOIC:SOIC-8_3.9x4.9mm_P1.27mm
- Y4: renamed from Y?; value Crystal -> 32.768kHz; footprint (none) -> Crystal:Crystal_SMD_EuroQuartz_EQ161-2Pin_3.2x1.5mm; Devtank (none) -> 181-005
- gave numbers to parts that had none: 13
Connections:
- wire segments 299 -> 300

Commit message: Schematics complete - 1st draft
Parts:
- added D38, D39, D40, D41, D42, D43, D44, D45, D46, D47, D48, D49, D50, D51, D52, D53, D54, D55, D56, D57, D58, D59, D60, D61, D62, D63, D64, D65, D66, D67, D68, D69, D70, D71, D72, D73, D74, D75, D76, D77, D78, D79, D80, D81, D82, D83: BAV99, Package_TO_SOT_SMD:SOT-23, symbol Diode:BAV99
- added R13, R15, R206, R207, R26, R29: 2K2, Resistor_SMD:R_0603_1608Metric, symbol device:R
- added R140, R141, R153, R154, R155, R156, R157, R158, R182, R183, R184, R185, R186, R187, R188, R189, R190, R191, R192, R193, R194, R195, R196, R197, R198, R28, R80, R82, R84, R86, R87, R88, R89, R90, R92, R93, R94, R95, R96, R97: 220R, Resistor_SMD:R_0603_1608Metric, symbol device:R
- added R178, R179, R180, R181: 100R, Resistor_SMD:R_0603_1608Metric, symbol device:R
- C106, C107, C109, C113, C114, C116, C47, C48, C49, C66, C68, C96, C97: symbol C -> device:C
- FB8: symbol L -> device:L
- J13: symbol DDR2_SODIMM_COMPUTE_MODULE_3 -> Devtank:DDR2_SODIMM_COMPUTE_MODULE_3
- R100, R101, R102, R103, R104, R159, R167, R168, R169, R170, R171, R172, R173, R174, R73, R77, R79, R91, R98, R99: symbol R -> device:R
- U22: footprint Package_SOIC:SOIC-8_3.9x4.9mm_P1.27mm -> Package_SO:SOIC-8_3.9x4.9mm_P1.27mm; symbol BQ32000 -> Devtank:BQ32000
- U23: symbol TPD12S016 -> Devtank:TPD12S016
- U26: value AT30TS75 -> LM75B; footprint Package_SOIC:SOIC-8_3.9x4.9mm_P1.27mm -> Package_SO:SOIC-8_3.9x4.9mm_P1.27mm; symbol AT30TS75 -> Devtank:AT30TS75
- Y3: symbol SuperCap -> Devtank:SuperCap
- Y4: symbol Crystal -> device:Crystal
Connections:
- net labels added: GPIO10, GPIO11, GPIO12, GPIO13, GPIO14, GPIO15, GPIO16, GPIO17, GPIO18, GPIO19, GPIO20, GPIO21, GPIO22, GPIO23, GPIO24, GPIO25, GPIO26, GPIO27, GPIO28, GPIO29, GPIO30, GPIO31, GPIO32, GPIO33, GPIO34, GPIO35, GPIO36, GPIO37, GPIO38, GPIO39, GPIO4, GPIO40, GPIO41, GPIO42, GPIO43, GPIO5, GPIO6, GPIO7, GPIO8, GPIO9, SCL_M0, SCL_M1, SDA_M0, SDA_M1
- wire segments 300 -> 870
Other:
- note added: "I/O Protection"
- note added: "Onboard Temperature Monitor"
- note added: "Raspberry Pi 3 Compute Module SO-DIMM"
- note added: "Real Time Clock"

Commit message: BOM nearly complete!
Parts:
- removed D66, D67, D69, D70, D71, D72, D73, D77, D78, D79, D80, D81, D82, D83: BAV99, Package_TO_SOT_SMD:SOT-23, symbol Diode:BAV99
- removed R159: 0R, Resistor_SMD:R_0603_1608Metric, symbol device:R
- removed R184, R185, R186, R187, R188, R192, R193, R194, R195, R196, R197, R198: 220R, Resistor_SMD:R_0603_1608Metric, symbol device:R
- removed R206, R207: 2K2, Resistor_SMD:R_0603_1608Metric, symbol device:R
- removed Y3: 0.22F, Devtank_PCB_Lib:Battery_SD_V_SuperCap, symbol Devtank:SuperCap
- added BT1: Battery_Cell, Devtank_PCB_Lib:BatteryHolder_Keystone_1061_1x20mm, symbol device:Battery_Cell
- added D66: MBR230LSFT, Diode_SMD:D_SOD-123F, symbol device:D_Schottky
- C47, C48: footprint Resistor_SMD:R_0603_1608Metric -> Capacitor_SMD:C_0603_1608Metric; Devtank (none) -> 106-009
- C49: footprint Resistor_SMD:R_0603_1608Metric -> Capacitor_SMD:C_0603_1608Metric; Devtank (none) -> 105-002
- C66: Devtank (none) -> 105-002
- D38, D39, D40, D41, D42, D43, D44, D45, D46, D47, D48, D49, D50, D51, D52, D53, D54, D55, D56, D57, D58, D59, D60, D61, D62, D63, D64, D65, D68, D74, D75, D76: Devtank (none) -> 134-001
- R140, R141, R153, R154, R155, R156, R157, R158, R178, R179, R180, R181, R182, R183, R189, R190, R191, R28, R80, R82, R84, R86, R87, R88, R89, R90, R92, R93, R94, R95, R96, R97: footprint Resistor_SMD:R_0603_1608Metric -> Resistor_SMD:R_0402_1005Metric
- R167: Devtank (none) -> 101-010
- U22: Devtank (none) -> 123-008
- U26: Devtank (none) -> 155-005
Connections:
- net GPIO29 is gone; now on net PI_GPIO29: J13.30 (GPIO29), R99.1
- net GPIO30 is gone; now on net PI_GPIO30: J13.34 (GPIO30)
- net GPIO31 is gone; now on net PI_GPIO31: J13.36 (GPIO31)
- net GPIO32 is gone; now on net PI_GPIO32: J13.46 (GPIO32)
- net GPIO33 is gone; now on net PI_GPIO33: J13.48 (GPIO33)
- net GPIO37 is gone; now on net PI_GPIO37: J13.60 (GPIO37)
- net GPIO38 is gone; now on net PI_GPIO38: J13.64 (GPIO38)
- net GPIO39 is gone; now on net PI_GPIO39: J13.66 (GPIO39)
- net GPIO40 is gone; now on net PI_GPIO40: J13.70 (GPIO40)
- net GPIO41 is gone; now on net PI_GPIO41: J13.72 (GPIO41)
- net GPIO42 is gone; now on net PI_GPIO42: J13.76 (GPIO42)
- net GPIO43 is gone; now on net PI_GPIO43: J13.78 (GPIO43)
- net GND: now also BT1.2 (-)
- net PI_GPIO44: now also J13.82 (GPIO44), R101.1
- net PI_GPIO45: now also J13.84 (GPIO45), R100.1
- net at U22.3 (Vback): now also D66.1 (K)
- new net: BT1.1 (+), D66.2 (A)
- no-connect marks 0 -> 41
Other:
- moved on the sheet: D68A, D68B, D74A, D74B, D75A, D75B, D76A, D76B, R183, R191

Commit message: nearly finished placing all parts!
Parts:
- removed D52, D53: BAV99, Package_TO_SOT_SMD:SOT-23, symbol Diode:BAV99
- removed R93, R94: 220R, Resistor_SMD:R_0402_1005Metric, symbol device:R
- R100, R101, R102, R99: footprint Resistor_SMD:R_0603_1608Metric -> Resistor_SMD:R_0402_1005Metric
Connections:
- net GPIO14 is gone; now on net PI_GPIO14_RS232_TX: J13.51 (GPIO14)
- net GPIO15 is gone; now on net PI_GPIO15_RS232_RX: J13.53 (GPIO15)
- net PI_GPIO2_I2C1_SDA: now also U22.5 (SDA)
- net PI_GPIO3_I2C1_SCL: now also U22.6 (SCL)
- net SCL_M1: now also U26.2 (SCL)
- net SDA_M1: now also U26.1 (SDA)
- removed net SCL1: U22.6 (SCL), U26.2 (SCL)
- removed net SDA1: U22.5 (SDA), U26.1 (SDA)
Changed lines of the file:
@@
 F 0 "R100" H 11100 10625 50  0000 C CNN
 F 1 "100K" H 11100 10525 50  0000 C CNN
-F 2 "Resistor_SMD:R_0603_1608Metric" V 10880 10575 50  0001 C CNN
+F 2 "Resistor_SMD:R_0402_1005Metric" V 10880 10575 50  0001 C CNN
 F 3 "" H 10950 10575 50  0000 C CNN
 F 4 "101-015" H 10950 10575 60  0001 C CNN "Devtank"
@@
 	1    0    0    -1
 $EndComp
-Text HLabel 2400 8975 0    60   Output ~ 0
+Text HLabel 6500 8725 0    60   Output ~ 0
 PI_GPIO15_RS232_RX
-Text HLabel 2400 8875 0    60   Output ~ 0
+Text HLabel 6500 8625 0    60   Output ~ 0
 PI_GPIO14_RS232_TX
 Text HLabel 6975 3075 0    60   Output ~ 0
@@
 F 0 "R101" H 11450 10625 50  0000 C CNN
 F 1 "100K" H 11450 10525 50  0000 C CNN
-F 2 "Resistor_SMD:R_0603_1608Metric" V 11230 10575 50  0001 C CNN
+F 2 "Resistor_SMD:R_0402_1005Metric" V 11230 10575 50  0001 C CNN
 F 3 "" H 11300 10575 50  0000 C CNN
 F 4 "101-015" H 11300 10575 60  0001 C CNN "Devtank"
@@
 F 0 "R99" H 11375 7825 50  0000 C CNN
 F 1 "100K" H 11375 7725 50  0000 C CNN
-F 2 "Resistor_SMD:R_0603_1608Metric" V 11155 7775 50  0001 C CNN
+F 2 "Resistor_SMD:R_0402_1005Metric" V 11155 7775 50  0001 C CNN
 F 3 "" H 11225 7775 50  0000 C CNN
 F 4 "101-015" H 11225 7775 60  0001 C CNN "Devtank"
@@
 F 0 "R102" H 11725 7825 50  0000 C CNN
 F 1 "100K" H 11725 7725 50  0000 C CNN
-F 2 "Resistor_SMD:R_0603_1608Metric" V 11505 7775 50  0001 C CNN
+F 2 "Resistor_SMD:R_0402_1005Metric" V 11505 7775 50  0001 C CNN
 F 3 "" H 11575 7775 50  0000 C CNN
 F 4 "101-015" H 11575 7775 60  0001 C CNN "Devtank"
@@
 Text Label 6500 6625 0    60   ~ 0
 SCL_M1
-Text Label 4650 2975 2    60   ~ 0
-SDA1
-Text Label 4650 2875 2    60   ~ 0
-SCL1
 $Comp
 L power:GND #PWR0232
@@
 	1    0    0    -1
 $EndComp
-Text Label 14525 2925 2    60   ~ 0
-SCL1
-Text Label 14525 3025 2    60   ~ 0
-SDA1
 Text HLabel 6575 14125 0    60   Output ~ 0
 CAM1_D0_N
@@
 Text Label 6500 8425 0    60   ~ 0
 GPIO13
-Text Label 6500 8625 0    60   ~ 0
-GPIO14
-Text Label 6500 8725 0    60   ~ 0
-GPIO15
 Text Label 6500 8925 0    60   ~ 0
 GPIO16
@@
 $EndComp
 $Comp
-L Diode:BAV99 D52
-U 1 1 5B5122F6
-P 3700 9825
-F 0 "D52" H 3875 9725 50  0000 C CNN
-F 1 "BAV99" H 3625 9725 50  0000 C CNN
-F 2 "Package_TO_SOT_SMD:SOT-23" H 3700 9675 50  0001 C CNN
-F 3 "" H 3700 9925 50  0001 C CNN
-F 4 "134-001" H 3700 9825 50  0001 C CNN "Devtank"
-	1    3700 9825
-	0    1    1    0
-$EndComp
-$Comp
-L Diode:BAV99 D53
-U 1 1 5B5122FC
-P 3900 9825
-F 0 "D53" H 4075 9725 50  0000 C CNN
-F 1 "BAV99" H 3825 9725 50  0000 C CNN
-F 2 "Package_TO_SOT_SMD:SOT-23" H 3900 9675 50  0001 C CNN
-F 3 "" H 3900 9925 50  0001 C CNN
-F 4 "134-001" H 3900 9825 50  0001 C CNN "Devtank"
-	1    3900 9825
-	0    1    1    0
-$EndComp
-$Comp
 L power:+3V3 #PWR0236
 U 1 1 5B512302
@@
 $EndComp
 $Comp
-L Diode:BAV99 D52
-U 2 1 5B51232C
-P 3650 8325
-F 0 "D52" H 3700 8225 50  0000 C CNN
-F 1 "BAV99" H 3450 8225 50  0000 C CNN
-F 2 "Package_TO_SOT_SMD:SOT-23" H 3650 8175 50  0001 C CNN
-F 3 "" H 3650 8425 50  0001 C CNN
-F 4 "134-001" H 3650 8325 50  0001 C CNN "Devtank"
-	2    3650 8325
-	0    1    1    0
-$EndComp
-$Comp
-L Diode:BAV99 D53
-U 2 1 5B512332
-P 3850 8325
-F 0 "D53" H 3900 8225 50  0000 C CNN
-F 1 "BAV99" H 3650 8225 50  0000 C CNN
-F 2 "Package_TO_SOT_SMD:SOT-23" H 3850 8175 50  0001 C CNN
-F 3 "" H 3850 8425 50  0001 C CNN
-F 4 "134-001" H 3850 8325 50  0001 C CNN "Devtank"
-	2    3850 8325
-	0    1    1    0
-$EndComp
-$Comp
 L Diode:BAV99 D54
 U 2 1 5B512338
@@
 	2400 8675 2650 8675
 Wire Wire Line
-	2400 8875 2650 8875
-Wire Wire Line
-	2650 8975 2400 8975
-Wire Wire Line
 	2400 9175 2650 9175
 Wire Wire Line
@@
 	2950 8575 3250 8575
 Wire Wire Line
-	2950 8875 3650 8875
-Wire Wire Line
-	2950 8975 3850 8975
-Wire Wire Line
 	2950 9175 4050 9175
 Wire Wire Line
@@
 Connection ~ 3500 8675
 Wire Wire Line
-	3650 8475 3650 8875
-Connection ~ 3650 8875
-Wire Wire Line
-	3700 9675 3700 8875
-Connection ~ 3700 8875
-Wire Wire Line
-	3850 8475 3850 8975
-Connection ~ 3850 8975
-Wire Wire Line
 	4050 8475 4050 9175
 Connection ~ 4050 9175
@@
 	3300 10125 3500 10125
 Connection ~ 3300 10125
-Wire Wire Line
-	3700 10125 3700 9975
 Connection ~ 3500 10125
 Wire Wire Line
-	3900 10125 3900 9975
-Connection ~ 3700 10125
-Wire Wire Line
 	4100 10125 4100 9975
-Connection ~ 3900 10125
 Wire Wire Line
 	4300 10125 4300 9975
@@
 Connection ~ 4500 10125
 Wire Wire Line
-	3900 9675 3900 8975
-Connection ~ 3900 8975
-Wire Wire Line
 	3450 8175 3450 8025
 Wire Wire Line
 	3250 8025 3450 8025
 Connection ~ 3250 8025
-Wire Wire Line
-	3650 8025 3650 8175
 Connection ~ 3450 8025
 Wire Wire Line
-	3850 8025 3850 8175
-Connection ~ 3650 8025
-Wire Wire Line
 	4050 8025 4050 8175
-Connection ~ 3850 8025
 Wire Wire Line
 	4250 8025 4250 8175
@@
 Text Label 5125 8675 2    60   ~ 0
 GPIO13
-Text Label 5125 8875 2    60   ~ 0
-GPIO14
-Text Label 5125 8975 2    60   ~ 0
-GPIO15
 Text Label 5125 9175 2    60   ~ 0
 GPIO16
@@
 	3500 8675 5125 8675
 Wire Wire Line
-	3650 8875 3700 8875
-Wire Wire Line
-	3700 8875 5125 8875
-Wire Wire Line
-	3850 8975 3900 8975
-Wire Wire Line
 	4050 9175 4100 9175
 Wire Wire Line
@@
 	3300 10125 3300 10200
 Wire Wire Line
-	3500 10125 3700 10125
-Wire Wire Line
-	3700 10125 3900 10125
-Wire Wire Line
-	3900 10125 4100 10125
-Wire Wire Line
 	4100 10125 4300 10125
 Wire Wire Line
@@
 	4500 10125 4700 10125
 Wire Wire Line
-	3900 8975 5125 8975
-Wire Wire Line
 	3250 8025 3250 8175
 Wire Wire Line
-	3450 8025 3650 8025
-Wire Wire Line
-	3650 8025 3850 8025
-Wire Wire Line
-	3850 8025 4050 8025
-Wire Wire Line
 	4050 8025 4250 8025
 Wire Wire Line
@@
 $EndComp
 $Comp
-L device:R R93
-U 1 1 5C5AF721
-P 2800 8875
-F 0 "R93" V 2750 8650 50  0000 C CNN
-F 1 "220R" V 2750 9100 50  0000 C CNN
-F 2 "Resistor_SMD:R_0402_1005Metric" V 2730 8875 50  0001 C CNN
-F 3 "" H 2800 8875 50  0000 C CNN
-F 4 "101-049" H 2800 8875 60  0001 C CNN "Devtank"
-	1    2800 8875
-	0    1    1    0
-$EndComp
-$Comp
-L device:R R94
-U 1 1 5C5AFCCB
-P 2800 8975
-F 0 "R94" V 2750 8750 50  0000 C CNN
-F 1 "220R" V 2750 9200 50  0000 C CNN
-F 2 "Resistor_SMD:R_0402_1005Metric" V 2730 8975 50  0001 C CNN
-F 3 "" H 2800 8975 50  0000 C CNN
-F 4 "101-049" H 2800 8975 60  0001 C CNN "Devtank"
-	1    2800 8975
-	0    1    1    0
-$EndComp
-$Comp
 L device:R R95
 U 1 1 5C5AFE45
@@
 Wire Wire Line
 	1875 3150 2175 3150
+Wire Wire Line
+	3450 8025 4050 8025
+Wire Wire Line
+	3500 10125 4100 10125
+Text Label 14525 3025 2    60   ~ 0
+SDA_M1
+Text Label 14525 2925 2    60   ~ 0
+SCL_M1
+Text HLabel 4650 2975 2    60   Output ~ 0
+PI_GPIO2_I2C1_SDA
+Text HLabel 4650 2875 2    60   Output ~ 0
+PI_GPIO3_I2C1_SCL
 $EndSCHEMATC
