File: HILTOP_motherboard/Processor.sch (KiCad schematic (older format))
At the start: 104 parts, among them J13 DDR2_SODIMM_COMPUTE_MODULE_3, U22 BQ32000, U23 TPD12S016, U26 LM75B, Y4 32.768kHz

Commit message: DRC checks complete, all errors and warnings cleared. BOM created and parts rationalised.
Parts:
- R100, R101, R102, R99: Devtank 101-015 -> 101-502
- R140, R141, R153, R154, R155, R156, R157, R158, R182, R183, R189, R190, R191, R28, R80, R82, R84, R86, R87, R88, R89, R90, R92, R95, R96, R97: Devtank 101-049 -> 101-503
- R178, R179, R180, R181: Devtank 101-018 -> 101-500
Connections:
- wire segments 712 -> 716
Changed lines of the file:
@@
 F 2 "Resistor_SMD:R_0402_1005Metric" V 10880 10575 50  0001 C CNN
 F 3 "" H 10950 10575 50  0000 C CNN
-F 4 "101-015" H 10950 10575 60  0001 C CNN "Devtank"
+F 4 "101-502" H 10950 10575 60  0001 C CNN "Devtank"
 	1    10950 10575
 	1    0    0    -1
@@
 F 2 "Resistor_SMD:R_0402_1005Metric" V 11230 10575 50  0001 C CNN
 F 3 "" H 11300 10575 50  0000 C CNN
-F 4 "101-015" H 11300 10575 60  0001 C CNN "Devtank"
+F 4 "101-502" H 11300 10575 60  0001 C CNN "Devtank"
 	1    11300 10575
 	1    0    0    -1
@@
 F 2 "Resistor_SMD:R_0402_1005Metric" V 11155 7775 50  0001 C CNN
 F 3 "" H 11225 7775 50  0000 C CNN
-F 4 "101-015" H 11225 7775 60  0001 C CNN "Devtank"
+F 4 "101-502" H 11225 7775 60  0001 C CNN "Devtank"
 	1    11225 7775
 	1    0    0    -1
@@
 F 2 "Resistor_SMD:R_0402_1005Metric" V 11505 7775 50  0001 C CNN
 F 3 "" H 11575 7775 50  0000 C CNN
-F 4 "101-015" H 11575 7775 60  0001 C CNN "Devtank"
+F 4 "101-502" H 11575 7775 60  0001 C CNN "Devtank"
 	1    11575 7775
 	1    0    0    -1
@@
 F 2 "Resistor_SMD:R_0402_1005Metric" V 7230 2875 50  0001 C CNN
 F 3 "" H 7300 2875 50  0000 C CNN
-F 4 "101-018" H 7300 2875 60  0001 C CNN "Devtank"
+F 4 "101-500" H 7300 2875 60  0001 C CNN "Devtank"
 	1    7300 2875
 	0    1    1    0
@@
 F 2 "Resistor_SMD:R_0402_1005Metric" V 7230 2975 50  0001 C CNN
 F 3 "" H 7300 2975 50  0000 C CNN
-F 4 "101-018" H 7300 2975 60  0001 C CNN "Devtank"
+F 4 "101-500" H 7300 2975 60  0001 C CNN "Devtank"
 	1    7300 2975
 	0    1    1    0
@@
 F 2 "Resistor_SMD:R_0402_1005Metric" V 7230 3075 50  0001 C CNN
 F 3 "" H 7300 3075 50  0000 C CNN
-F 4 "101-018" H 7300 3075 60  0001 C CNN "Devtank"
+F 4 "101-500" H 7300 3075 60  0001 C CNN "Devtank"
 	1    7300 3075
 	0    1    1    0
@@
 F 2 "Resistor_SMD:R_0402_1005Metric" V 7230 3175 50  0001 C CNN
 F 3 "" H 7300 3175 50  0000 C CNN
-F 4 "101-018" H 7300 3175 60  0001 C CNN "Devtank"
+F 4 "101-500" H 7300 3175 60  0001 C CNN "Devtank"
 	1    7300 3175
 	0    1    1    0
@@
 F 2 "Resistor_SMD:R_0402_1005Metric" V 2730 5850 50  0001 C CNN
 F 3 "" H 2800 5850 50  0000 C CNN
-F 4 "101-049" H 2800 5850 60  0001 C CNN "Devtank"
+F 4 "101-503" H 2800 5850 60  0001 C CNN "Devtank"
 	1    2800 5850
 	0    1    1    0
@@
 F 2 "Resistor_SMD:R_0402_1005Metric" V 2730 5950 50  0001 C CNN
 F 3 "" H 2800 5950 50  0000 C CNN
-F 4 "101-049" H 2800 5950 60  0001 C CNN "Devtank"
+F 4 "101-503" H 2800 5950 60  0001 C CNN "Devtank"
 	1    2800 5950
 	0    1    1    0
@@
 F 2 "Resistor_SMD:R_0402_1005Metric" V 2730 6150 50  0001 C CNN
 F 3 "" H 2800 6150 50  0000 C CNN
-F 4 "101-049" H 2800 6150 60  0001 C CNN "Devtank"
+F 4 "101-503" H 2800 6150 60  0001 C CNN "Devtank"
 	1    2800 6150
 	0    1    1    0
@@
 F 2 "Resistor_SMD:R_0402_1005Metric" V 2730 6250 50  0001 C CNN
 F 3 "" H 2800 6250 50  0000 C CNN
-F 4 "101-049" H 2800 6250 60  0001 C CNN "Devtank"
+F 4 "101-503" H 2800 6250 60  0001 C CNN "Devtank"
 	1    2800 6250
 	0    1    1    0
@@
 F 2 "Resistor_SMD:R_0402_1005Metric" V 2730 6450 50  0001 C CNN
 F 3 "" H 2800 6450 50  0000 C CNN
-F 4 "101-049" H 2800 6450 60  0001 C CNN "Devtank"
+F 4 "101-503" H 2800 6450 60  0001 C CNN "Devtank"
 	1    2800 6450
 	0    1    1    0
@@
 F 2 "Resistor_SMD:R_0402_1005Metric" V 2730 6550 50  0001 C CNN
 F 3 "" H 2800 6550 50  0000 C CNN
-F 4 "101-049" H 2800 6550 60  0001 C CNN "Devtank"
+F 4 "101-503" H 2800 6550 60  0001 C CNN "Devtank"
 	1    2800 6550
 	0    1    1    0
@@
 F 2 "Resistor_SMD:R_0402_1005Metric" V 2730 6750 50  0001 C CNN
 F 3 "" H 2800 6750 50  0000 C CNN
-F 4 "101-049" H 2800 6750 60  0001 C CNN "Devtank"
+F 4 "101-503" H 2800 6750 60  0001 C CNN "Devtank"
 	1    2800 6750
 	0    1    1    0
@@
 F 2 "Resistor_SMD:R_0402_1005Metric" V 2730 6850 50  0001 C CNN
 F 3 "" H 2800 6850 50  0000 C CNN
-F 4 "101-049" H 2800 6850 60  0001 C CNN "Devtank"
+F 4 "101-503" H 2800 6850 60  0001 C CNN "Devtank"
 	1    2800 6850
 	0    1    1    0
@@
 F 2 "Resistor_SMD:R_0402_1005Metric" V 2730 8575 50  0001 C CNN
 F 3 "" H 2800 8575 50  0000 C CNN
-F 4 "101-049" H 2800 8575 60  0001 C CNN "Devtank"
+F 4 "101-503" H 2800 8575 60  0001 C CNN "Devtank"
 	1    2800 8575
 	0    1    1    0
@@
 F 2 "Resistor_SMD:R_0402_1005Metric" V 2730 9175 50  0001 C CNN
 F 3 "" H 2800 9175 50  0000 C CNN
-F 4 "101-049" H 2800 9175 60  0001 C CNN "Devtank"
+F 4 "101-503" H 2800 9175 60  0001 C CNN "Devtank"
 	1    2800 9175
 	0    1    1    0
@@
 F 2 "Resistor_SMD:R_0402_1005Metric" V 2730 9275 50  0001 C CNN
 F 3 "" H 2800 9275 50  0000 C CNN
-F 4 "101-049" H 2800 9275 60  0001 C CNN "Devtank"
+F 4 "101-503" H 2800 9275 60  0001 C CNN "Devtank"
 	1    2800 9275
 	0    1    1    0
@@
 F 2 "Resistor_SMD:R_0402_1005Metric" V 2730 9475 50  0001 C CNN
 F 3 "" H 2800 9475 50  0000 C CNN
-F 4 "101-049" H 2800 9475 60  0001 C CNN "Devtank"
+F 4 "101-503" H 2800 9475 60  0001 C CNN "Devtank"
 	1    2800 9475
 	0    1    1    0
@@
 F 2 "Resistor_SMD:R_0402_1005Metric" V 2730 9575 50  0001 C CNN
 F 3 "" H 2800 9575 50  0000 C CNN
-F 4 "101-049" H 2800 9575 60  0001 C CNN "Devtank"
+F 4 "101-503" H 2800 9575 60  0001 C CNN "Devtank"
 	1    2800 9575
 	0    1    1    0
@@
 F 2 "Resistor_SMD:R_0402_1005Metric" V 2730 11500 50  0001 C CNN
 F 3 "" H 2800 11500 50  0000 C CNN
-F 4 "101-049" H 2800 11500 60  0001 C CNN "Devtank"
+F 4 "101-503" H 2800 11500 60  0001 C CNN "Devtank"
 	1    2800 11500
 	0    1    1    0
@@
 F 2 "Resistor_SMD:R_0402_1005Metric" V 2730 11600 50  0001 C CNN
 F 3 "" H 2800 11600 50  0000 C CNN
-F 4 "101-049" H 2800 11600 60  0001 C CNN "Devtank"
+F 4 "101-503" H 2800 11600 60  0001 C CNN "Devtank"
 	1    2800 11600
 	0    1    1    0
@@
 F 2 "Resistor_SMD:R_0402_1005Metric" V 2730 11800 50  0001 C CNN
 F 3 "" H 2800 11800 50  0000 C CNN
-F 4 "101-049" H 2800 11800 60  0001 C CNN "Devtank"
+F 4 "101-503" H 2800 11800 60  0001 C CNN "Devtank"
 	1    2800 11800
 	0    1    1    0
@@
 F 2 "Resistor_SMD:R_0402_1005Metric" V 2730 11900 50  0001 C CNN
 F 3 "" H 2800 11900 50  0000 C CNN
-F 4 "101-049" H 2800 11900 60  0001 C CNN "Devtank"
+F 4 "101-503" H 2800 11900 60  0001 C CNN "Devtank"
 	1    2800 11900
 	0    1    1    0
@@
 F 2 "Resistor_SMD:R_0402_1005Metric" V 2730 12100 50  0001 C CNN
 F 3 "" H 2800 12100 50  0000 C CNN
-F 4 "101-049" H 2800 12100 60  0001 C CNN "Devtank"
+F 4 "101-503" H 2800 12100 60  0001 C CNN "Devtank"
 	1    2800 12100
 	0    1    1    0
@@
 F 2 "Resistor_SMD:R_0402_1005Metric" V 2730 12200 50  0001 C CNN
 F 3 "" H 2800 12200 50  0000 C CNN
-F 4 "101-049" H 2800 12200 60  0001 C CNN "Devtank"
+F 4 "101-503" H 2800 12200 60  0001 C CNN "Devtank"
 	1    2800 12200
 	0    1    1    0
@@
 F 2 "Resistor_SMD:R_0402_1005Metric" V 2730 12400 50  0001 C CNN
 F 3 "" H 2800 12400 50  0000 C CNN
-F 4 "101-049" H 2800 12400 60  0001 C CNN "Devtank"
+F 4 "101-503" H 2800 12400 60  0001 C CNN "Devtank"
 	1    2800 12400
 	0    1    1    0
@@
 F 2 "Resistor_SMD:R_0402_1005Metric" V 2730 12500 50  0001 C CNN
 F 3 "" H 2800 12500 50  0000 C CNN
-F 4 "101-049" H 2800 12500 60  0001 C CNN "Devtank"
+F 4 "101-503" H 2800 12500 60  0001 C CNN "Devtank"
 	1    2800 12500
 	0    1    1    0
@@
 F 2 "Resistor_SMD:R_0402_1005Metric" V 14180 13000 50  0001 C CNN
 F 3 "" H 14250 13000 50  0000 C CNN
-F 4 "101-049" H 14250 13000 60  0001 C CNN "Devtank"
+F 4 "101-503" H 14250 13000 60  0001 C CNN "Devtank"
 	1    14250 13000
 	0    1    1    0
@@
 F 2 "Resistor_SMD:R_0402_1005Metric" V 14180 13100 50  0001 C CNN
 F 3 "" H 14250 13100 50  0000 C CNN
-F 4 "101-049" H 14250 13100 60  0001 C CNN "Devtank"
+F 4 "101-503" H 14250 13100 60  0001 C CNN "Devtank"
 	1    14250 13100
 	0    1    1    0
@@
 F 2 "Resistor_SMD:R_0402_1005Metric" V 14180 13200 50  0001 C CNN
 F 3 "" H 14250 13200 50  0000 C CNN
-F 4 "101-049" H 14250 13200 60  0001 C CNN "Devtank"
+F 4 "101-503" H 14250 13200 60  0001 C CNN "Devtank"
 	1    14250 13200
 	0    1    1    0
@@
 F 2 "Resistor_SMD:R_0402_1005Metric" V 14180 13300 50  0001 C CNN
 F 3 "" H 14250 13300 50  0000 C CNN
-F 4 "101-049" H 14250 13300 60  0001 C CNN "Devtank"
+F 4 "101-503" H 14250 13300 60  0001 C CNN "Devtank"
 	1    14250 13300
 	0    1    1    0
@@
 F 2 "Resistor_SMD:R_0402_1005Metric" V 2730 8675 50  0001 C CNN
 F 3 "" H 2800 8675 50  0000 C CNN
-F 4 "101-049" H 2800 8675 60  0001 C CNN "Devtank"
+F 4 "101-503" H 2800 8675 60  0001 C CNN "Devtank"
 	1    2800 8675
 	0    1    1    0
@@
 Text HLabel 4650 2875 2    60   Output ~ 0
 PI_GPIO3_I2C1_SCL
+$Comp
+L power:PWR_FLAG #FLG0109
+U 1 1 5CAC4CA0
+P 9375 19325
+F 0 "#FLG0109" H 9375 19400 50  0001 C CNN
+F 1 "PWR_FLAG" V 9375 19650 50  0000 C CNN
+F 2 "" H 9375 19325 50  0001 C CNN
+F 3 "" H 9375 19325 50  0001 C CNN
+	1    9375 19325
+	-1   0    0    1
+$EndComp
+Wire Wire Line
+	9375 19325 9375 19225
+Connection ~ 9375 19225
+$Comp
+L power:PWR_FLAG #FLG0110
+U 1 1 5CBF6595
+P 10575 19300
+F 0 "#FLG0110" H 10575 19375 50  0001 C CNN
+F 1 "PWR_FLAG" V 10575 19625 50  0000 C CNN
+F 2 "" H 10575 19300 50  0001 C CNN
+F 3 "" H 10575 19300 50  0001 C CNN
+	1    10575 19300
+	-1   0    0    1
+$EndComp
+Wire Wire Line
+	10575 19300 10575 19225
+Connection ~ 10575 19225
+$Comp
+L power:PWR_FLAG #FLG0111
+U 1 1 5CC8900F
+P 11425 19275
+F 0 "#FLG0111" H 11425 19350 50  0001 C CNN
+F 1 "PWR_FLAG" V 11425 19600 50  0000 C CNN
+F 2 "" H 11425 19275 50  0001 C CNN
+F 3 "" H 11425 19275 50  0001 C CNN
+	1    11425 19275
+	-1   0    0    1
+$EndComp
+Wire Wire Line
+	11425 19275 11425 19225
+Connection ~ 11425 19225
+$Comp
+L power:PWR_FLAG #FLG0112
+U 1 1 5CD1BFB8
+P 12325 19300
+F 0 "#FLG0112" H 12325 19375 50  0001 C CNN
+F 1 "PWR_FLAG" V 12325 19625 50  0000 C CNN
+F 2 "" H 12325 19300 50  0001 C CNN
+F 3 "" H 12325 19300 50  0001 C CNN
+	1    12325 19300
+	-1   0    0    1
+$EndComp
+Wire Wire Line
+	12325 19300 12325 19225
+Connection ~ 12325 19225
 $EndSCHEMATC

Commit message: finished new tracking for RS485 signals and general house keeping
Parts:
- R168, R170, R172: value DNF -> 0R
Changed lines of the file:
@@
 Sheet 4 12
 Title "HILTOP Motherboard"
-Date "2019-01-10"
-Rev "Issue 1"
+Date "2019-07-03"
+Rev "Rev B"
 Comp "Devtank Ltd"
 Comment1 ""
@@
 P 12350 2775
 F 0 "R168" H 12450 2825 50  0000 C CNN
-F 1 "DNF" H 12475 2725 50  0000 C CNN
+F 1 "0R" H 12475 2725 50  0000 C CNN
 F 2 "Resistor_SMD:R_0402_1005Metric" V 12280 2775 50  0001 C CNN
 F 3 "" H 12350 2775 50  0000 C CNN
@@
 P 12600 2775
 F 0 "R170" H 12700 2825 50  0000 C CNN
-F 1 "DNF" H 12725 2725 50  0000 C CNN
+F 1 "0R" H 12725 2725 50  0000 C CNN
 F 2 "Resistor_SMD:R_0402_1005Metric" V 12530 2775 50  0001 C CNN
 F 3 "" H 12600 2775 50  0000 C CNN
@@
 P 12850 2775
 F 0 "R172" H 13000 2825 50  0000 C CNN
-F 1 "DNF" H 12975 2725 50  0000 C CNN
+F 1 "0R" H 12975 2725 50  0000 C CNN
 F 2 "Resistor_SMD:R_0402_1005Metric" V 12780 2775 50  0001 C CNN
 F 3 "" H 12850 2775 50  0000 C CNN

Commit message: Rev B
Parts:
- R168, R170, R172: Devtank (none) -> 101-506
Changed lines of the file:
@@
 F 2 "Resistor_SMD:R_0402_1005Metric" V 12280 2775 50  0001 C CNN
 F 3 "" H 12350 2775 50  0000 C CNN
+F 4 "101-506" H 12350 2775 50  0001 C CNN "Devtank"
 	1    12350 2775
 	1    0    0    -1
@@
 F 2 "Resistor_SMD:R_0402_1005Metric" V 12530 2775 50  0001 C CNN
 F 3 "" H 12600 2775 50  0000 C CNN
+F 4 "101-506" H 12600 2775 50  0001 C CNN "Devtank"
 	1    12600 2775
 	1    0    0    -1
@@
 F 2 "Resistor_SMD:R_0402_1005Metric" V 12780 2775 50  0001 C CNN
 F 3 "" H 12850 2775 50  0000 C CNN
+F 4 "101-506" H 12850 2775 50  0001 C CNN "Devtank"
 	1    12850 2775
 	1    0    0    -1

Commit message: Rev C - pre-release
Parts:
- BT1: symbol device:Battery_Cell -> HILTOP_Motherboard-rescue:Battery_Cell-device
- C106, C107, C109, C113, C114, C116, C47, C48, C49, C66, C68, C96, C97: symbol device:C -> HILTOP_Motherboard-rescue:C-device
- D38, D39, D40, D41, D42, D43, D44, D45, D46, D47, D48, D49, D50, D51, D54, D55, D56, D57, D58, D59, D60, D61, D62, D63, D64, D65, D68, D74, D75, D76: symbol Diode:BAV99 -> HILTOP_Motherboard-rescue:BAV99-Diode
- D66: symbol device:D_Schottky -> HILTOP_Motherboard-rescue:D_Schottky-device
- FB8: symbol device:L -> HILTOP_Motherboard-rescue:L-device
- R100, R101, R102, R103, R104, R13, R140, R141, R15, R153, R154, R155, R156, R157, R158, R167, R168, R169, R170, R171, R172, R173, R174, R178, R179, R180, R181, R182, R183, R189, R190, R191, R26, R28, R29, R73, R77, R79, R80, R82, R84, R86, R87, R88, R89, R90, R91, R92, R95, R96, R97, R98, R99: symbol device:R -> HILTOP_Motherboard-rescue:R-device
- Y4: symbol device:Crystal -> HILTOP_Motherboard-rescue:Crystal-device
Connections:
- net labels added: RUN
- wire segments 716 -> 717
- no-connect marks 41 -> 40

Commit message: changed silkscreen to revD and updated sheet information
Parts:
- J13: symbol Devtank:DDR2_SODIMM_COMPUTE_MODULE_3 -> HILTOP_Motherboard-rescue:DDR2_SODIMM_COMPUTE_MODULE_3-Devtank
- U22: symbol Devtank:BQ32000 -> HILTOP_Motherboard-rescue:BQ32000-Devtank
- U23: symbol Devtank:TPD12S016 -> HILTOP_Motherboard-rescue:TPD12S016-Devtank
- U26: symbol Devtank:AT30TS75 -> HILTOP_Motherboard-rescue:AT30TS75-Devtank
Changed lines of the file:
@@
 Sheet 4 12
 Title "HILTOP Motherboard"
-Date "2020-04-28"
-Rev "Rev C"
+Date "2021-02-17"
+Rev "Rev D"
 Comp "Devtank Ltd"
-Comment1 ""
+Comment1 "Part No: 304-001"
 Comment2 ""
 Comment3 ""
@@
 $EndDescr
 $Comp
-L Devtank:TPD12S016 U23
+L HILTOP_Motherboard-rescue:TPD12S016-Devtank U23
 U 1 1 58C8C84B
 P 4175 19375
@@
 $EndComp
 $Comp
-L Devtank:DDR2_SODIMM_COMPUTE_MODULE_3 J13
+L HILTOP_Motherboard-rescue:DDR2_SODIMM_COMPUTE_MODULE_3-Devtank J13
 U 1 1 58C8E0D6
 P 8050 11075
@@
 $EndComp
 $Comp
-L Devtank:+CM_3V3 #PWR0264
+L HILTOP_Motherboard-rescue:+CM_3V3-Devtank #PWR0264
 U 1 1 58CDF819
 P 10200 15525
@@
 $EndComp
 $Comp
-L Devtank:+CM_VDAC #PWR0261
+L HILTOP_Motherboard-rescue:+CM_VDAC-Devtank #PWR0261
 U 1 1 58CDF843
 P 10050 15275
@@
 $EndComp
 $Comp
-L Devtank:+CM_3V3 #PWR0276
+L HILTOP_Motherboard-rescue:+CM_3V3-Devtank #PWR0276
 U 1 1 58CDF86D
 P 11425 19125
@@
 $EndComp
 $Comp
-L Devtank:+CM_3V3 #PWR0250
+L HILTOP_Motherboard-rescue:+CM_3V3-Devtank #PWR0250
 U 1 1 58CE0542
 P 6550 15525
@@
 $EndComp
 $Comp
-L Devtank:+CM_VDAC #PWR0251
+L HILTOP_Motherboard-rescue:+CM_VDAC-Devtank #PWR0251
 U 1 1 58CE084D
 P 6750 15325
@@
 $EndComp
 $Comp
-L Devtank:+CM_VDAC #PWR0257
+L HILTOP_Motherboard-rescue:+CM_VDAC-Devtank #PWR0257
 U 1 1 58CE158C
 P 9375 19125
@@
 $EndComp
 $Comp
-L Devtank:+CM_1V8 #PWR0260
+L HILTOP_Motherboard-rescue:+CM_1V8-Devtank #PWR0260
 U 1 1 58CE15AF
 P 9850 14975
@@
 $EndComp
 $Comp
-L Devtank:+CM_1V8 #PWR0252
+L HILTOP_Motherboard-rescue:+CM_1V8-Devtank #PWR0252
 U 1 1 58CE15E2
 P 6950 15075
@@
 $EndComp
 $Comp
-L Devtank:+CM_1V8 #PWR0267
+L HILTOP_Motherboard-rescue:+CM_1V8-Devtank #PWR0267
 U 1 1 58CE1D8C
 P 10575 19125
@@
 SDX_D3
 $Comp
-L Devtank:+CM_3V3 #PWR0248
+L HILTOP_Motherboard-rescue:+CM_3V3-Devtank #PWR0248
 U 1 1 58CE7EA6
 P 6225 7950
@@
 $EndComp
 $Comp
-L Devtank:+CM_3V3 #PWR0270
+L HILTOP_Motherboard-rescue:+CM_3V3-Devtank #PWR0270
 U 1 1 58CE8109
 P 10925 7975
@@
 HDMI_CK_N
 $Comp
-L Devtank:+CM_1V8 #PWR0233
+L HILTOP_Motherboard-rescue:+CM_1V8-Devtank #PWR0233
 U 1 1 59325D05
 P 3025 18075
@@
 $EndComp
 $Comp
-L Devtank:+CM_3V3 #PWR0231
+L HILTOP_Motherboard-rescue:+CM_3V3-Devtank #PWR0231
 U 1 1 59325DF0
 P 2575 18075
@@
 $EndComp
 $Comp
-L Devtank:+CM_5V #PWR0285
+L HILTOP_Motherboard-rescue:+CM_5V-Devtank #PWR0285
 U 1 1 5A76E760
 P 12325 19125
@@
 $EndComp
 $Comp
-L Devtank:+CM_5V #PWR0266
+L HILTOP_Motherboard-rescue:+CM_5V-Devtank #PWR0266
 U 1 1 5A76EDE6
 P 10500 15875
@@
 $EndComp
 $Comp
-L Devtank:+CM_5V #PWR0249
+L HILTOP_Motherboard-rescue:+CM_5V-Devtank #PWR0249
 U 1 1 5A76FB57
 P 6250 15875
@@
 $EndComp
 $Comp
-L Devtank:BQ32000 U22
+L HILTOP_Motherboard-rescue:BQ32000-Devtank U22
 U 1 1 5A954FD3
 P 3375 3175
@@
 $EndComp
 $Comp
-L Devtank:AT30TS75 U?
+L HILTOP_Motherboard-rescue:AT30TS75-Devtank U?
 U 1 1 5A94C016
 P 13425 2775
