File: HILTOP_motherboard/BoardPower.sch (KiCad schematic (older format))
At the start: 50 parts, among them Q3 2N7002, U24 MAX16054, U27 TPS54394, U28 LP2985

Commit message: Furthe progress on Schematics, assigned all main footprints using latest libraries, removed unwanted tracking and parts from original PCB layout
Parts:
- C110, C135, C136, C137, C138, C139, C140, C141, C142, C143, C144, C145, C146, C147, C148, C149, C150, C167, C169, C173, C175, C176, C177: footprint Capacitors_SMD:C_0603 -> Capacitor_SMD:C_0603_1608Metric
- C133, C134, C168, C174: footprint Capacitors_SMD:C_1206 -> Capacitor_SMD:C_1206_3216Metric
- C170, C171, C172, C178: footprint Capacitors_SMD:C_0805 -> Capacitor_SMD:C_0805_2012Metric
- L10, L9: footprint KiCAD_PCB_Lib:Inductor_8x8 -> Devtank_PCB_Lib:Inductor_8x8
- Q3: footprint TO_SOT_Packages_SMD:SOT-23 -> Package_TO_SOT_SMD:SOT-23
- R106, R107, R108, R109, R110, R111, R160, R161, R162, R163, R164: footprint Resistors_SMD:R_0603 -> Resistor_SMD:R_0603_1608Metric
- U24: footprint TO_SOT_Packages_SMD:TSOT-23-6_MK06A -> Package_TO_SOT_SMD:TSOT-23-6
- U27: footprint KiCAD_PCB_Lib:HTSSOP-16_4.4x5mm_Pitch0.65mm -> Devtank_PCB_Lib:HTSSOP-16_4.4x5mm_Pitch0.65mm
- U28: footprint TO_SOT_Packages_SMD:SOT-23-5 -> Package_TO_SOT_SMD:SOT-23-5

Commit message: Schematics complete - 1st draft
Parts:
- C110, C133, C134, C135, C136, C137, C138, C139, C140, C141, C142, C143, C144, C145, C146, C147, C148, C149, C150, C167, C168, C169, C170, C171, C172, C173, C174, C175, C176, C177, C178: symbol C -> device:C
- D18: symbol LED -> device:LED
- D24: symbol D_Schottky -> device:D_Schottky
- L10, L9: symbol L -> device:L
- Q3: symbol 2N7002 -> Transistor:2N7002
- R106, R107, R108, R109, R110, R111, R160, R161, R162, R163, R164: symbol R -> device:R
- U24: symbol MAX16054 -> Devtank:MAX16054
- U27: symbol TPS54394 -> Devtank:TPS54394
- U28: symbol LP2985 -> Devtank:LP2985

Commit message: BOM nearly complete!
Parts:
- D18: value Green_LED -> GRN; footprint LEDs:LED_0603 -> LED_SMD:LED_0402_1005Metric; Devtank 110-002 -> 110-005
Connections:
- net at Q3.1 (G): now also R108.1, R110.2
- no-connect marks 0 -> 2
Changed lines of the file:
@@
 	4700 4700 4700 4850
 Wire Wire Line
-	4700 5150 4700 5450
+	4700 5150 4700 5300
 Connection ~ 4700 5300
 Wire Wire Line
-	4700 5850 4700 6200
+	4700 5850 4700 5950
 Text Notes 4500 6750 0    60   ~ 0
 LOW = PSU ON\nHIGH or FLOATING = PSU OFF
@@
 $EndComp
 Wire Wire Line
-	3950 5700 4400 5700
+	3950 5700 4000 5700
 Wire Wire Line
 	4450 5950 4700 5950
@@
 	3200 6000 3450 6000
 Wire Wire Line
-	3450 6000 3450 6350
+	3450 6000 3450 6250
 Wire Wire Line
 	2000 5850 1750 5850
 Wire Wire Line
-	2600 4400 2600 5300
+	2600 4400 2600 4600
 $Comp
 L power:GND #PWR0301
@@
 P 3550 5250
 F 0 "D18" H 3550 5350 50  0000 C CNN
-F 1 "Green_LED" H 3550 5150 50  0000 C CNN
-F 2 "LEDs:LED_0603" H 3550 5250 50  0001 C CNN
+F 1 "GRN" H 3550 5150 50  0000 C CNN
+F 2 "LED_SMD:LED_0402_1005Metric" H 3550 5250 50  0001 C CNN
 F 3 "" H 3550 5250 50  0000 C CNN
-F 4 "110-002" H 3550 5250 60  0001 C CNN "Devtank"
+F 4 "110-005" H 3550 5250 60  0001 C CNN "Devtank"
 	1    3550 5250
 	0    -1   -1   0
@@
 $EndComp
 Wire Wire Line
-	10150 2350 10150 2800
+	10150 2350 10150 2650
 Wire Wire Line
 	10150 2350 10450 2350
@@
 	7450 2800 7450 2650
 Wire Wire Line
-	7100 2650 10150 2650
+	7100 2650 7450 2650
 Connection ~ 10150 2650
 Wire Wire Line
@@
 	7450 3100 7450 3250
 Wire Wire Line
-	10150 3100 10150 3350
+	10150 3100 10150 3250
 Wire Wire Line
 	9700 3250 9700 3100
@@
 $EndComp
 Wire Wire Line
-	10150 650  10150 1250
+	10150 650  10150 1100
 Wire Wire Line
 	7450 1250 7450 1100
 Wire Wire Line
-	1250 1100 10150 1100
+	1250 1100 7450 1100
 Connection ~ 10150 1100
 Wire Wire Line
@@
 	7450 1550 7450 1700
 Wire Wire Line
-	10150 1550 10150 1800
+	10150 1550 10150 1700
 Wire Wire Line
 	9700 1700 9700 1550
@@
 $EndComp
 Wire Wire Line
-	10050 4350 10050 4950
+	10050 4350 10050 4800
 Connection ~ 10050 4800
 Wire Wire Line
@@
 Connection ~ 9600 4800
 Wire Wire Line
-	10050 5250 10050 5500
+	10050 5250 10050 5400
 Wire Wire Line
 	9600 5400 9600 5250
@@
 Connection ~ 10050 5400
 Wire Wire Line
-	8250 5400 10050 5400
-Wire Wire Line
-	8000 4800 10050 4800
+	8250 5400 8700 5400
+Wire Wire Line
+	8000 4800 8050 4800
 Wire Wire Line
 	10350 4350 10050 4350
@@
 Connection ~ 8050 4800
 Wire Wire Line
-	6200 4800 6500 4800
-Wire Wire Line
-	6450 4400 6450 5500
-Wire Wire Line
-	6150 4400 7100 4400
+	6200 4800 6450 4800
+Wire Wire Line
+	6450 4400 6450 4800
+Wire Wire Line
+	6150 4400 6450 4400
 Wire Wire Line
 	6150 4300 6150 4400
@@
 $EndComp
 Wire Wire Line
-	6200 5100 6200 5300
+	6200 5100 6200 5150
 Wire Wire Line
 	6200 5150 6500 5150
@@
 $EndComp
 Wire Wire Line
-	4500 2150 5350 2150
+	4500 2150 5100 2150
 Connection ~ 5100 2150
 $Comp
@@
 $EndComp
 Wire Wire Line
-	5800 2450 5800 2550
-Wire Wire Line
-	5650 2150 7100 2150
+	5800 2450 5800 2500
+Wire Wire Line
+	5650 2150 5800 2150
 Wire Wire Line
 	4500 2300 5400 2300
@@
 	4600 1850 4600 1500
 Wire Wire Line
-	2700 1500 4800 1500
+	2700 1500 2900 1500
 Wire Wire Line
 	2900 1500 2900 1850
@@
 	2750 2000 3000 2000
 Wire Wire Line
-	2200 2150 3000 2150
+	2200 2150 2400 2150
 Connection ~ 2400 2150
 $Comp
@@
 $EndComp
 Wire Wire Line
-	900  2150 1900 2150
-Wire Wire Line
-	1700 2450 1700 2550
+	900  2150 1250 2150
+Wire Wire Line
+	1700 2450 1700 2500
 Wire Wire Line
 	3000 2300 2150 2300
@@
 $EndComp
 Wire Wire Line
-	900  2750 3000 2750
-Wire Wire Line
-	1250 2600 1250 2950
+	900  2750 1250 2750
+Wire Wire Line
+	1250 2600 1250 2750
 Connection ~ 1250 2750
 $Comp
@@
 	1250 3350 1250 3250
 Wire Wire Line
-	4500 2750 6650 2750
-Wire Wire Line
-	6300 2600 6300 2950
+	4500 2750 6300 2750
+Wire Wire Line
+	6300 2600 6300 2750
 Connection ~ 6300 2750
 $Comp
@@
 	6300 3250 6300 3350
 Wire Wire Line
-	1250 1100 1250 2300
+	1250 1100 1250 2150
 Connection ~ 7450 1100
 Connection ~ 1250 2150
@@
 	1    0    0    -1
 $EndComp
-Connection ~ 7450 1700
 $Comp
 L device:C C168
@@
 	1    0    0    -1
 $EndComp
-Connection ~ 7450 3250
-Wire Wire Line
-	7450 1700 10150 1700
+Wire Wire Line
+	7450 1700 7900 1700
 Wire Wire Line
 	7100 2150 7100 2650
 Wire Wire Line
-	7450 3250 10150 3250
+	7450 3250 7900 3250
 $Comp
 L device:C C171
@@
 Wire Wire Line
 	5250 5300 5500 5300
+Wire Wire Line
+	4400 5700 4400 5650
+Wire Wire Line
+	4700 5300 4700 5450
+Wire Wire Line
+	4700 5950 4700 6200
+Wire Wire Line
+	4000 5700 4400 5700
+Wire Wire Line
+	3450 6250 3450 6350
+Wire Wire Line
+	2600 4600 2600 5000
+Wire Wire Line
+	2600 5000 2600 5300
+Wire Wire Line
+	10150 2650 10150 2800
+Wire Wire Line
+	7900 2650 8350 2650
+Wire Wire Line
+	8350 2650 8800 2650
+Wire Wire Line
+	8800 2650 9250 2650
+Wire Wire Line
+	9250 2650 9700 2650
+Wire Wire Line
+	9700 2650 10150 2650
+Wire Wire Line
+	9700 3250 10150 3250
+Wire Wire Line
+	9250 3250 9700 3250
+Wire Wire Line
+	8800 3250 9250 3250
+Wire Wire Line
+	8350 3250 8800 3250
+Wire Wire Line
+	7900 3250 8350 3250
+Wire Wire Line
+	10150 3250 10150 3350
+Wire Wire Line
+	10150 1100 10150 1250
+Wire Wire Line
+	7900 1100 8350 1100
+Wire Wire Line
+	8350 1100 8800 1100
+Wire Wire Line
+	8800 1100 9250 1100
+Wire Wire Line
+	9250 1100 9700 1100
+Wire Wire Line
+	9700 1100 10150 1100
+Wire Wire Line
+	9700 1700 10150 1700
+Wire Wire Line
+	9250 1700 9700 1700
+Wire Wire Line
+	8800 1700 9250 1700
+Wire Wire Line
+	8350 1700 8800 1700
+Wire Wire Line
+	7900 1700 8350 1700
+Wire Wire Line
+	10150 1700 10150 1800
+Wire Wire Line
+	10050 4800 10050 4950
+Wire Wire Line
+	8700 4800 9150 4800
+Wire Wire Line
+	9150 4800 9600 4800
+Wire Wire Line
+	9600 4800 10050 4800
+Wire Wire Line
+	9600 5400 10050 5400
+Wire Wire Line
+	9150 5400 9600 5400
+Wire Wire Line
+	8700 5400 9150 5400
+Wire Wire Line
+	10050 5400 10050 5500
+Wire Wire Line
+	8050 4800 8250 4800
+Wire Wire Line
+	6450 4400 7100 4400
+Wire Wire Line
+	6450 4800 6500 4800
+Wire Wire Line
+	6450 4800 6450 5500
+Wire Wire Line
+	6200 5150 6200 5300
+Wire Wire Line
+	8250 4800 8700 4800
+Wire Wire Line
+	5100 2150 5350 2150
+Wire Wire Line
+	5800 2500 5800 2550
+Wire Wire Line
+	3800 1500 4600 1500
+Wire Wire Line
+	2400 2150 3000 2150
+Wire Wire Line
+	1700 2500 1700 2550
+Wire Wire Line
+	4600 1500 4800 1500
+Wire Wire Line
+	2900 1500 3800 1500
+Wire Wire Line
+	1250 2750 3000 2750
+Wire Wire Line
+	1250 2750 1250 2950
+Wire Wire Line
+	6300 2750 6650 2750
+Wire Wire Line
+	6300 2750 6300 2950
+Wire Wire Line
+	7450 1100 7900 1100
+Wire Wire Line
+	1250 2150 1700 2150
+Wire Wire Line
+	1250 2150 1250 2300
+Wire Wire Line
+	1700 2150 1900 2150
+Wire Wire Line
+	5800 2150 6300 2150
+Wire Wire Line
+	7450 2650 7900 2650
+Wire Wire Line
+	6300 2150 6650 2150
+Wire Wire Line
+	6650 2150 7100 2150
+NoConn ~ 4500 2600
+NoConn ~ 3000 2600
 $EndSCHEMATC
