File: HILTOP_motherboard/BoardPower.sch (KiCad schematic (older format))
At the start: 50 parts, among them Q3 2N7002, U24 MAX16054, U27 TPS54394, U28 LP2985

Commit message: DRC checks complete, all errors and warnings cleared. BOM created and parts rationalised.
Parts:
- C175: Devtank 105-004 -> 105-010
Changed lines of the file:
@@
 F 2 "Capacitor_SMD:C_0603_1608Metric" H 6238 4800 50  0001 C CNN
 F 3 "" H 6200 4950 50  0000 C CNN
-F 4 "105-004" H 6200 4950 60  0001 C CNN "Devtank"
+F 4 "105-010" H 6200 4950 60  0001 C CNN "Devtank"
 	1    6200 4950
 	1    0    0    -1

Commit message: Rev B
Parts:
- C175: Devtank 105-010 -> 105-014
Changed lines of the file:
@@
 F 2 "Capacitor_SMD:C_0603_1608Metric" H 6238 4800 50  0001 C CNN
 F 3 "" H 6200 4950 50  0000 C CNN
-F 4 "105-010" H 6200 4950 60  0001 C CNN "Devtank"
+F 4 "105-014" H 6200 4950 60  0001 C CNN "Devtank"
 	1    6200 4950
 	1    0    0    -1

Commit message: Rev C - pre-release
Parts:
- added R256: 10K, Resistor_SMD:R_0603_1608Metric, symbol HILTOP_Motherboard-rescue:R-device
- added U48: 74LVC1G3157, Package_SO:TSOP-6_1.65x3.05mm_P0.95mm, symbol Devtank:74LVC1G3157
- C110, C133, C134, C135, C136, C137, C138, C139, C140, C141, C142, C143, C144, C145, C146, C147, C148, C149, C150, C167, C168, C169, C170, C171, C172, C173, C174, C175, C176, C177, C178: symbol device:C -> HILTOP_Motherboard-rescue:C-device
- D18: symbol device:LED -> HILTOP_Motherboard-rescue:LED-device
- D24: symbol device:D_Schottky -> HILTOP_Motherboard-rescue:D_Schottky-device
- L10, L9: symbol device:L -> HILTOP_Motherboard-rescue:L-device
- Q3: symbol Transistor:2N7002 -> HILTOP_Motherboard-rescue:2N7002-Transistor
- R106, R107, R108, R109, R110, R111, R160, R161, R162, R163, R164: symbol device:R -> HILTOP_Motherboard-rescue:R-device
Connections:
- net labels added: PWR_SW_CPU
- wire segments 199 -> 209
Other:
- moved on the sheet: U24, U28

Commit message: changed silkscreen to revD and updated sheet information
Parts:
- U24: symbol Devtank:MAX16054 -> HILTOP_Motherboard-rescue:MAX16054-Devtank
- U27: symbol Devtank:TPS54394 -> HILTOP_Motherboard-rescue:TPS54394-Devtank
- U28: symbol Devtank:LP2985 -> HILTOP_Motherboard-rescue:LP2985-Devtank
- U48: symbol Devtank:74LVC1G3157 -> HILTOP_Motherboard-rescue:74LVC1G3157-Devtank
Changed lines of the file:
@@
 Sheet 12 12
 Title "HILTOP Motherboard"
-Date "2020-04-28"
-Rev "Rev C"
+Date "2021-02-17"
+Rev "Rev D"
 Comp "Devtank Ltd"
-Comment1 ""
+Comment1 "Part No: 304-001"
 Comment2 ""
 Comment3 ""
@@
 $EndComp
 $Comp
-L Devtank:+5V_STBY #PWR0297
+L HILTOP_Motherboard-rescue:+5V_STBY-Devtank #PWR0297
 U 1 1 58D213A1
 P 3100 4200
@@
 $EndComp
 $Comp
-L Devtank:+5V_STBY #PWR0304
+L HILTOP_Motherboard-rescue:+5V_STBY-Devtank #PWR0304
 U 1 1 58D22774
 P 5200 4500
@@
 Connection ~ 4500 5500
 $Comp
-L Devtank:MAX16054 U24
+L HILTOP_Motherboard-rescue:MAX16054-Devtank U24
 U 1 1 58D8CF7C
 P 3100 5650
@@
 	10750 4250 10450 4250
 $Comp
-L Devtank:LP2985 U28
+L HILTOP_Motherboard-rescue:LP2985-Devtank U28
 U 1 1 5916D0DB
 P 7650 5050
@@
 $EndComp
 $Comp
-L Devtank:TPS54394 U27
+L HILTOP_Motherboard-rescue:TPS54394-Devtank U27
 U 1 1 59171F2D
 P 3750 2450
@@
 $EndComp
 $Comp
-L Devtank:+5V_STBY #PWR074
+L HILTOP_Motherboard-rescue:+5V_STBY-Devtank #PWR074
 U 1 1 5EC078CC
 P 1800 5100
@@
 $EndComp
 $Comp
-L Devtank:74LVC1G3157 U48
+L HILTOP_Motherboard-rescue:74LVC1G3157-Devtank U48
 U 1 1 5EC02D31
 P 1800 5550
