File: HILTOP_motherboard/Ethernet.sch (KiCad schematic (older format))
At the start: 52 parts, among them U7 LAN7500, Y2 25MHz Crystal

Commit message: Furthe progress on Schematics, assigned all main footprints using latest libraries, removed unwanted tracking and parts from original PCB layout
Parts:
- C123, C124, C125, C126, C127, C128, C130, C131, C151, C152, C85, C86, C87, C88, C89, C90, C91, C92, C93, C94, C95: footprint Capacitors_SMD:C_0603 -> Capacitor_SMD:C_0603_1608Metric
- C132: footprint Capacitors_SMD:C_0603 -> Capacitor_SMD:C_0603_1608Metric_Pad0.84x1.00mm_HandSolder
- C52: footprint Capacitors_SMD:C_0603 -> Capacitor_SMD:C_0201_0603Metric
- D21, D22, D23: footprint LEDs:LED_0603 -> LED_SMD:LED_0603_1608Metric
- FB1, FB2, FB3, FB4, FB5, R126, R127, R128, R129, R130, R131, R134, R135, R136, R137, R138, R139, R144, R145, R146, R147, R55, R70, R71: footprint Resistors_SMD:R_0603 -> Resistor_SMD:R_0603_1608Metric
- U7: footprint KiCAD_PCB_Lib:QFN-56_8x8mm_Pitch0.5mm -> Devtank_PCB_Lib:QFN-56_8x8mm_Pitch0.5mm
- Y2: footprint Crystals:Crystal_SMD_SeikoEpson_FA238V-4pin_3.2x2.5mm -> Crystal:Crystal_SMD_SeikoEpson_FA238V-4Pin_3.2x2.5mm

Commit message: Schematics complete - 1st draft
Parts:
- added C236: 100nF, Capacitor_SMD:C_0603_1608Metric, symbol device:C
- added U45: 93AAxxA, Package_SO:SOIC-8_3.9x4.9mm_P1.27mm, symbol memory:93AAxxA
- C123, C124, C125, C126, C127, C128, C130, C131, C132, C151, C152, C52, C85, C86, C87, C88, C89, C90, C91, C92, C93, C94, C95: symbol C -> device:C
- D21, D22, D23: symbol LED -> device:LED
- FB1, FB2, FB3, FB4, FB5: symbol L -> device:L
- R126, R127, R128, R129, R130, R131, R134, R135, R136, R137, R138, R139, R144, R145, R146, R147, R55, R70, R71: symbol R -> device:R
- U7: symbol LAN7500 -> Devtank:LAN7500
- Y2: symbol Crystal_GND24 -> device:Crystal_GND24
Connections:
- net +2V5: now also C236.1, U45.8 (VCC)
- net GND: now also C236.2, U45.5 (GND)
- net EECLK: now reaches U7.26 (EECLK)
- net EECLK: now also U45.2 (SCLK)
- net EEDI: now reaches U7.27 (EEDI)
- net EEDI: now also U45.4 (DO)
- net EEDO: now reaches U7.28 (EEDO)
- net EEDO: now also U45.3 (DI)
- net EECS: now reaches U7.29 (EECS)
- net EECS: now also U45.1 (CS)

Commit message: BOM nearly complete!
Parts:
- D21, D22, D23: value Green_LED -> GRN; footprint LED_SMD:LED_0603_1608Metric -> LED_SMD:LED_0402_1005Metric; Devtank 110-002 -> 110-005
Connections:
- no-connect marks 0 -> 11
Changed lines of the file:
@@
 P 3950 4950
 F 0 "D23" H 3950 5050 50  0000 C CNN
-F 1 "Green_LED" H 3950 4850 50  0000 C CNN
-F 2 "LED_SMD:LED_0603_1608Metric" H 3950 4950 50  0001 C CNN
+F 1 "GRN" H 3950 4850 50  0000 C CNN
+F 2 "LED_SMD:LED_0402_1005Metric" H 3950 4950 50  0001 C CNN
 F 3 "" H 3950 4950 50  0000 C CNN
-F 4 "110-002" H 3950 4950 60  0001 C CNN "Devtank"
+F 4 "110-005" H 3950 4950 60  0001 C CNN "Devtank"
 	1    3950 4950
 	-1   0    0    1
@@
 P 3950 4650
 F 0 "D22" H 3950 4750 50  0000 C CNN
-F 1 "Green_LED" H 3950 4550 50  0000 C CNN
-F 2 "LED_SMD:LED_0603_1608Metric" H 3950 4650 50  0001 C CNN
+F 1 "GRN" H 3950 4550 50  0000 C CNN
+F 2 "LED_SMD:LED_0402_1005Metric" H 3950 4650 50  0001 C CNN
 F 3 "" H 3950 4650 50  0000 C CNN
-F 4 "110-002" H 3950 4650 60  0001 C CNN "Devtank"
+F 4 "110-005" H 3950 4650 60  0001 C CNN "Devtank"
 	1    3950 4650
 	-1   0    0    1
@@
 P 3950 4350
 F 0 "D21" H 3950 4450 50  0000 C CNN
-F 1 "Green_LED" H 3950 4250 50  0000 C CNN
-F 2 "LED_SMD:LED_0603_1608Metric" H 3950 4350 50  0001 C CNN
+F 1 "GRN" H 3950 4250 50  0000 C CNN
+F 2 "LED_SMD:LED_0402_1005Metric" H 3950 4350 50  0001 C CNN
 F 3 "" H 3950 4350 50  0000 C CNN
-F 4 "110-002" H 3950 4350 60  0001 C CNN "Devtank"
+F 4 "110-005" H 3950 4350 60  0001 C CNN "Devtank"
 	1    3950 4350
 	-1   0    0    1
@@
 Wire Wire Line
 	5350 6000 4450 6000
+NoConn ~ 3125 2650
+NoConn ~ 3125 2550
+NoConn ~ 5350 4100
+NoConn ~ 5350 4200
+NoConn ~ 5350 4300
+NoConn ~ 5350 4400
+NoConn ~ 5350 4500
+NoConn ~ 5350 4600
+NoConn ~ 5350 4700
+NoConn ~ 5350 6400
+NoConn ~ 5350 6950
 $EndSCHEMATC
