File: HILTOP_motherboard/Ethernet.sch (KiCad schematic (older format))
At the start: 54 parts, among them U45 93AAxxA, U7 LAN7500, Y2 25MHz Crystal

Commit message: DRC checks complete, all errors and warnings cleared. BOM created and parts rationalised.
Parts:
- C132: footprint Capacitor_SMD:C_0603_1608Metric_Pad0.84x1.00mm_HandSolder -> Capacitor_SMD:C_0402_1005Metric; Devtank 106-003 -> 106-010
- C151: footprint Capacitor_SMD:C_0603_1608Metric -> Capacitor_SMD:C_0402_1005Metric; Devtank 106-003 -> 106-010
- C52: footprint Capacitor_SMD:C_0201_0603Metric -> Capacitor_SMD:C_0402_1005Metric; Devtank 105-002 -> 105-019
- R134: Devtank 101-014 -> 101-044
Connections:
- wire segments 254 -> 264
Changed lines of the file:
@@
 F 0 "C52" H 3875 9000 50  0000 L CNN
 F 1 "100nF" H 3875 8800 50  0000 L CNN
-F 2 "Capacitor_SMD:C_0201_0603Metric" H 3888 8750 50  0001 C CNN
+F 2 "Capacitor_SMD:C_0402_1005Metric" H 3888 8750 50  0001 C CNN
 F 3 "" H 3850 8900 50  0000 C CNN
-F 4 "105-002" H 3850 8900 60  0001 C CNN "Devtank"
+F 4 "105-019" H 3850 8900 60  0001 C CNN "Devtank"
 	1    3850 8900
 	1    0    0    -1
@@
 L Devtank:+2V5_LAN_A #PWR0167
 U 1 1 590BD202
-P 10250 2850
-F 0 "#PWR0167" H 10250 2700 50  0001 C CNN
-F 1 "+2V5_LAN_A" H 10250 2990 50  0000 C CNN
-F 2 "" H 10250 2850 50  0000 C CNN
-F 3 "" H 10250 2850 50  0000 C CNN
-	1    10250 2850
+P 10250 2725
+F 0 "#PWR0167" H 10250 2575 50  0001 C CNN
+F 1 "+2V5_LAN_A" H 10250 2865 50  0000 C CNN
+F 2 "" H 10250 2725 50  0000 C CNN
+F 3 "" H 10250 2725 50  0000 C CNN
+	1    10250 2725
 	1    0    0    -1
 $EndComp
@@
 F 2 "Resistor_SMD:R_0603_1608Metric" V 9330 5850 50  0001 C CNN
 F 3 "" H 9400 5850 50  0000 C CNN
-F 4 "101-014" V 9400 5850 60  0001 C CNN "Devtank"
+F 4 "101-044" V 9400 5850 60  0001 C CNN "Devtank"
 	1    9400 5850
 	0    1    1    0
@@
 F 0 "C151" H 9175 7550 50  0000 L CNN
 F 1 "18pF" H 9175 7350 50  0000 L CNN
-F 2 "Capacitor_SMD:C_0603_1608Metric" H 9188 7300 50  0001 C CNN
+F 2 "Capacitor_SMD:C_0402_1005Metric" H 9188 7300 50  0001 C CNN
 F 3 "" H 9150 7450 50  0000 C CNN
-F 4 "106-003" H 9150 7450 60  0001 C CNN "Devtank"
+F 4 "106-010" H 9150 7450 60  0001 C CNN "Devtank"
 	1    9150 7450
 	1    0    0    -1
@@
 F 0 "C132" H 9875 7550 50  0000 L CNN
 F 1 "18pF" H 9875 7350 50  0000 L CNN
-F 2 "Capacitor_SMD:C_0603_1608Metric_Pad0.84x1.00mm_HandSolder" H 9888 7300 50  0001 C CNN
+F 2 "Capacitor_SMD:C_0402_1005Metric" H 9888 7300 50  0001 C CNN
 F 3 "" H 9850 7450 50  0000 C CNN
-F 4 "106-003" H 9850 7450 60  0001 C CNN "Devtank"
+F 4 "106-010" H 9850 7450 60  0001 C CNN "Devtank"
 	1    9850 7450
 	1    0    0    -1
@@
 Connection ~ 10250 3000
 Wire Wire Line
-	10250 2850 10250 3000
+	10250 2725 10250 2900
 Wire Wire Line
 	11150 3000 11150 3250
@@
 	8450 8600 8650 8600
 Wire Wire Line
-	8450 8300 8450 8600
+	8450 8300 8450 8375
 Wire Wire Line
 	7550 8600 7800 8600
@@
 	7050 8600 7250 8600
 Wire Wire Line
-	7050 8300 7050 8600
+	7050 8300 7050 8375
 Wire Wire Line
 	5950 8600 6200 8600
@@
 	6200 9300 6200 9050
 Wire Wire Line
-	6200 8300 6200 8600
+	6200 8300 6200 8425
 Wire Wire Line
 	5450 8600 5650 8600
@@
 	3850 9050 3850 9200
 Wire Wire Line
-	3850 8300 3850 8600
+	3850 8300 3850 8425
 Wire Wire Line
 	3600 8600 3850 8600
@@
 NoConn ~ 5350 6400
 NoConn ~ 5350 6950
+$Comp
+L power:PWR_FLAG #FLG0122
+U 1 1 5DE7D97F
+P 3975 8425
+F 0 "#FLG0122" H 3975 8500 50  0001 C CNN
+F 1 "PWR_FLAG" V 3975 8553 50  0000 L CNN
+F 2 "" H 3975 8425 50  0001 C CNN
+F 3 "" H 3975 8425 50  0001 C CNN
+	1    3975 8425
+	0    1    1    0
+$EndComp
+Wire Wire Line
+	3975 8425 3850 8425
+Connection ~ 3850 8425
+Wire Wire Line
+	3850 8425 3850 8600
+$Comp
+L power:PWR_FLAG #FLG0123
+U 1 1 5DEA3326
+P 7125 8375
+F 0 "#FLG0123" H 7125 8450 50  0001 C CNN
+F 1 "PWR_FLAG" V 7125 8503 50  0000 L CNN
+F 2 "" H 7125 8375 50  0001 C CNN
+F 3 "" H 7125 8375 50  0001 C CNN
+	1    7125 8375
+	0    1    1    0
+$EndComp
+$Comp
+L power:PWR_FLAG #FLG0124
+U 1 1 5DEA343F
+P 6300 8425
+F 0 "#FLG0124" H 6300 8500 50  0001 C CNN
+F 1 "PWR_FLAG" V 6300 8553 50  0000 L CNN
+F 2 "" H 6300 8425 50  0001 C CNN
+F 3 "" H 6300 8425 50  0001 C CNN
+	1    6300 8425
+	0    1    1    0
+$EndComp
+Wire Wire Line
+	6300 8425 6200 8425
+Connection ~ 6200 8425
+Wire Wire Line
+	6200 8425 6200 8600
+Wire Wire Line
+	7125 8375 7050 8375
+Connection ~ 7050 8375
+Wire Wire Line
+	7050 8375 7050 8600
+$Comp
+L power:PWR_FLAG #FLG0125
+U 1 1 5DEC9B4A
+P 8525 8375
+F 0 "#FLG0125" H 8525 8450 50  0001 C CNN
+F 1 "PWR_FLAG" V 8525 8503 50  0000 L CNN
+F 2 "" H 8525 8375 50  0001 C CNN
+F 3 "" H 8525 8375 50  0001 C CNN
+	1    8525 8375
+	0    1    1    0
+$EndComp
+Wire Wire Line
+	8525 8375 8450 8375
+Connection ~ 8450 8375
+Wire Wire Line
+	8450 8375 8450 8600
+$Comp
+L power:PWR_FLAG #FLG0126
+U 1 1 5DEFE1D5
+P 10100 2900
+F 0 "#FLG0126" H 10100 2975 50  0001 C CNN
+F 1 "PWR_FLAG" V 10100 3028 50  0000 L CNN
+F 2 "" H 10100 2900 50  0001 C CNN
+F 3 "" H 10100 2900 50  0001 C CNN
+	1    10100 2900
+	0    -1   -1   0
+$EndComp
+Wire Wire Line
+	10100 2900 10250 2900
+Connection ~ 10250 2900
+Wire Wire Line
+	10250 2900 10250 3000
 $EndSCHEMATC

Commit message: Rev C - pre-release
Parts:
- C123, C124, C125, C126, C127, C128, C130, C131, C132, C151, C152, C236, C52, C85, C86, C87, C88, C89, C90, C91, C92, C93, C94, C95: symbol device:C -> HILTOP_Motherboard-rescue:C-device
- D21, D22, D23: symbol device:LED -> HILTOP_Motherboard-rescue:LED-device
- FB1, FB2, FB3, FB4, FB5: symbol device:L -> HILTOP_Motherboard-rescue:L-device
- R126, R127, R128, R129, R130, R131, R134, R135, R136, R137, R138, R139, R144, R145, R146, R147, R55, R70, R71: symbol device:R -> HILTOP_Motherboard-rescue:R-device
- U45: symbol memory:93AAxxA -> HILTOP_Motherboard-rescue:93AAxxA-memory
- Y2: symbol device:Crystal_GND24 -> HILTOP_Motherboard-rescue:Crystal_GND24-device
Changed lines of the file:
@@
 $EndDescr
 $Comp
-L device:R R55
+L HILTOP_Motherboard-rescue:R-device R55
 U 1 1 58C6DA55
 P 9300 4100
@@
 $EndComp
 $Comp
-L device:L FB1
+L HILTOP_Motherboard-rescue:L-device FB1
 U 1 1 590A7475
 P 3450 8600
@@
 $EndComp
 $Comp
-L device:C C52
+L HILTOP_Motherboard-rescue:C-device C52
 U 1 1 590A7619
 P 3850 8900
@@
 TR1_N
 $Comp
-L device:R R135
+L HILTOP_Motherboard-rescue:R-device R135
 U 1 1 590BCB34
 P 10250 3400
@@
 $EndComp
 $Comp
-L device:C C131
+L HILTOP_Motherboard-rescue:C-device C131
 U 1 1 590BD929
 P 13000 3350
@@
 $EndComp
 $Comp
-L device:C C130
+L HILTOP_Motherboard-rescue:C-device C130
 U 1 1 590BEF54
 P 12650 6250
@@
 LEDY_K
 $Comp
-L device:LED D23
+L HILTOP_Motherboard-rescue:LED-device D23
 U 1 1 590C1A7E
 P 3950 4950
@@
 $EndComp
 $Comp
-L device:LED D22
+L HILTOP_Motherboard-rescue:LED-device D22
 U 1 1 590C1D5A
 P 3950 4650
@@
 $EndComp
 $Comp
-L device:LED D21
+L HILTOP_Motherboard-rescue:LED-device D21
 U 1 1 590C1DDE
 P 3950 4350
@@
 $EndComp
 $Comp
-L device:R R129
+L HILTOP_Motherboard-rescue:R-device R129
 U 1 1 590C22F5
 P 3400 4950
@@
 $EndComp
 $Comp
-L device:R R128
+L HILTOP_Motherboard-rescue:R-device R128
 U 1 1 590C26FF
 P 3400 4650
@@
 $EndComp
 $Comp
-L device:R R127
+L HILTOP_Motherboard-rescue:R-device R127
 U 1 1 590C2776
 P 3400 4350
@@
 $EndComp
 $Comp
-L device:R R136
+L HILTOP_Motherboard-rescue:R-device R136
 U 1 1 590C329E
 P 10300 5750
@@
 $EndComp
 $Comp
-L device:R R134
+L HILTOP_Motherboard-rescue:R-device R134
 U 1 1 590C3524
 P 9400 5850
@@
 $EndComp
 $Comp
-L device:R R131
+L HILTOP_Motherboard-rescue:R-device R131
 U 1 1 590C5133
 P 4400 6500
@@
 $EndComp
 $Comp
-L device:R R130
+L HILTOP_Motherboard-rescue:R-device R130
 U 1 1 590C6A25
 P 3750 5650
@@
 $EndComp
 $Comp
-L device:R R126
+L HILTOP_Motherboard-rescue:R-device R126
 U 1 1 590F1317
 P 3350 5900
@@
 ~RESET
 $Comp
-L device:Crystal_GND24 Y2
+L HILTOP_Motherboard-rescue:Crystal_GND24-device Y2
 U 1 1 5917EAD2
 P 9500 7200
@@
 $EndComp
 $Comp
-L device:C C151
+L HILTOP_Motherboard-rescue:C-device C151
 U 1 1 5917EEF0
 P 9150 7450
@@
 $EndComp
 $Comp
-L device:R R70
+L HILTOP_Motherboard-rescue:R-device R70
 U 1 1 5940C111
 P 4400 6800
@@
 $EndComp
 $Comp
-L device:R R71
+L HILTOP_Motherboard-rescue:R-device R71
 U 1 1 5940C1AB
 P 4900 7150
@@
 $EndComp
 $Comp
-L device:L FB2
+L HILTOP_Motherboard-rescue:L-device FB2
 U 1 1 5940C6F3
 P 5800 8600
@@
 $EndComp
 $Comp
-L device:L FB3
+L HILTOP_Motherboard-rescue:L-device FB3
 U 1 1 5940C796
 P 7400 8600
@@
 $EndComp
 $Comp
-L device:L FB4
+L HILTOP_Motherboard-rescue:L-device FB4
 U 1 1 5940C834
 P 8800 8600
@@
 $EndComp
 $Comp
-L device:L FB5
+L HILTOP_Motherboard-rescue:L-device FB5
 U 1 1 5940D00E
 P 13600 3000
@@
 $EndComp
 $Comp
-L device:R R137
+L HILTOP_Motherboard-rescue:R-device R137
 U 1 1 5940D65E
 P 10550 3400
@@
 $EndComp
 $Comp
-L device:R R138
+L HILTOP_Motherboard-rescue:R-device R138
 U 1 1 5940D6ED
 P 10850 3400
@@
 $EndComp
 $Comp
-L device:R R139
+L HILTOP_Motherboard-rescue:R-device R139
 U 1 1 5940D77B
 P 11150 3400
@@
 $EndComp
 $Comp
-L device:C C123
+L HILTOP_Motherboard-rescue:C-device C123
 U 1 1 5940E631
 P 4450 8900
@@
 $EndComp
 $Comp
-L device:C C124
+L HILTOP_Motherboard-rescue:C-device C124
 U 1 1 5940E6BC
 P 4750 8900
@@
 $EndComp
 $Comp
-L device:C C125
+L HILTOP_Motherboard-rescue:C-device C125
 U 1 1 5940E748
 P 5050 8900
@@
 $EndComp
 $Comp
-L device:C C126
+L HILTOP_Motherboard-rescue:C-device C126
 U 1 1 5940E870
 P 6200 8900
@@
 $EndComp
 $Comp
-L device:C C127
+L HILTOP_Motherboard-rescue:C-device C127
 U 1 1 5940E939
 P 7050 8900
@@
 $EndComp
 $Comp
-L device:C C128
+L HILTOP_Motherboard-rescue:C-device C128
 U 1 1 5940EAD3
 P 8450 8900
@@
 $EndComp
 $Comp
-L device:C C152
+L HILTOP_Motherboard-rescue:C-device C152
 U 1 1 5940EE83
 P 13350 3350
@@
 $EndComp
 $Comp
-L device:C C132
+L HILTOP_Motherboard-rescue:C-device C132
 U 1 1 5940FDC6
 P 9850 7450
@@
 TR3_N
 $Comp
-L device:R R144
+L HILTOP_Motherboard-rescue:R-device R144
 U 1 1 59254E5D
 P 11450 3400
@@
 $EndComp
 $Comp
-L device:R R145
+L HILTOP_Motherboard-rescue:R-device R145
 U 1 1 59254F5C
 P 11750 3400
@@
 $EndComp
 $Comp
-L device:R R146
+L HILTOP_Motherboard-rescue:R-device R146
 U 1 1 59254FE8
 P 12050 3400
@@
 $EndComp
 $Comp
-L device:R R147
+L HILTOP_Motherboard-rescue:R-device R147
 U 1 1 59255081
 P 12350 3400
@@
 $EndComp
 $Comp
-L device:C C85
+L HILTOP_Motherboard-rescue:C-device C85
 U 1 1 593198EF
 P 4800 10200
@@
 $EndComp
 $Comp
-L device:C C86
+L HILTOP_Motherboard-rescue:C-device C86
 U 1 1 593199D8
 P 5150 10200
@@
 $EndComp
 $Comp
-L device:C C87
+L HILTOP_Motherboard-rescue:C-device C87
 U 1 1 59319A9A
 P 5500 10200
@@
 $EndComp
 $Comp
-L device:C C88
+L HILTOP_Motherboard-rescue:C-device C88
 U 1 1 59319BD0
 P 5850 10200
@@
 $EndComp
 $Comp
-L device:C C89
+L HILTOP_Motherboard-rescue:C-device C89
 U 1 1 59319CDA
 P 6200 10200
@@
 $EndComp
 $Comp
-L device:C C90
+L HILTOP_Motherboard-rescue:C-device C90
 U 1 1 59319D87
 P 6550 10200
@@
 $EndComp
 $Comp
-L device:C C91
+L HILTOP_Motherboard-rescue:C-device C91
 U 1 1 59319E33
 P 6900 10200
@@
 Connection ~ 8450 8600
 $Comp
-L device:C C92
+L HILTOP_Motherboard-rescue:C-device C92
 U 1 1 5931CF25
 P 1950 10200
@@
 $EndComp
 $Comp
-L device:C C93
+L HILTOP_Motherboard-rescue:C-device C93
 U 1 1 5931CF2C
 P 2300 10200
@@
 $EndComp
 $Comp
-L device:C C94
+L HILTOP_Motherboard-rescue:C-device C94
 U 1 1 5931CF33
 P 2650 10200
@@
 $EndComp
 $Comp
-L device:C C95
+L HILTOP_Motherboard-rescue:C-device C95
 U 1 1 5931CF3A
 P 3000 10200
@@
 	13350 3000 13450 3000
 $Comp
-L memory:93AAxxA U45
+L HILTOP_Motherboard-rescue:93AAxxA-memory U45
 U 1 1 5C611530
 P 2825 2550
@@
 $EndComp
 $Comp
-L device:C C236
+L HILTOP_Motherboard-rescue:C-device C236
 U 1 1 5C635038
 P 2075 2075

Commit message: changed silkscreen to revD and updated sheet information
Parts:
- U7: symbol Devtank:LAN7500 -> HILTOP_Motherboard-rescue:LAN7500-Devtank
Changed lines of the file:
@@
 Sheet 3 12
 Title "HILTOP Motherboard"
-Date "2020-04-28"
-Rev "Rev C"
+Date "2021-02-17"
+Rev "Rev D"
 Comp "Devtank Ltd"
-Comment1 ""
+Comment1 "Part No: 304-001"
 Comment2 ""
 Comment3 ""
@@
 LAN_USB_N
 $Comp
-L Devtank:LAN7500 U7
+L HILTOP_Motherboard-rescue:LAN7500-Devtank U7
 U 1 1 58C6D418
 P 7150 5250
@@
 $EndComp
 $Comp
-L Devtank:+1V2_LAN_A #PWR0156
+L HILTOP_Motherboard-rescue:+1V2_LAN_A-Devtank #PWR0156
 U 1 1 590A6232
 P 7400 2550
@@
 $EndComp
 $Comp
-L Devtank:+1V2_LAN_PLL #PWR0152
+L HILTOP_Motherboard-rescue:+1V2_LAN_PLL-Devtank #PWR0152
 U 1 1 590A6254
 P 7000 2550
@@
 $EndComp
 $Comp
-L Devtank:+1V2_USB_PLL #PWR0150
+L HILTOP_Motherboard-rescue:+1V2_USB_PLL-Devtank #PWR0150
 U 1 1 590A6276
 P 6700 2550
@@
 $EndComp
 $Comp
-L Devtank:+3V3_LAN_A #PWR0159
+L HILTOP_Motherboard-rescue:+3V3_LAN_A-Devtank #PWR0159
 U 1 1 590A6298
 P 8350 2550
@@
 $EndComp
 $Comp
-L Devtank:+1V2_USB_PLL #PWR0148
+L HILTOP_Motherboard-rescue:+1V2_USB_PLL-Devtank #PWR0148
 U 1 1 590A71EA
 P 6200 8300
@@
 $EndComp
 $Comp
-L Devtank:+1V2_LAN_PLL #PWR0153
+L HILTOP_Motherboard-rescue:+1V2_LAN_PLL-Devtank #PWR0153
 U 1 1 590A722D
 P 7050 8300
@@
 $EndComp
 $Comp
-L Devtank:+1V2_LAN_A #PWR0139
+L HILTOP_Motherboard-rescue:+1V2_LAN_A-Devtank #PWR0139
 U 1 1 590A72DD
 P 3850 8300
@@
 $EndComp
 $Comp
-L Devtank:+3V3_LAN_A #PWR0160
+L HILTOP_Motherboard-rescue:+3V3_LAN_A-Devtank #PWR0160
 U 1 1 590A734A
 P 8450 8300
@@
 $EndComp
 $Comp
-L Devtank:+2V5_LAN_A #PWR0167
+L HILTOP_Motherboard-rescue:+2V5_LAN_A-Devtank #PWR0167
 U 1 1 590BD202
 P 10250 2725
@@
 $EndComp
 $Comp
-L Devtank:+3V3_LAN_A #PWR0168
+L HILTOP_Motherboard-rescue:+3V3_LAN_A-Devtank #PWR0168
 U 1 1 590C3AC5
 P 10300 5550
