File: HILTOP_motherboard/BackPlane.sch (KiCad schematic (older format))
At the start: 10 parts

Commit message: Furthe progress on Schematics, assigned all main footprints using latest libraries, removed unwanted tracking and parts from original PCB layout
Parts:
- J23: renamed from J?; footprint TE_1-5145154-2 -> Devtank_PCB_Lib:TE_1-5145154-2_PCI_120
- gave numbers to parts that had none: 9
Changed lines of the file:
@@
 $EndDescr
 $Comp
-L 1-5145154-2 J?
+L 1-5145154-2 J23
 U 1 1 5AB59F67
 P 3800 5525
-F 0 "J?" H 3500 8659 50  0000 L BNN
+F 0 "J23" H 3500 8659 50  0000 L BNN
 F 1 "1-5145154-2" H 4000 2325 50  0000 L BNN
-F 2 "TE_1-5145154-2" H 3875 2325 50  0001 L BNN
+F 2 "Devtank_PCB_Lib:TE_1-5145154-2_PCI_120" H 3875 2325 50  0001 L BNN
 F 3 "" H 5225 5900 50  0001 L BNN
 	1    3800 5525
@@
 USB_BACKPLANE_N
 $Comp
-L GND #PWR?
+L GND #PWR0396
 U 1 1 5AB5CC98
 P 3100 8900
-F 0 "#PWR?" H 3100 8650 50  0001 C CNN
+F 0 "#PWR0396" H 3100 8650 50  0001 C CNN
 F 1 "GND" H 3100 8750 50  0000 C CNN
 F 2 "" H 3100 8900 50  0001 C CNN
@@
 $EndComp
 $Comp
-L GND #PWR?
+L GND #PWR0397
 U 1 1 5AB5CCB7
 P 5325 8875
-F 0 "#PWR?" H 5325 8625 50  0001 C CNN
+F 0 "#PWR0397" H 5325 8625 50  0001 C CNN
 F 1 "GND" H 5325 8725 50  0000 C CNN
 F 2 "" H 5325 8875 50  0001 C CNN
@@
 	5100 7025 5675 7025
 $Comp
-L ADJ_DC #PWR?
+L ADJ_DC #PWR0398
 U 1 1 5ABB1D84
 P 5700 8175
-F 0 "#PWR?" H 5700 8025 50  0001 C CNN
+F 0 "#PWR0398" H 5700 8025 50  0001 C CNN
 F 1 "ADJ_DC" H 5700 8315 50  0000 C CNN
 F 2 "" H 5700 8175 50  0000 C CNN
@@
 $EndComp
 $Comp
-L ADJ_DC #PWR?
+L ADJ_DC #PWR0399
 U 1 1 5ABB1D9E
 P 2800 8175
-F 0 "#PWR?" H 2800 8025 50  0001 C CNN
+F 0 "#PWR0399" H 2800 8025 50  0001 C CNN
 F 1 "ADJ_DC" H 2800 8315 50  0000 C CNN
 F 2 "" H 2800 8175 50  0000 C CNN
@@
 Connection ~ 5700 8425
 $Comp
-L +12V #PWR?
+L +12V #PWR0400
 U 1 1 5ABB2B24
 P 5975 7725
-F 0 "#PWR?" H 5975 7575 50  0001 C CNN
+F 0 "#PWR0400" H 5975 7575 50  0001 C CNN
 F 1 "+12V" H 5975 7865 50  0000 C CNN
 F 2 "" H 5975 7725 50  0001 C CNN
@@
 $EndComp
 $Comp
-L +12V #PWR?
+L +12V #PWR0401
 U 1 1 5ABB2B3A
 P 1575 7650
-F 0 "#PWR?" H 1575 7500 50  0001 C CNN
+F 0 "#PWR0401" H 1575 7500 50  0001 C CNN
 F 1 "+12V" H 1575 7790 50  0000 C CNN
 F 2 "" H 1575 7650 50  0001 C CNN
@@
 $EndComp
 $Comp
-L +3V3 #PWR?
+L +3V3 #PWR0402
 U 1 1 5ABB2B55
 P 6425 7150
-F 0 "#PWR?" H 6425 7000 50  0001 C CNN
+F 0 "#PWR0402" H 6425 7000 50  0001 C CNN
 F 1 "+3V3" H 6425 7290 50  0000 C CNN
 F 2 "" H 6425 7150 50  0001 C CNN
@@
 $EndComp
 $Comp
-L +5V #PWR?
+L +5V #PWR0403
 U 1 1 5ABB2B6B
 P 6725 7275
-F 0 "#PWR?" H 6725 7125 50  0001 C CNN
+F 0 "#PWR0403" H 6725 7125 50  0001 C CNN
 F 1 "+5V" H 6725 7415 50  0000 C CNN
 F 2 "" H 6725 7275 50  0001 C CNN
@@
 $EndComp
 $Comp
-L -5V #PWR?
+L -5V #PWR0404
 U 1 1 5ABB2B83
 P 2800 7150
-F 0 "#PWR?" H 2800 7000 50  0001 C CNN
+F 0 "#PWR0404" H 2800 7000 50  0001 C CNN
 F 1 "-5V" H 2800 7290 50  0000 C CNN
 F 2 "" H 2800 7150 50  0000 C CNN
@@
 $EndComp
 $Comp
-L +3V3 #PWR?
+L +3V3 #PWR0405
 U 1 1 5ABB2B9B
 P 2150 7150
-F 0 "#PWR?" H 2150 7000 50  0001 C CNN
+F 0 "#PWR0405" H 2150 7000 50  0001 C CNN
 F 1 "+3V3" H 2150 7290 50  0000 C CNN
 F 2 "" H 2150 7150 50  0001 C CNN
@@
 Connection ~ 3200 7325
 $Comp
-L +5V #PWR?
+L +5V #PWR0406
 U 1 1 5ABB2E25
 P 1850 7325
-F 0 "#PWR?" H 1850 7175 50  0001 C CNN
+F 0 "#PWR0406" H 1850 7175 50  0001 C CNN
 F 1 "+5V" H 1850 7465 50  0000 C CNN
 F 2 "" H 1850 7325 50  0001 C CNN
@@
 Connection ~ 5700 7925
 $Comp
-L ADJ_DC #PWR?
+L ADJ_DC #PWR0407
 U 1 1 5ABB53C5
 P 7050 8875
-F 0 "#PWR?" H 7050 8725 50  0001 C CNN
+F 0 "#PWR0407" H 7050 8725 50  0001 C CNN
 F 1 "ADJ_DC" H 7050 9015 50  0000 C CNN
 F 2 "" H 7050 8875 50  0000 C CNN
@@
 $EndComp
 $Comp
-L +3V3 #PWR?
+L +3V3 #PWR0408
 U 1 1 5ABB53E1
 P 975 9425
-F 0 "#PWR?" H 975 9275 50  0001 C CNN
+F 0 "#PWR0408" H 975 9275 50  0001 C CNN
 F 1 "+3V3" H 975 9565 50  0000 C CNN
 F 2 "" H 975 9425 50  0001 C CNN
@@
 $EndComp
 $Comp
-L +5V #PWR?
+L +5V #PWR0409
 U 1 1 5ABB5403
 P 1875 9450
-F 0 "#PWR?" H 1875 9300 50  0001 C CNN
+F 0 "#PWR0409" H 1875 9300 50  0001 C CNN
 F 1 "+5V" H 1875 9590 50  0000 C CNN
 F 2 "" H 1875 9450 50  0001 C CNN
@@
 $EndComp
 $Comp
-L +12V #PWR?
+L +12V #PWR0410
 U 1 1 5ABB5428
 P 6300 8875
-F 0 "#PWR?" H 6300 8725 50  0001 C CNN
+F 0 "#PWR0410" H 6300 8725 50  0001 C CNN
 F 1 "+12V" H 6300 9015 50  0000 C CNN
 F 2 "" H 6300 8875 50  0001 C CNN
@@
 $EndComp
 $Comp
-L C C?
+L C C229
 U 1 1 5ABB6904
 P 6300 9125
-F 0 "C?" H 6325 9225 50  0000 L CNN
+F 0 "C229" H 6325 9225 50  0000 L CNN
 F 1 "100nF" H 6325 9025 50  0000 L CNN
 F 2 "Capacitor_SMD:C_0603_1608Metric" H 6338 8975 50  0001 C CNN
@@
 $EndComp
 $Comp
-L C C?
+L C C230
 U 1 1 5ABB6A44
 P 6600 9125
-F 0 "C?" H 6625 9225 50  0000 L CNN
+F 0 "C230" H 6625 9225 50  0000 L CNN
 F 1 "100nF" H 6625 9025 50  0000 L CNN
 F 2 "Capacitor_SMD:C_0603_1608Metric" H 6638 8975 50  0001 C CNN
@@
 $EndComp
 $Comp
-L C C?
+L C C231
 U 1 1 5ABB6AE4
 P 7050 9125
-F 0 "C?" H 7075 9225 50  0000 L CNN
+F 0 "C231" H 7075 9225 50  0000 L CNN
 F 1 "100nF" H 7075 9025 50  0000 L CNN
 F 2 "Capacitor_SMD:C_0603_1608Metric" H 7088 8975 50  0001 C CNN
@@
 $EndComp
 $Comp
-L C C?
+L C C232
 U 1 1 5ABB6B20
 P 7350 9125
-F 0 "C?" H 7375 9225 50  0000 L CNN
+F 0 "C232" H 7375 9225 50  0000 L CNN
 F 1 "100nF" H 7375 9025 50  0000 L CNN
 F 2 "Capacitor_SMD:C_0603_1608Metric" H 7388 8975 50  0001 C CNN
@@
 $EndComp
 $Comp
-L C C?
+L C C228
 U 1 1 5ABB6C6E
 P 2450 10150
-F 0 "C?" H 2475 10250 50  0000 L CNN
+F 0 "C228" H 2475 10250 50  0000 L CNN
 F 1 "100nF" H 2475 10050 50  0000 L CNN
 F 2 "Capacitor_SMD:C_0603_1608Metric" H 2488 10000 50  0001 C CNN
@@
 $EndComp
 $Comp
-L C C?
+L C C226
 U 1 1 5ABB6CAD
 P 1875 9700
-F 0 "C?" H 1900 9800 50  0000 L CNN
+F 0 "C226" H 1900 9800 50  0000 L CNN
 F 1 "100nF" H 1900 9600 50  0000 L CNN
 F 2 "Capacitor_SMD:C_0603_1608Metric" H 1913 9550 50  0001 C CNN
@@
 $EndComp
 $Comp
-L C C?
+L C C227
 U 1 1 5ABB6D0F
 P 2175 9700
-F 0 "C?" H 2200 9800 50  0000 L CNN
+F 0 "C227" H 2200 9800 50  0000 L CNN
 F 1 "100nF" H 2200 9600 50  0000 L CNN
 F 2 "Capacitor_SMD:C_0603_1608Metric" H 2213 9550 50  0001 C CNN
@@
 $EndComp
 $Comp
-L C C?
+L C C225
 U 1 1 5ABB6D54
 P 1275 9700
-F 0 "C?" H 1300 9800 50  0000 L CNN
+F 0 "C225" H 1300 9800 50  0000 L CNN
 F 1 "100nF" H 1300 9600 50  0000 L CNN
 F 2 "Capacitor_SMD:C_0603_1608Metric" H 1313 9550 50  0001 C CNN
@@
 $EndComp
 $Comp
-L C C?
+L C C224
 U 1 1 5ABB6DB6
 P 975 9700
-F 0 "C?" H 1000 9800 50  0000 L CNN
+F 0 "C224" H 1000 9800 50  0000 L CNN
 F 1 "100nF" H 1000 9600 50  0000 L CNN
 F 2 "Capacitor_SMD:C_0603_1608Metric" H 1013 9550 50  0001 C CNN
@@
 $EndComp
 $Comp
-L -5V #PWR?
+L -5V #PWR0411
 U 1 1 5ABB70EC
 P 2450 10400
-F 0 "#PWR?" H 2450 10250 50  0001 C CNN
+F 0 "#PWR0411" H 2450 10250 50  0001 C CNN
 F 1 "-5V" H 2450 10540 50  0000 C CNN
 F 2 "" H 2450 10400 50  0000 C CNN
@@
 $EndComp
 $Comp
-L GND #PWR?
+L GND #PWR0412
 U 1 1 5ABB72D6
 P 975 9975
-F 0 "#PWR?" H 975 9725 50  0001 C CNN
+F 0 "#PWR0412" H 975 9725 50  0001 C CNN
 F 1 "GND" H 975 9825 50  0000 C CNN
 F 2 "" H 975 9975 50  0001 C CNN
@@
 $EndComp
 $Comp
-L GND #PWR?
+L GND #PWR0413
 U 1 1 5ABB7323
 P 1875 9975
-F 0 "#PWR?" H 1875 9725 50  0001 C CNN
+F 0 "#PWR0413" H 1875 9725 50  0001 C CNN
 F 1 "GND" H 1875 9825 50  0000 C CNN
 F 2 "" H 1875 9975 50  0001 C CNN
@@
 	2450 10300 2450 10400
 $Comp
-L GND #PWR?
+L GND #PWR0414
 U 1 1 5ABB7E85
 P 6300 9425
-F 0 "#PWR?" H 6300 9175 50  0001 C CNN
+F 0 "#PWR0414" H 6300 9175 50  0001 C CNN
 F 1 "GND" H 6300 9275 50  0000 C CNN
 F 2 "" H 6300 9425 50  0001 C CNN
@@
 $EndComp
 $Comp
-L GND #PWR?
+L GND #PWR0415
 U 1 1 5ABB7EF4
 P 7050 9425
-F 0 "#PWR?" H 7050 9175 50  0001 C CNN
+F 0 "#PWR0415" H 7050 9175 50  0001 C CNN
 F 1 "GND" H 7050 9275 50  0000 C CNN
 F 2 "" H 7050 9425 50  0001 C CNN

Commit message: Schematics complete - 1st draft
Parts:
- removed C224, C225, C226, C227, C228, C229, C230, C231, C232: 100nF, Capacitor_SMD:C_0603_1608Metric, symbol C
- removed J23: 1-5145154-2, Devtank_PCB_Lib:TE_1-5145154-2_PCI_120, symbol 1-5145154-2
- added J24: HILTOP_PCIE-64_CONN, Devtank_PCB_Lib:PCIE-064-02-X-D-TH, symbol Devtank:HILTOP_PCIE-64_CONN
Connections:
- net labels added: GPIO1, GPIO10, GPIO11_SPI1_CS2, GPIO2, GPIO3, GPIO4, GPIO5, GPIO6, GPIO7, GPIO8, GPIO9
- net labels removed: +12V, +3V3, +5V, -5V, ADJ_DC, CLK_LVDS_N, CLK_LVDS_P, DATA_MISO_1_LVDS_N, DATA_MISO_1_LVDS_P, DATA_MISO_2_LVDS_N, DATA_MISO_2_LVDS_P, DATA_MISO_3_LVDS_N, DATA_MISO_3_LVDS_P, DATA_MISO_4_LVDS_N, DATA_MISO_4_LVDS_P, DATA_MISO_5_LVDS_N, DATA_MISO_5_LVDS_P, DATA_MISO_6_LVDS_N, DATA_MISO_6_LVDS_P, DATA_MOSI_1_LVDS_N, DATA_MOSI_1_LVDS_P, DATA_MOSI_2_LVDS_N, DATA_MOSI_2_LVDS_P, DATA_MOSI_3_LVDS_N, DATA_MOSI_3_LVDS_P, DATA_MOSI_4_LVDS_N, DATA_MOSI_4_LVDS_P, DATA_MOSI_5_LVDS_N, DATA_MOSI_5_LVDS_P, DATA_MOSI_6_LVDS_N, DATA_MOSI_6_LVDS_P, FP_GPIO1, FP_GPIO10, FP_GPIO2, FP_GPIO3, FP_GPIO4, FP_GPIO5, FP_GPIO6, FP_GPIO7, FP_GPIO8, FP_GPIO9, PR_GPIO1, PR_GPIO10, PR_GPIO2, PR_GPIO3, PR_GPIO4, PR_GPIO5, PR_GPIO6, PR_GPIO7, PR_GPIO8, PR_GPIO9, SPI1_CS2
- wire segments 161 -> 72

Commit message: BOM nearly complete!
Connections:
- no-connect marks 0 -> 9
Changed lines of the file:
@@
 Wire Wire Line
 	2550 6275 3325 6275
+NoConn ~ 5225 4575
+NoConn ~ 5225 4675
+NoConn ~ 5225 4775
+NoConn ~ 5225 4875
+NoConn ~ 5225 6275
+NoConn ~ 5225 6375
+NoConn ~ 5225 6475
+NoConn ~ 3325 6375
+NoConn ~ 3325 6475
 $EndSCHEMATC
