File: HILTOP_motherboard/BackPlane.sch (KiCad schematic (older format))
At the start: 1 part, among them J24 HILTOP_PCIE-64_CONN

Commit message: changed silkscreen to revD and updated sheet information
Parts:
- J24: symbol Devtank:HILTOP_PCIE-64_CONN -> HILTOP_Motherboard-rescue:HILTOP_PCIE-64_CONN-Devtank
Changed lines of the file:
@@
 Sheet 8 12
 Title "HILTOP Motherboard"
-Date "2020-04-28"
-Rev "Rev C"
+Date "2021-02-17"
+Rev "Rev D"
 Comp "Devtank Ltd"
-Comment1 ""
+Comment1 "Part No: 304-001"
 Comment2 ""
 Comment3 ""
@@
 $EndComp
 $Comp
-L Devtank:HILTOP_PCIE-64_CONN J24
+L HILTOP_Motherboard-rescue:HILTOP_PCIE-64_CONN-Devtank J24
 U 1 1 5F3C0F7D
 P 4275 4825
