File: HILTOP_motherboard/USBHub.sch (KiCad schematic (older format))
At the start: 71 parts, among them U14 SP3003-02XJ, U2 MIC2026-1YM, U3 USB2517, U4 MIC2026-1YM, U5 SP3003-02XJ, U6 SP3003-02XJ, Y1 24MHz Crystal

Commit message: BOM nearly complete!
Parts:
- D11, D13, D15, D17, D28, D30: footprint LED_SMD:LED_0603_1608Metric -> LED_SMD:LED_0402_1005Metric; Devtank (none) -> 110-005
- D12, D14, D16, D27, D29, D31: footprint LED_SMD:LED_0603_1608Metric -> LED_SMD:LED_0402_1005Metric; Devtank (none) -> 110-007
- D2, D3, D4: footprint LED_SMD:LED_0603_1608Metric -> LED_SMD:LED_0402_1005Metric; Devtank (none) -> 110-004
- D25, D26: footprint LED_SMD:LED_0603_1608Metric -> LED_SMD:LED_0402_1005Metric
- R35, R36, R37, R38, R39, R40, R41, R42, R43, R44, R45, R46, R47, R48: footprint Resistor_SMD:R_0603_1608Metric -> Resistor_SMD:R_0402_1005Metric
- U14, U5, U6: Devtank (none) -> 153-004
- U2, U4: Devtank (none) -> 153-003
- U3: Devtank (none) -> 118-004
Connections:
- no-connect marks 0 -> 13

Commit message: nearly finished placing all parts!
Parts:
- D25: Devtank (none) -> 110-007
- D26: Devtank (none) -> 110-005
- R31, R32, R33: footprint Resistor_SMD:R_0603_1608Metric -> Resistor_SMD:R_0402_1005Metric
Changed lines of the file:
@@
 F 2 "LED_SMD:LED_0402_1005Metric" H 8675 8500 50  0001 C CNN
 F 3 "" H 8675 8500 50  0001 C CNN
+F 4 "110-007" H 8675 8500 50  0001 C CNN "Devtank"
 	1    8675 8500
 	1    0    0    -1
@@
 F 2 "LED_SMD:LED_0402_1005Metric" H 8675 8925 50  0001 C CNN
 F 3 "" H 8675 8925 50  0001 C CNN
+F 4 "110-005" H 8675 8925 50  0001 C CNN "Devtank"
 	1    8675 8925
 	1    0    0    -1
@@
 F 0 "R31" H 3425 8000 50  0000 C CNN
 F 1 "330R" H 3475 7900 50  0000 C CNN
-F 2 "Resistor_SMD:R_0603_1608Metric" V 3230 7950 50  0001 C CNN
+F 2 "Resistor_SMD:R_0402_1005Metric" V 3230 7950 50  0001 C CNN
 F 3 "" H 3300 7950 50  0000 C CNN
 F 4 "101-024" V 3300 7950 60  0001 C CNN "Devtank"
@@
 F 0 "R33" H 3750 8000 50  0000 C CNN
 F 1 "330R" H 3800 7900 50  0000 C CNN
-F 2 "Resistor_SMD:R_0603_1608Metric" V 3555 7950 50  0001 C CNN
+F 2 "Resistor_SMD:R_0402_1005Metric" V 3555 7950 50  0001 C CNN
 F 3 "" H 3625 7950 50  0000 C CNN
 F 4 "101-024" V 3625 7950 60  0001 C CNN "Devtank"
@@
 F 0 "R32" H 3625 9450 50  0000 C CNN
 F 1 "330R" H 3675 9350 50  0000 C CNN
-F 2 "Resistor_SMD:R_0603_1608Metric" V 3430 9400 50  0001 C CNN
+F 2 "Resistor_SMD:R_0402_1005Metric" V 3430 9400 50  0001 C CNN
 F 3 "" H 3500 9400 50  0000 C CNN
 F 4 "101-024" V 3500 9400 60  0001 C CNN "Devtank"

Commit message: All parts placed and backplane connector checked and locked
Parts:
- R30, R34, R49, R50, R51, R52, R53, R72, R78: footprint Resistor_SMD:R_0603_1608Metric -> Resistor_SMD:R_0402_1005Metric
Connections:
- net labels added: OCS3, PWR3_5V, USB3_EN
- net labels removed: OCS4, PWR4_5V, USB4_EN
- wire segments 296 -> 300
Other:
- moved on the sheet: U14
Changed lines of the file:
@@
 Sheet 2 12
 Title "HILTOP Motherboard"
-Date "26th January 2018"
+Date "2019-01-10"
 Rev "Issue 1"
 Comp "Devtank Ltd"
@@
 USB2_P
 Text HLabel 3750 8450 2    60   Output ~ 0
-PWR4_5V
+PWR3_5V
 Text HLabel 11300 7475 2    60   Output ~ 0
 USB2_N
 Text HLabel 3750 7025 2    60   Output ~ 0
 PWR2_5V
-Text HLabel 10150 7425 2    60   Output ~ 0
+Text HLabel 11700 7650 2    60   Output ~ 0
 USB3_P
-Text HLabel 10150 7525 2    60   Output ~ 0
+Text HLabel 11700 8525 2    60   Output ~ 0
 USB3_N
 Text HLabel 3750 6925 2    60   Output ~ 0
 PWR1_5V
-Text HLabel 11300 7650 2    60   Output ~ 0
+Text HLabel 10150 8025 2    60   Output ~ 0
 USB4_P
-Text HLabel 11300 8525 2    60   Output ~ 0
+Text HLabel 10150 8125 2    60   Output ~ 0
 USB4_N
 Text HLabel 10150 8625 2    60   Output ~ 0
@@
 F 0 "R34" H 4475 2425 50  0000 C CNN
 F 1 "10K" H 4475 2525 50  0000 C CNN
-F 2 "Resistor_SMD:R_0603_1608Metric" V 4255 2475 50  0001 C CNN
+F 2 "Resistor_SMD:R_0402_1005Metric" V 4255 2475 50  0001 C CNN
 F 3 "" H 4325 2475 50  0000 C CNN
 F 4 "101-010" H 4325 2475 60  0001 C CNN "Devtank"
@@
 F 0 "R49" H 8650 1450 50  0000 C CNN
 F 1 "10K" H 8650 1550 50  0000 C CNN
-F 2 "Resistor_SMD:R_0603_1608Metric" V 8430 1500 50  0001 C CNN
+F 2 "Resistor_SMD:R_0402_1005Metric" V 8430 1500 50  0001 C CNN
 F 3 "" H 8500 1500 50  0000 C CNN
 F 4 "101-010" H 8500 1500 60  0001 C CNN "Devtank"
@@
 F 0 "R50" H 8975 1450 50  0000 C CNN
 F 1 "10K" H 8975 1550 50  0000 C CNN
-F 2 "Resistor_SMD:R_0603_1608Metric" V 8755 1500 50  0001 C CNN
+F 2 "Resistor_SMD:R_0402_1005Metric" V 8755 1500 50  0001 C CNN
 F 3 "" H 8825 1500 50  0000 C CNN
 F 4 "101-010" H 8825 1500 60  0001 C CNN "Devtank"
@@
 F 0 "R52" H 9300 1450 50  0000 C CNN
 F 1 "DNF" H 9300 1550 50  0000 C CNN
-F 2 "Resistor_SMD:R_0603_1608Metric" V 9080 1500 50  0001 C CNN
+F 2 "Resistor_SMD:R_0402_1005Metric" V 9080 1500 50  0001 C CNN
 F 3 "" H 9150 1500 50  0000 C CNN
 	1    9150 1500
@@
 F 0 "R72" H 9625 1450 50  0000 C CNN
 F 1 "10K" H 9625 1550 50  0000 C CNN
-F 2 "Resistor_SMD:R_0603_1608Metric" V 9405 1500 50  0001 C CNN
+F 2 "Resistor_SMD:R_0402_1005Metric" V 9405 1500 50  0001 C CNN
 F 3 "" H 9475 1500 50  0000 C CNN
 F 4 "101-010" H 9475 1500 60  0001 C CNN "Devtank"
@@
 F 0 "R51" H 8975 2325 50  0000 C CNN
 F 1 "DNF" H 8975 2425 50  0000 C CNN
-F 2 "Resistor_SMD:R_0603_1608Metric" V 8755 2375 50  0001 C CNN
+F 2 "Resistor_SMD:R_0402_1005Metric" V 8755 2375 50  0001 C CNN
 F 3 "" H 8825 2375 50  0000 C CNN
 	1    8825 2375
@@
 F 0 "R53" H 9300 2325 50  0000 C CNN
 F 1 "10K" H 9300 2425 50  0000 C CNN
-F 2 "Resistor_SMD:R_0603_1608Metric" V 9080 2375 50  0001 C CNN
+F 2 "Resistor_SMD:R_0402_1005Metric" V 9080 2375 50  0001 C CNN
 F 3 "" H 9150 2375 50  0000 C CNN
 F 4 "101-010" H 9150 2375 60  0001 C CNN "Devtank"
@@
 F 0 "R78" H 9625 2325 50  0000 C CNN
 F 1 "DNF" H 9625 2425 50  0000 C CNN
-F 2 "Resistor_SMD:R_0603_1608Metric" V 9405 2375 50  0001 C CNN
+F 2 "Resistor_SMD:R_0402_1005Metric" V 9405 2375 50  0001 C CNN
 F 3 "" H 9475 2375 50  0000 C CNN
 	1    9475 2375
@@
 F 0 "R30" H 1500 8700 50  0000 C CNN
 F 1 "10K" H 1500 8800 50  0000 C CNN
-F 2 "Resistor_SMD:R_0603_1608Metric" V 1280 8750 50  0001 C CNN
+F 2 "Resistor_SMD:R_0402_1005Metric" V 1280 8750 50  0001 C CNN
 F 3 "" H 1350 8750 50  0000 C CNN
 F 4 "101-010" H 1350 8750 60  0001 C CNN "Devtank"
@@
 Text Label 8400 6425 2    60   ~ 0
 USB1_EN
-Text Label 8400 8225 2    60   ~ 0
-USB4_EN
+Text Label 8400 7625 2    60   ~ 0
+USB3_EN
 Text Label 4475 7025 0    60   ~ 0
 OCS2
 Text Notes 675  6225 0    60   ~ 0
 Over-current Monitoring on external ports only
-Text Label 4475 8225 0    60   ~ 0
-OCS4
+Text Label 4475 7625 0    60   ~ 0
+OCS3
 Text Label 1450 6925 0    60   ~ 0
 USB1_EN
@@
 USB2_EN
 Text Label 1450 8450 0    60   ~ 0
-USB4_EN
+USB3_EN
 Text Label 4225 7225 2    60   ~ 0
 OCS1
@@
 OCS2
 Text Label 3900 8750 2    60   ~ 0
-OCS4
+OCS3
 $Comp
 L device:R R35
@@
 $EndComp
 Wire Wire Line
-	10825 8025 7550 8025
-Wire Wire Line
-	7550 8125 10825 8125
-Wire Wire Line
 	7550 8625 10150 8625
 Wire Wire Line
@@
 Wire Wire Line
 	7550 9925 10150 9925
-Wire Wire Line
-	7550 7425 10150 7425
-Wire Wire Line
-	7550 7525 10150 7525
 Wire Wire Line
 	3300 2175 3300 2250
@@
 	8400 7025 7550 7025
 Wire Wire Line
-	8400 8225 7550 8225
+	8400 7625 7550 7625
 Wire Wire Line
 	5150 6425 4475 6425
@@
 	5150 7025 4475 7025
 Wire Wire Line
-	5150 8225 4475 8225
+	5150 7625 4475 7625
 Wire Wire Line
 	2100 6925 1450 6925
@@
 L Devtank:SP3003-02XJ U14
 U 1 1 5A948EB7
-P 11650 8100
-F 0 "U14" H 11250 7800 50  0000 C CNN
-F 1 "SP3003-02XJ" H 11450 8400 50  0000 C CNN
-F 2 "Devtank_PCB_Lib:SC70-5" H 11800 7600 50  0001 C CNN
-F 3 "DOCUMENTATION" H 11650 7700 50  0001 C CNN
-F 4 "153-004" H 11650 8100 50  0001 C CNN "Devtank"
-	1    11650 8100
+P 12050 8100
+F 0 "U14" H 11650 7800 50  0000 C CNN
+F 1 "SP3003-02XJ" H 11850 8400 50  0000 C CNN
+F 2 "Devtank_PCB_Lib:SC70-5" H 12200 7600 50  0001 C CNN
+F 3 "DOCUMENTATION" H 12050 7700 50  0001 C CNN
+F 4 "153-004" H 12050 8100 50  0001 C CNN "Devtank"
+	1    12050 8100
 	-1   0    0    -1
 $EndComp
@@
 L power:+5V #PWR0133
 U 1 1 5A948EBD
-P 12700 7950
-F 0 "#PWR0133" H 12700 7800 50  0001 C CNN
-F 1 "+5V" H 12700 8090 50  0000 C CNN
-F 2 "" H 12700 7950 50  0000 C CNN
-F 3 "" H 12700 7950 50  0000 C CNN
-	1    12700 7950
+P 13100 7950
+F 0 "#PWR0133" H 13100 7800 50  0001 C CNN
+F 1 "+5V" H 13100 8090 50  0000 C CNN
+F 2 "" H 13100 7950 50  0000 C CNN
+F 3 "" H 13100 7950 50  0000 C CNN
+	1    13100 7950
 	1    0    0    -1
 $EndComp
@@
 L power:GND #PWR0130
 U 1 1 5A948EC3
-P 12525 8400
-F 0 "#PWR0130" H 12525 8150 50  0001 C CNN
-F 1 "GND" H 12525 8250 50  0000 C CNN
-F 2 "" H 12525 8400 50  0000 C CNN
-F 3 "" H 12525 8400 50  0000 C CNN
-	1    12525 8400
-	1    0    0    -1
-$EndComp
-Wire Wire Line
-	11250 7950 10825 7950
-Wire Wire Line
-	10825 7650 10825 7950
-Wire Wire Line
-	10825 8125 10825 8250
-Wire Wire Line
-	10825 8250 11250 8250
-Wire Wire Line
-	11300 7650 10825 7650
-Connection ~ 10825 7950
-Wire Wire Line
-	10825 8525 11300 8525
-Connection ~ 10825 8250
-Wire Wire Line
-	12400 8250 12700 8250
-Wire Wire Line
-	12700 8250 12700 7950
-Wire Wire Line
-	12525 8400 12525 8100
-Wire Wire Line
-	12525 8100 12400 8100
+P 12925 8400
+F 0 "#PWR0130" H 12925 8150 50  0001 C CNN
+F 1 "GND" H 12925 8250 50  0000 C CNN
+F 2 "" H 12925 8400 50  0000 C CNN
+F 3 "" H 12925 8400 50  0000 C CNN
+	1    12925 8400
+	1    0    0    -1
+$EndComp
+Wire Wire Line
+	11650 7950 11225 7950
+Wire Wire Line
+	11225 7650 11225 7950
+Wire Wire Line
+	11225 8250 11650 8250
+Wire Wire Line
+	11700 7650 11225 7650
+Wire Wire Line
+	11225 8525 11700 8525
+Wire Wire Line
+	12800 8250 13100 8250
+Wire Wire Line
+	13100 8250 13100 7950
+Wire Wire Line
+	12925 8400 12925 8100
+Wire Wire Line
+	12925 8100 12800 8100
 Text Notes 11625 4850 0    60   ~ 0
 USB Signals to be tracked as 90R differential matched pairs
@@
 	10825 7200 10825 7475
 Wire Wire Line
-	10825 7950 10825 8025
-Wire Wire Line
-	10825 8250 10825 8525
+	11225 8250 11225 8525
 NoConn ~ 7550 8825
 NoConn ~ 7550 9425
 NoConn ~ 7550 10025
-NoConn ~ 5150 7625
 NoConn ~ 5150 8825
 NoConn ~ 5150 9425
 NoConn ~ 12400 5825
 NoConn ~ 12400 6900
-NoConn ~ 12400 7950
+NoConn ~ 12800 7950
 NoConn ~ 5150 10025
-NoConn ~ 7550 7625
 NoConn ~ 3250 8550
 NoConn ~ 3250 8850
+NoConn ~ 7550 8225
+NoConn ~ 5150 8225
+Wire Wire Line
+	7550 8125 10150 8125
+Wire Wire Line
+	7550 8025 10150 8025
+Wire Wire Line
+	10625 7425 10625 7650
+Wire Wire Line
+	10625 7650 11225 7650
+Wire Wire Line
+	7550 7425 10625 7425
+Connection ~ 11225 7650
+Wire Wire Line
+	10525 7525 10525 7775
+Wire Wire Line
+	10525 7775 11000 7775
+Wire Wire Line
+	11000 7775 11000 8525
+Wire Wire Line
+	11000 8525 11225 8525
+Wire Wire Line
+	7550 7525 10525 7525
+Connection ~ 11225 8525
 $EndSCHEMATC

Commit message: DRC checks complete, all errors and warnings cleared. BOM created and parts rationalised.
Parts:
- C28: Devtank 105-002 -> 105-019
- C29, C37, C42: footprint Capacitor_SMD:C_0201_0603Metric -> Capacitor_SMD:C_0603_1608Metric
- C30, C33: footprint Capacitor_SMD:C_0201_0603Metric -> Capacitor_SMD:C_0402_1005Metric; Devtank 106-003 -> 106-010
- C31, C32, C34, C35, C36, C38, C39, C40, C41: footprint Capacitor_SMD:C_0201_0603Metric -> Capacitor_SMD:C_0402_1005Metric; Devtank 105-002 -> 105-019
- R30, R34, R49, R50, R53, R72: Devtank 101-010 -> 101-501
- R31, R32, R33, R35, R36, R37, R38, R39, R40, R41, R42, R43, R44, R45, R46, R47, R48: Devtank 101-024 -> 101-504

Commit message: finished new tracking for RS485 signals and general house keeping
Parts:
- U3: symbol Devtank:USB2517 -> HILTOP_Motherboard-rescue:USB2517-Devtank
Changed lines of the file:
@@
 Sheet 2 12
 Title "HILTOP Motherboard"
-Date "2019-01-10"
-Rev "Issue 1"
+Date "2019-07-03"
+Rev "Rev B"
 Comp "Devtank Ltd"
 Comment1 ""
@@
 $EndComp
 $Comp
-L Devtank:USB2517 U3
+L HILTOP_Motherboard-rescue:USB2517-Devtank U3
 U 1 1 5A933E77
 P 6325 2875
+AR Path="/5A933E77" Ref="U3"  Part="1"
+AR Path="/589A1B39/5A933E77" Ref="U3"  Part="1"
 F 0 "U3" H 5500 450 50  0000 C CNN
 F 1 "USB2517" H 7050 450 50  0000 C CNN
@@
 $EndComp
 $Comp
-L Devtank:USB2517 U3
+L HILTOP_Motherboard-rescue:USB2517-Devtank U3
 U 2 1 5A934048
 P 6350 7975
+AR Path="/5A934048" Ref="U3"  Part="2"
+AR Path="/589A1B39/5A934048" Ref="U3"  Part="2"
 F 0 "U3" H 5525 5550 50  0000 C CNN
 F 1 "USB2517" H 7075 5550 50  0000 C CNN

Commit message: Rev B
Parts:
- C28: footprint Capacitor_SMD:C_0201_0603Metric -> Capacitor_SMD:C_0402_1005Metric
Changed lines of the file:
@@
 F 0 "C28" H 4400 4425 50  0000 L CNN
 F 1 "100nF" H 4400 4225 50  0000 L CNN
-F 2 "Capacitor_SMD:C_0201_0603Metric" H 4413 4175 50  0001 C CNN
+F 2 "Capacitor_SMD:C_0402_1005Metric" H 4413 4175 50  0001 C CNN
 F 3 "" H 4375 4325 50  0000 C CNN
 F 4 "105-019" H 4375 4325 60  0001 C CNN "Devtank"

Commit message: Rev C - pre-release
Parts:
- removed R30: 10K, Resistor_SMD:R_0402_1005Metric, symbol device:R
- added U47: SP3003-02XJ, Devtank_PCB_Lib:SC70-5, symbol Devtank:SP3003-02XJ
- C21, C23, C28, C29, C30, C31, C32, C33, C34, C35, C36, C37, C38, C39, C40, C41, C42: symbol device:C -> HILTOP_Motherboard-rescue:C-device
- D11, D12, D13, D14, D15, D16, D17, D2, D25, D26, D27, D28, D29, D3, D30, D31, D4: symbol device:LED -> HILTOP_Motherboard-rescue:LED-device
- R152, R20, R21, R27, R31, R32, R33, R34, R35, R36, R37, R38, R39, R40, R41, R42, R43, R44, R45, R46, R47, R48, R49, R50, R51, R52, R53, R72, R78: symbol device:R -> HILTOP_Motherboard-rescue:R-device
- Y1: footprint Crystal:Crystal_SMD_7050-2Pin_7.0x5.0mm -> Crystal:Crystal_SMD_5032-2Pin_5.0x3.2mm; symbol device:Crystal -> HILTOP_Motherboard-rescue:Crystal-device
Connections:
- net +5V: now also U47.3 (VCC)
- net GND: now also U47.2 (GND)
- net USB6_N: now also U47.4 (IO2)
- net USB6_P: now also U47.5 (IO1)
- net OCS6: now reaches U3.38 (~OSC6)
- net OCS6: now also U4.3 (FLAGB)
- net USB6_EN: now reaches U3.39 (PRTPWR6)
- net USB6_EN: now also U4.4 (ENB)
- net PWR6_5V: now reaches U4.5 (OUTB)
- no-connect marks 13 -> 10
