File: HILTOP_motherboard/USBHub.sch (KiCad schematic (older format))
At the start: 71 parts, among them U14 SP3003-02XJ, U2 MIC2026-1YM, U3 USB2517, U4 MIC2026-1YM, U47 SP3003-02XJ, U5 SP3003-02XJ, U6 SP3003-02XJ, Y1 24MHz Crystal

Commit message: updates to include - license, remove U46, swap crystal Y1
Parts:
- Y1: footprint Crystal:Crystal_SMD_5032-2Pin_5.0x3.2mm -> Crystal:Crystal_SMD_3225-4Pin_3.2x2.5mm; symbol HILTOP_Motherboard-rescue:Crystal-device -> Device:Crystal_GND24
Connections:
- net GND: now also Y1.2, Y1.4
- net at C33.1, R21.1, U3.60 (XTAL2): now also Y1.3; no longer Y1.2
Other:
- moved on the sheet: R21
Changed lines of the file:
@@
 $EndComp
 $Comp
-L HILTOP_Motherboard-rescue:Crystal-device Y1
+L Device:Crystal_GND24 Y1
 U 1 1 58CDD1CB
 P 4575 3475
-F 0 "Y1" H 4575 3625 50  0000 C CNN
-F 1 "24MHz Crystal" H 4625 3325 50  0000 C CNN
-F 2 "Crystal:Crystal_SMD_5032-2Pin_5.0x3.2mm" H 4575 3475 50  0001 C CNN
+F 0 "Y1" V 4725 3600 50  0000 C CNN
+F 1 "24MHz Crystal" V 4375 3500 50  0000 C CNN
+F 2 "Crystal:Crystal_SMD_3225-4Pin_3.2x2.5mm" H 4575 3475 50  0001 C CNN
 F 3 "" H 4575 3475 50  0000 C CNN
 F 4 "181-003" H 4575 3475 60  0001 C CNN "Devtank"
@@
 L HILTOP_Motherboard-rescue:R-device R21
 U 1 1 58CDFBA7
-P 4875 3500
-F 0 "R21" V 4775 3400 50  0000 C CNN
-F 1 "1M" V 4775 3600 50  0000 C CNN
-F 2 "Resistor_SMD:R_0603_1608Metric" V 4805 3500 50  0001 C CNN
-F 3 "" H 4875 3500 50  0000 C CNN
-F 4 "101-019" V 4875 3500 60  0001 C CNN "Devtank"
-	1    4875 3500
+P 5075 3500
+F 0 "R21" V 4975 3400 50  0000 C CNN
+F 1 "1M" V 4975 3600 50  0000 C CNN
+F 2 "Resistor_SMD:R_0603_1608Metric" V 5005 3500 50  0001 C CNN
+F 3 "" H 5075 3500 50  0000 C CNN
+F 4 "101-019" V 5075 3500 60  0001 C CNN "Devtank"
+	1    5075 3500
 	-1   0    0    1
 $EndComp
@@
 Connection ~ 4575 3775
 Wire Wire Line
-	4875 3350 4875 3225
-Connection ~ 4875 3225
-Wire Wire Line
-	4875 3650 4875 3775
-Connection ~ 4875 3775
+	5075 3350 5075 3225
+Wire Wire Line
+	5075 3650 5075 3775
 Wire Wire Line
 	3950 3225 3675 3225
@@
 	3300 2250 3300 2325
 Wire Wire Line
-	4575 3225 4875 3225
-Wire Wire Line
-	4575 3775 4875 3775
-Wire Wire Line
-	4875 3225 5125 3225
-Wire Wire Line
-	4875 3775 5125 3775
-Wire Wire Line
 	3675 3775 3675 4050
 Wire Wire Line
@@
 Wire Wire Line
 	3250 8850 4225 8850
+Connection ~ 5075 3225
+Wire Wire Line
+	5075 3225 5125 3225
+Connection ~ 5075 3775
+Wire Wire Line
+	5075 3775 5125 3775
+Wire Wire Line
+	4575 3225 5075 3225
+Wire Wire Line
+	4575 3775 5075 3775
+$Comp
+L power:GND #PWR0471
+U 1 1 6071BBD6
+P 4875 3525
+F 0 "#PWR0471" H 4875 3275 50  0001 C CNN
+F 1 "GND" H 4875 3375 50  0000 C CNN
+F 2 "" H 4875 3525 50  0000 C CNN
+F 3 "" H 4875 3525 50  0000 C CNN
+	1    4875 3525
+	1    0    0    -1
+$EndComp
+$Comp
+L power:GND #PWR0472
+U 1 1 6071C35E
+P 4250 3500
+F 0 "#PWR0472" H 4250 3250 50  0001 C CNN
+F 1 "GND" H 4250 3350 50  0000 C CNN
+F 2 "" H 4250 3500 50  0000 C CNN
+F 3 "" H 4250 3500 50  0000 C CNN
+	1    4250 3500
+	1    0    0    -1
+$EndComp
+Wire Wire Line
+	4250 3500 4250 3475
+Wire Wire Line
+	4250 3475 4375 3475
+Wire Wire Line
+	4775 3475 4875 3475
+Wire Wire Line
+	4875 3475 4875 3525
 $EndSCHEMATC

Commit message: changed silkscreen to revD and updated sheet information
Parts:
- U14, U47, U5, U6: symbol Devtank:SP3003-02XJ -> HILTOP_Motherboard-rescue:SP3003-02XJ-Devtank
- U2, U4: symbol Devtank:MIC2026-1YM -> HILTOP_Motherboard-rescue:MIC2026-1YM-Devtank
- Y1: symbol Device:Crystal_GND24 -> HILTOP_Motherboard-rescue:Crystal_GND24-Device
Changed lines of the file:
@@
 Sheet 2 12
 Title "HILTOP Motherboard"
-Date "2020-04-28"
-Rev "Rev C"
+Date "2021-02-17"
+Rev "Rev D"
 Comp "Devtank Ltd"
-Comment1 ""
+Comment1 "Part No: 304-001"
 Comment2 ""
 Comment3 ""
@@
 $EndComp
 $Comp
-L Device:Crystal_GND24 Y1
+L HILTOP_Motherboard-rescue:Crystal_GND24-Device Y1
 U 1 1 58CDD1CB
 P 4575 3475
@@
 Default Config - 101\nInternal Defaults\nDynamic Power (local)\nUSB LED Mode
 $Comp
-L Devtank:MIC2026-1YM U2
+L HILTOP_Motherboard-rescue:MIC2026-1YM-Devtank U2
 U 1 1 5A95A96A
 P 2700 7175
@@
 $EndComp
 $Comp
-L Devtank:MIC2026-1YM U4
+L HILTOP_Motherboard-rescue:MIC2026-1YM-Devtank U4
 U 1 1 5A97EF81
 P 2700 8700
@@
 $EndComp
 $Comp
-L Devtank:SP3003-02XJ U5
+L HILTOP_Motherboard-rescue:SP3003-02XJ-Devtank U5
 U 1 1 5A940AEC
 P 11650 5975
@@
 	12525 5975 12400 5975
 $Comp
-L Devtank:SP3003-02XJ U6
+L HILTOP_Motherboard-rescue:SP3003-02XJ-Devtank U6
 U 1 1 5A94659D
 P 11650 7050
@@
 	10175 5925 10825 5925
 $Comp
-L Devtank:SP3003-02XJ U14
+L HILTOP_Motherboard-rescue:SP3003-02XJ-Devtank U14
 U 1 1 5A948EB7
 P 12050 8100
@@
 Connection ~ 11225 8525
 $Comp
-L Devtank:SP3003-02XJ U47
+L HILTOP_Motherboard-rescue:SP3003-02XJ-Devtank U47
 U 1 1 5F90CFEF
 P 11325 9375
