File: HILTOP_motherboard/USB_Debug.sch (KiCad schematic (older format))
At the start: 0 parts

Commit message: Schematics complete - 1st draft
Parts:
- added C217, C224: 4.7uF, Capacitor_SMD:C_0805_2012Metric, symbol device:C
- added C219, C225: 100nF, Capacitor_SMD:C_0603_1608Metric, symbol device:C
- added D32, D33: GRN, LED_SMD:LED_0603_1608Metric, symbol device:LED
- added R201, R203, R208, R209: 0R, Resistor_SMD:R_0603_1608Metric, symbol device:R
- added R202: DNF, Resistor_SMD:R_0603_1608Metric, symbol device:R
- added R204, R205: 330R, Resistor_SMD:R_0603_1608Metric, symbol device:R
- added U40: SP3003-02XJ, Devtank_PCB_Lib:SC70-5, symbol Devtank:SP3003-02XJ
- added U41: CP2102N-A01-GQFN24, Package_DFN_QFN:QFN-24-1EP_4x4mm_P0.5mm_EP2.6x2.6mm_ThermalVias, symbol silabs:CP2102N-A01-GQFN24
Connections:
- net RS232_RX: now also R209.1
- net RS232_TX: now also R208.1
- net USB_N: now also U40.4 (IO2), U41.4 (D-)
- net USB_P: now also U40.5 (IO1), U41.3 (D+)
- new net: R204.2, U41.13 (GPIO.1)
- new net: R205.2, U41.14 (GPIO.0)
- new net: R208.2, U41.20 (RXD)
- new net: R209.2, U41.21 (TXD)
- new net: R203.1, U41.8 (VBUS)
- new net: R201.1, R202.1, U41.9 (~RSTb)
- new net: D32.1 (K), R204.1
- new net: D33.1 (K), R205.1
- new net +3V3: C217.1, C219.1, C224.1, C225.1, D32.2 (A), D33.2 (A), R202.2, U41.5 (VIO), U41.6 (VDD), U41.7 (REGIN)
- new net +5V: U40.3 (VCC)
- new net GND: C217.2, C219.2, C224.2, C225.2, U40.2 (GND), U41.2 (GND), U41.25 (GND)
- new net USB_BUS_PWR: R203.2
- new net USB_~RESET: R201.2
Other:
- note added: "RXT"
- note added: "TXT"

Commit message: BOM nearly complete!
Parts:
- D32, D33: footprint LED_SMD:LED_0603_1608Metric -> LED_SMD:LED_0402_1005Metric
- U40: Devtank (none) -> 153-004
- U41: Devtank (none) -> 118-007
Connections:
- no-connect marks 0 -> 11
Changed lines of the file:
@@
 $Descr A4 11693 8268
 encoding utf-8
-Sheet 11 12
+Sheet 10 12
 Title ""
 Date ""
@@
 F 2 "Package_DFN_QFN:QFN-24-1EP_4x4mm_P0.5mm_EP2.6x2.6mm_ThermalVias" H 5975 2675 50  0001 L CNN
 F 3 "http://www.silabs.com/support%20documents/technicaldocs/cp2102n-datasheet.pdf" H 5575 2425 50  0001 C CNN
+F 4 "118-007" H 5525 3475 50  0001 C CNN "Devtank"
 	1    5525 3475
 	1    0    0    -1
@@
 F 2 "Devtank_PCB_Lib:SC70-5" H 4150 4275 50  0001 C CNN
 F 3 "DOCUMENTATION" H 4000 4375 50  0001 C CNN
+F 4 "153-004" H 4000 4775 50  0001 C CNN "Devtank"
 	1    4000 4775
 	-1   0    0    -1
@@
 F 0 "D32" H 7150 3900 50  0000 C CNN
 F 1 "GRN" H 7575 3900 50  0000 C CNN
-F 2 "LED_SMD:LED_0603_1608Metric" H 7350 3850 50  0001 C CNN
+F 2 "LED_SMD:LED_0402_1005Metric" H 7350 3850 50  0001 C CNN
 F 3 "" H 7350 3850 50  0001 C CNN
 	1    7350 3850
@@
 F 0 "D33" H 7150 4125 50  0000 C CNN
 F 1 "GRN" H 7575 4125 50  0000 C CNN
-F 2 "LED_SMD:LED_0603_1608Metric" H 7350 4075 50  0001 C CNN
+F 2 "LED_SMD:LED_0402_1005Metric" H 7350 4075 50  0001 C CNN
 F 3 "" H 7350 4075 50  0001 C CNN
 	1    7350 4075
@@
 	7875 4075 7875 3850
 Connection ~ 7875 3850
+NoConn ~ 4925 3175
+NoConn ~ 4925 3275
+NoConn ~ 6125 2875
+NoConn ~ 6125 2975
+NoConn ~ 6125 3075
+NoConn ~ 6125 3375
+NoConn ~ 6125 3475
+NoConn ~ 6125 3575
+NoConn ~ 6125 3775
+NoConn ~ 6125 3875
+NoConn ~ 4750 4625
 $EndSCHEMATC

Commit message: nearly finished placing all parts!
Parts:
- D32, D33: Devtank (none) -> 110-005
Changed lines of the file:
@@
 F 2 "LED_SMD:LED_0402_1005Metric" H 7350 3850 50  0001 C CNN
 F 3 "" H 7350 3850 50  0001 C CNN
+F 4 "110-005" H 7350 3850 50  0001 C CNN "Devtank"
 	1    7350 3850
 	1    0    0    -1
@@
 F 2 "LED_SMD:LED_0402_1005Metric" H 7350 4075 50  0001 C CNN
 F 3 "" H 7350 4075 50  0001 C CNN
+F 4 "110-005" H 7350 4075 50  0001 C CNN "Devtank"
 	1    7350 4075
 	1    0    0    -1

Commit message: Rev B
Parts:
- added R251: 47K, Resistor_SMD:R_0603_1608Metric, symbol device:R
- R203: value 0R -> 24K
Connections:
- net GND: now also R251.1
- net at R203.1, U41.8 (VBUS): now also R251.2
Other:
- moved on the sheet: U40
Changed lines of the file:
@@
 Wire Wire Line
 	5525 4525 5525 4375
-$Comp
-L Devtank:SP3003-02XJ U?
-U 1 1 5C3985E5
-P 4000 4775
-AR Path="/589A1B39/5C3985E5" Ref="U?"  Part="1"
-AR Path="/5AFBC859/5C3985E5" Ref="U40"  Part="1"
-F 0 "U40" H 3600 4475 50  0000 C CNN
-F 1 "SP3003-02XJ" H 3800 5075 50  0000 C CNN
-F 2 "Devtank_PCB_Lib:SC70-5" H 4150 4275 50  0001 C CNN
-F 3 "DOCUMENTATION" H 4000 4375 50  0001 C CNN
-F 4 "153-004" H 4000 4775 50  0001 C CNN "Devtank"
-	1    4000 4775
-	-1   0    0    -1
-$EndComp
-$Comp
-L power:+5V #PWR?
-U 1 1 5C3985EC
-P 5050 4625
-AR Path="/589A1B39/5C3985EC" Ref="#PWR?"  Part="1"
-AR Path="/5AFBC859/5C3985EC" Ref="#PWR0222"  Part="1"
-F 0 "#PWR0222" H 5050 4475 50  0001 C CNN
-F 1 "+5V" H 5050 4765 50  0000 C CNN
-F 2 "" H 5050 4625 50  0000 C CNN
-F 3 "" H 5050 4625 50  0000 C CNN
-	1    5050 4625
-	1    0    0    -1
-$EndComp
-$Comp
-L power:GND #PWR?
-U 1 1 5C3985F2
-P 4875 5075
-AR Path="/589A1B39/5C3985F2" Ref="#PWR?"  Part="1"
-AR Path="/5AFBC859/5C3985F2" Ref="#PWR0221"  Part="1"
-F 0 "#PWR0221" H 4875 4825 50  0001 C CNN
-F 1 "GND" H 4875 4925 50  0000 C CNN
-F 2 "" H 4875 5075 50  0000 C CNN
-F 3 "" H 4875 5075 50  0000 C CNN
-	1    4875 5075
-	1    0    0    -1
-$EndComp
-Wire Wire Line
-	4750 4925 5050 4925
-Wire Wire Line
-	5050 4925 5050 4625
-Wire Wire Line
-	4875 5075 4875 4775
-Wire Wire Line
-	4875 4775 4750 4775
 Wire Wire Line
 	3025 3875 3325 3875
 Wire Wire Line
 	3025 3975 3250 3975
-Wire Wire Line
-	3600 4625 3325 4625
-Wire Wire Line
-	3325 4625 3325 3875
 Connection ~ 3325 3875
 Wire Wire Line
 	3325 3875 4925 3875
-Wire Wire Line
-	3600 4925 3250 4925
-Wire Wire Line
-	3250 4925 3250 3975
 Connection ~ 3250 3975
 Wire Wire Line
@@
 P 4050 3775
 F 0 "R203" V 3950 3675 50  0000 C CNN
-F 1 "0R" V 3950 3850 50  0000 C CNN
+F 1 "24K" V 3950 3900 50  0000 C CNN
 F 2 "Resistor_SMD:R_0603_1608Metric" V 3980 3775 50  0001 C CNN
 F 3 "" H 4050 3775 50  0001 C CNN
@@
 $EndComp
 Wire Wire Line
-	4925 3775 4200 3775
+	4925 3775 4650 3775
 Text HLabel 3025 3600 0    60   Input ~ 0
 USB_BUS_PWR
@@
 NoConn ~ 6125 3775
 NoConn ~ 6125 3875
-NoConn ~ 4750 4625
+$Comp
+L device:R R251
+U 1 1 5D3E6FB7
+P 4650 4175
+F 0 "R251" H 4475 4125 50  0000 C CNN
+F 1 "47K" H 4500 4225 50  0000 C CNN
+F 2 "Resistor_SMD:R_0603_1608Metric" V 4580 4175 50  0001 C CNN
+F 3 "" H 4650 4175 50  0001 C CNN
+F 4 "101-016" H 4650 4175 50  0001 C CNN "Devtank"
+	1    4650 4175
+	-1   0    0    1
+$EndComp
+Wire Wire Line
+	4650 4325 4650 4375
+Wire Wire Line
+	4650 4025 4650 3775
+Connection ~ 4650 3775
+Wire Wire Line
+	4650 3775 4200 3775
+$Comp
+L power:GND #PWR?
+U 1 1 5D3EEA95
+P 4650 4375
+AR Path="/589A1B39/5D3EEA95" Ref="#PWR?"  Part="1"
+AR Path="/5AFBC859/5D3EEA95" Ref="#PWR051"  Part="1"
+F 0 "#PWR051" H 4650 4125 50  0001 C CNN
+F 1 "GND" H 4650 4225 50  0000 C CNN
+F 2 "" H 4650 4375 50  0000 C CNN
+F 3 "" H 4650 4375 50  0000 C CNN
+	1    4650 4375
+	1    0    0    -1
+$EndComp
+NoConn ~ 4750 4750
+Wire Wire Line
+	3600 5050 3250 5050
+Wire Wire Line
+	3600 4750 3325 4750
+Wire Wire Line
+	4875 4900 4750 4900
+Wire Wire Line
+	4875 5200 4875 4900
+Wire Wire Line
+	5050 5050 5050 4750
+Wire Wire Line
+	4750 5050 5050 5050
+$Comp
+L power:GND #PWR?
+U 1 1 5C3985F2
+P 4875 5200
+AR Path="/589A1B39/5C3985F2" Ref="#PWR?"  Part="1"
+AR Path="/5AFBC859/5C3985F2" Ref="#PWR0221"  Part="1"
+F 0 "#PWR0221" H 4875 4950 50  0001 C CNN
+F 1 "GND" H 4875 5050 50  0000 C CNN
+F 2 "" H 4875 5200 50  0000 C CNN
+F 3 "" H 4875 5200 50  0000 C CNN
+	1    4875 5200
+	1    0    0    -1
+$EndComp
+$Comp
+L power:+5V #PWR?
+U 1 1 5C3985EC
+P 5050 4750
+AR Path="/589A1B39/5C3985EC" Ref="#PWR?"  Part="1"
+AR Path="/5AFBC859/5C3985EC" Ref="#PWR0222"  Part="1"
+F 0 "#PWR0222" H 5050 4600 50  0001 C CNN
+F 1 "+5V" H 5050 4890 50  0000 C CNN
+F 2 "" H 5050 4750 50  0000 C CNN
+F 3 "" H 5050 4750 50  0000 C CNN
+	1    5050 4750
+	1    0    0    -1
+$EndComp
+$Comp
+L Devtank:SP3003-02XJ U?
+U 1 1 5C3985E5
+P 4000 4900
+AR Path="/589A1B39/5C3985E5" Ref="U?"  Part="1"
+AR Path="/5AFBC859/5C3985E5" Ref="U40"  Part="1"
+F 0 "U40" H 3600 4600 50  0000 C CNN
+F 1 "SP3003-02XJ" H 3800 5200 50  0000 C CNN
+F 2 "Devtank_PCB_Lib:SC70-5" H 4150 4400 50  0001 C CNN
+F 3 "DOCUMENTATION" H 4000 4500 50  0001 C CNN
+F 4 "153-004" H 4000 4900 50  0001 C CNN "Devtank"
+	1    4000 4900
+	-1   0    0    -1
+$EndComp
+Wire Wire Line
+	3325 3875 3325 4750
+Wire Wire Line
+	3250 3975 3250 5050
 $EndSCHEMATC

Commit message: Rev C - pre-release
Parts:
- C217, C219, C224, C225: symbol device:C -> HILTOP_Motherboard-rescue:C-device
- D32, D33: symbol device:LED -> HILTOP_Motherboard-rescue:LED-device
- R201, R202, R204, R205, R208, R209: symbol device:R -> HILTOP_Motherboard-rescue:R-device
- R203: value 24K -> 0R; symbol device:R -> HILTOP_Motherboard-rescue:R-device
- R251: value 47K -> DNF; symbol device:R -> HILTOP_Motherboard-rescue:R-device
- U41: symbol silabs:CP2102N-A01-GQFN24 -> HILTOP_Motherboard-rescue:CP2102N-A01-GQFN24-silabs
Connections:
- net +3V3: no longer C217.1, C219.1, C224.1, C225.1, D32.2 (A), D33.2 (A), U41.5 (VIO), U41.6 (VDD), U41.7 (REGIN)
- net USB_BUS_PWR: now also C217.1, C219.1, U41.7 (REGIN)
- new net VDD: C224.1, C225.1, D32.2 (A), D33.2 (A), U41.5 (VIO), U41.6 (VDD)
Changed lines of the file:
@@
 $Descr A4 11693 8268
 encoding utf-8
-Sheet 10 12
+Sheet 9 12
 Title "HILTOP Motherboard"
 Date "2019-07-03"
@@
 USB_N
 $Comp
-L silabs:CP2102N-A01-GQFN24 U41
+L HILTOP_Motherboard-rescue:CP2102N-A01-GQFN24-silabs U41
 U 1 1 5C2328D1
 P 5525 3475
@@
 Wire Wire Line
 	3250 3975 4925 3975
-$Comp
-L power:+3V3 #PWR0223
-U 1 1 5C39C355
-P 5525 1850
-F 0 "#PWR0223" H 5525 1700 50  0001 C CNN
-F 1 "+3V3" H 5540 2023 50  0000 C CNN
-F 2 "" H 5525 1850 50  0001 C CNN
-F 3 "" H 5525 1850 50  0001 C CNN
-	1    5525 1850
-	1    0    0    -1
-$EndComp
-Wire Wire Line
-	5525 1850 5525 1925
 Wire Wire Line
 	5425 2575 5425 2450
@@
 Wire Wire Line
 	4650 3475 4650 2975
-Wire Wire Line
-	4650 2325 5525 2325
-Connection ~ 5525 2325
-Wire Wire Line
-	5525 2325 5525 2450
-$Comp
-L device:R R203
+$Comp
+L HILTOP_Motherboard-rescue:R-device R203
 U 1 1 5C3A3F19
 P 4050 3775
 F 0 "R203" V 3950 3675 50  0000 C CNN
-F 1 "24K" V 3950 3900 50  0000 C CNN
+F 1 "0R" V 3950 3900 50  0000 C CNN
 F 2 "Resistor_SMD:R_0603_1608Metric" V 3980 3775 50  0001 C CNN
 F 3 "" H 4050 3775 50  0001 C CNN
@@
 	3000 2875 3300 2875
 $Comp
-L device:R R?
+L HILTOP_Motherboard-rescue:R-device R?
 U 1 1 5C3AE29F
 P 6650 3850
@@
 $EndComp
 $Comp
-L device:LED D?
+L HILTOP_Motherboard-rescue:LED-device D?
 U 1 1 5C3AE2A6
 P 7350 3850
@@
 	6800 3850 7200 3850
 $Comp
-L device:R R?
+L HILTOP_Motherboard-rescue:R-device R?
 U 1 1 5C3AF9C1
 P 6650 4075
@@
 $EndComp
 $Comp
-L device:LED D?
+L HILTOP_Motherboard-rescue:LED-device D?
 U 1 1 5C3AF9C7
 P 7350 4075
@@
 	6125 3275 7125 3275
 $Comp
-L device:R R208
+L HILTOP_Motherboard-rescue:R-device R208
 U 1 1 5C3B4D7B
 P 7275 3175
@@
 $EndComp
 $Comp
-L device:R R209
+L HILTOP_Motherboard-rescue:R-device R209
 U 1 1 5C3B4EF0
 P 7275 3275
@@
 	7425 3275 7575 3275
 $Comp
-L device:C C219
+L HILTOP_Motherboard-rescue:C-device C219
 U 1 1 5C3B9E2E
 P 4350 3250
@@
 	4350 3425 4350 3400
 $Comp
-L device:C C217
+L HILTOP_Motherboard-rescue:C-device C217
 U 1 1 5C3BA6B6
 P 3900 3250
@@
 Wire Wire Line
 	4350 2975 4650 2975
-Connection ~ 4650 2975
-Wire Wire Line
-	4650 2975 4650 2325
 Wire Wire Line
 	3900 3100 3900 2975
@@
 	3900 3425 3900 3400
 $Comp
-L device:R R201
+L HILTOP_Motherboard-rescue:R-device R201
 U 1 1 5C3C0EE1
 P 3450 2875
@@
 	3600 2875 3825 2875
 $Comp
-L device:R R202
+L HILTOP_Motherboard-rescue:R-device R202
 U 1 1 5C3C0F83
 P 3825 2625
@@
 	3825 2400 3825 2475
 $Comp
-L device:C C224
+L HILTOP_Motherboard-rescue:C-device C224
 U 1 1 5C3C60B5
 P 5800 2225
@@
 $EndComp
 $Comp
-L device:C C225
+L HILTOP_Motherboard-rescue:C-device C225
 U 1 1 5C3C6FB8
 P 6225 2225
@@
 Wire Wire Line
 	5800 1925 5525 1925
-Connection ~ 5525 1925
-Wire Wire Line
-	5525 1925 5525 2325
 Wire Wire Line
 	6225 2075 6225 1925
@@
 Wire Wire Line
 	5800 2375 5800 2425
-$Comp
-L power:+3V3 #PWR0227
-U 1 1 5C3D2F35
-P 7875 3675
-F 0 "#PWR0227" H 7875 3525 50  0001 C CNN
-F 1 "+3V3" H 7890 3848 50  0000 C CNN
-F 2 "" H 7875 3675 50  0001 C CNN
-F 3 "" H 7875 3675 50  0001 C CNN
-	1    7875 3675
-	1    0    0    -1
-$EndComp
 Wire Wire Line
 	7875 3675 7875 3850
@@
 NoConn ~ 6125 3875
 $Comp
-L device:R R251
+L HILTOP_Motherboard-rescue:R-device R251
 U 1 1 5D3E6FB7
 P 4650 4175
 F 0 "R251" H 4475 4125 50  0000 C CNN
-F 1 "47K" H 4500 4225 50  0000 C CNN
+F 1 "DNF" H 4500 4225 50  0000 C CNN
 F 2 "Resistor_SMD:R_0603_1608Metric" V 4580 4175 50  0001 C CNN
 F 3 "" H 4650 4175 50  0001 C CNN
@@
 Wire Wire Line
 	3250 3975 3250 5050
+Wire Wire Line
+	3900 2975 3425 2975
+Wire Wire Line
+	3425 2975 3425 3600
+Connection ~ 3900 2975
+Connection ~ 3425 3600
+Wire Wire Line
+	5525 1925 5525 2450
+$Comp
+L power:VDD #PWR067
+U 1 1 5EBB4275
+P 7875 3675
+F 0 "#PWR067" H 7875 3525 50  0001 C CNN
+F 1 "VDD" H 7890 3848 50  0000 C CNN
+F 2 "" H 7875 3675 50  0001 C CNN
+F 3 "" H 7875 3675 50  0001 C CNN
+	1    7875 3675
+	1    0    0    -1
+$EndComp
+$Comp
+L power:VDD #PWR063
+U 1 1 5EBB4893
+P 5525 1825
+F 0 "#PWR063" H 5525 1675 50  0001 C CNN
+F 1 "VDD" H 5540 1998 50  0000 C CNN
+F 2 "" H 5525 1825 50  0001 C CNN
+F 3 "" H 5525 1825 50  0001 C CNN
+	1    5525 1825
+	1    0    0    -1
+$EndComp
+Connection ~ 5525 1925
+Wire Wire Line
+	5525 1825 5525 1925
 $EndSCHEMATC
