File: HILTOP_motherboard/RS485.sch (KiCad schematic (older format))
At the start: 58 parts, among them U13 CME0505S3C, U15 ISO3080, U16 ISO3080, U17 CME0505S3C, U18 USB6B1, U19 USB6B1, U20 USB6B1, U21 USB6B1, U43 MAX3107, U44 MAX3107, Y8 3.6864MHz Crystal, Y9 3.6864MHz Crystal

Commit message: Rev C - pre-release
Parts:
- C202, C214, C220, C226, C227, C228, C229, C230, C231, C232, C233, C234, C235, C239, C240, C43, C44, C45, C46, C71, C72, C73, C76, C78, C80, C81, C82, C83: symbol device:C -> HILTOP_Motherboard-rescue:C-device
- FB10, FB6, L5, L6: symbol device:L -> HILTOP_Motherboard-rescue:L-device
- R188, R192, R193, R194, R195, R196, R197, R198, R221, R222, R223, R243, R244, R81: symbol device:R -> HILTOP_Motherboard-rescue:R-device
- U18, U19, U20, U21: symbol ESD_Protection:USB6B1 -> HILTOP_Motherboard-rescue:USB6B1-ESD_Protection
- Y8, Y9: symbol device:Crystal -> HILTOP_Motherboard-rescue:Crystal-device
Changed lines of the file:
@@
 $Descr A3 16535 11693
 encoding utf-8
-Sheet 12 12
+Sheet 11 12
 Title "HILTOP Motherboard"
 Date "2019-07-03"
@@
 $EndDescr
 $Comp
-L device:C C76
+L HILTOP_Motherboard-rescue:C-device C76
 U 1 1 589A9057
 P 5725 7775
@@
 $EndComp
 $Comp
-L device:L L5
+L HILTOP_Motherboard-rescue:L-device L5
 U 1 1 589A9058
 P 5475 7525
@@
 $EndComp
 $Comp
-L device:C C82
+L HILTOP_Motherboard-rescue:C-device C82
 U 1 1 593A8F03
 P 9175 2275
@@
 $EndComp
 $Comp
-L device:C C80
+L HILTOP_Motherboard-rescue:C-device C80
 U 1 1 593A8F8E
 P 7275 2075
@@
 $EndComp
 $Comp
-L device:C C81
+L HILTOP_Motherboard-rescue:C-device C81
 U 1 1 593A9026
 P 7275 4525
@@
 $EndComp
 $Comp
-L device:C C83
+L HILTOP_Motherboard-rescue:C-device C83
 U 1 1 593A90C1
 P 9175 4725
@@
 $EndComp
 $Comp
-L device:C C78
+L HILTOP_Motherboard-rescue:C-device C78
 U 1 1 593AACE9
 P 3300 7750
@@
 Connection ~ 8875 5775
 $Comp
-L ESD_Protection:USB6B1 U18
+L HILTOP_Motherboard-rescue:USB6B1-ESD_Protection U18
 U 1 1 5AE93D3E
 P 10150 2725
@@
 	10550 2825 11350 2825
 $Comp
-L ESD_Protection:USB6B1 U19
+L HILTOP_Motherboard-rescue:USB6B1-ESD_Protection U19
 U 1 1 5AE94628
 P 10150 3275
@@
 RS485_CH2_A
 $Comp
-L ESD_Protection:USB6B1 U20
+L HILTOP_Motherboard-rescue:USB6B1-ESD_Protection U20
 U 1 1 5AE951A9
 P 10150 5175
@@
 	10550 5275 11350 5275
 $Comp
-L ESD_Protection:USB6B1 U21
+L HILTOP_Motherboard-rescue:USB6B1-ESD_Protection U21
 U 1 1 5AE951B5
 P 10150 5725
@@
 $EndComp
 $Comp
-L device:C C43
+L HILTOP_Motherboard-rescue:C-device C43
 U 1 1 5AEA5E9A
 P 6050 7775
@@
 Connection ~ 6050 7525
 $Comp
-L device:C C45
+L HILTOP_Motherboard-rescue:C-device C45
 U 1 1 5AEA8912
 P 10275 7775
@@
 $EndComp
 $Comp
-L device:L L6
+L HILTOP_Motherboard-rescue:L-device L6
 U 1 1 5AEA8919
 P 9825 7525
@@
 $EndComp
 $Comp
-L device:C C44
+L HILTOP_Motherboard-rescue:C-device C44
 U 1 1 5AEA8920
 P 7875 7750
@@
 $EndComp
 $Comp
-L device:C C46
+L HILTOP_Motherboard-rescue:C-device C46
 U 1 1 5AEA8954
 P 10600 7775
@@
 	5725 2925 7025 2925
 $Comp
-L device:R R81
+L HILTOP_Motherboard-rescue:R-device R81
 U 1 1 5AEADA7B
 P 7025 3325
@@
 	4275 3125 2750 3125
 $Comp
-L device:C C227
+L HILTOP_Motherboard-rescue:C-device C227
 U 1 1 5C5CB8C9
 P 3200 2825
@@
 	4275 3625 3925 3625
 $Comp
-L device:Crystal Y8
+L HILTOP_Motherboard-rescue:Crystal-device Y8
 U 1 1 5C654B76
 P 5000 1900
@@
 	5925 2525 5725 2525
 $Comp
-L device:C C234
+L HILTOP_Motherboard-rescue:C-device C234
 U 1 1 5C6CD0D0
 P 6450 2425
@@
 $EndComp
 $Comp
-L device:C C226
+L HILTOP_Motherboard-rescue:C-device C226
 U 1 1 5C6CD1CB
 P 3200 2475
@@
 	6725 2425 6725 2500
 $Comp
-L device:C C232
+L HILTOP_Motherboard-rescue:C-device C232
 U 1 1 5C74CC3E
 P 6400 3525
@@
 	3825 2725 4275 2725
 $Comp
-L device:C C230
+L HILTOP_Motherboard-rescue:C-device C230
 U 1 1 5C7C435E
 P 3525 1800
@@
 	3250 1850 3250 1800
 $Comp
-L device:L FB?
+L HILTOP_Motherboard-rescue:L-device FB?
 U 1 1 5C7E6C55
 P 3525 1350
@@
 	5725 5375 7025 5375
 $Comp
-L device:R R244
+L HILTOP_Motherboard-rescue:R-device R244
 U 1 1 5C8947B9
 P 7025 5775
@@
 	4275 5775 1500 5775
 $Comp
-L device:C C229
+L HILTOP_Motherboard-rescue:C-device C229
 U 1 1 5C8947F0
 P 3200 5275
@@
 	4275 5975 2150 5975
 $Comp
-L device:Crystal Y9
+L HILTOP_Motherboard-rescue:Crystal-device Y9
 U 1 1 5C894804
 P 5000 4350
@@
 	5925 4975 5725 4975
 $Comp
-L device:C C235
+L HILTOP_Motherboard-rescue:C-device C235
 U 1 1 5C894812
 P 6450 4875
@@
 $EndComp
 $Comp
-L device:C C228
+L HILTOP_Motherboard-rescue:C-device C228
 U 1 1 5C894820
 P 3200 4925
@@
 	6725 4875 6725 4950
 $Comp
-L device:C C233
+L HILTOP_Motherboard-rescue:C-device C233
 U 1 1 5C894837
 P 6400 5975
@@
 	3825 5175 4275 5175
 $Comp
-L device:C C231
+L HILTOP_Motherboard-rescue:C-device C231
 U 1 1 5C894855
 P 3525 4250
@@
 	3250 4250 3375 4250
 $Comp
-L device:L FB?
+L HILTOP_Motherboard-rescue:L-device FB?
 U 1 1 5C894865
 P 3525 3950
@@
 	2550 3425 1900 3425
 $Comp
-L device:R R243
+L HILTOP_Motherboard-rescue:R-device R243
 U 1 1 5CB00B06
 P 2225 2800
@@
 $EndComp
 $Comp
-L device:R R223
+L HILTOP_Motherboard-rescue:R-device R223
 U 1 1 5CB01064
 P 1875 3625
@@
 	2225 2550 2225 2650
 $Comp
-L device:R R221
+L HILTOP_Motherboard-rescue:R-device R221
 U 1 1 5F293824
 P 1450 2800
@@
 	1450 2550 1450 2650
 $Comp
-L device:R R222
+L HILTOP_Motherboard-rescue:R-device R222
 U 1 1 5F2E18EC
 P 1500 5250
@@
 	11650 2725 11975 2725
 $Comp
-L device:R R188
+L HILTOP_Motherboard-rescue:R-device R188
 U 1 1 5D858A1B
 P 11500 2725
@@
 $EndComp
 $Comp
-L device:R R192
+L HILTOP_Motherboard-rescue:R-device R192
 U 1 1 5D85A242
 P 11500 2825
@@
 	11650 2825 12200 2825
 $Comp
-L device:R R193
+L HILTOP_Motherboard-rescue:R-device R193
 U 1 1 5D85D232
 P 11500 3275
@@
 	11650 3275 12425 3275
 $Comp
-L device:R R194
+L HILTOP_Motherboard-rescue:R-device R194
 U 1 1 5D85D2C2
 P 11500 3375
@@
 Connection ~ 12425 3950
 $Comp
-L device:R R195
+L HILTOP_Motherboard-rescue:R-device R195
 U 1 1 5DA74035
 P 11500 5175
@@
 	11650 5175 11975 5175
 $Comp
-L device:R R196
+L HILTOP_Motherboard-rescue:R-device R196
 U 1 1 5DA743A6
 P 11500 5275
@@
 	11650 5275 12200 5275
 $Comp
-L device:R R197
+L HILTOP_Motherboard-rescue:R-device R197
 U 1 1 5DA74436
 P 11500 5725
@@
 	11650 5725 12425 5725
 $Comp
-L device:R R198
+L HILTOP_Motherboard-rescue:R-device R198
 U 1 1 5DA744DA
 P 11500 5825
@@
 	11650 5825 12650 5825
 $Comp
-L device:C C72
+L HILTOP_Motherboard-rescue:C-device C72
 U 1 1 5DA74A70
 P 11975 6150
@@
 	12650 5825 12900 5825
 $Comp
-L device:C C202
+L HILTOP_Motherboard-rescue:C-device C202
 U 1 1 5DB2DE7B
 P 12200 6150
@@
 $EndComp
 $Comp
-L device:C C220
+L HILTOP_Motherboard-rescue:C-device C220
 U 1 1 5DB2DF5B
 P 12425 6150
@@
 $EndComp
 $Comp
-L device:C C240
+L HILTOP_Motherboard-rescue:C-device C240
 U 1 1 5DB2DFF1
 P 12650 6150
@@
 $EndComp
 $Comp
-L device:C C71
+L HILTOP_Motherboard-rescue:C-device C71
 U 1 1 5DB2E101
 P 11975 3675
@@
 $EndComp
 $Comp
-L device:C C73
+L HILTOP_Motherboard-rescue:C-device C73
 U 1 1 5DB2E508
 P 12200 3675
@@
 $EndComp
 $Comp
-L device:C C214
+L HILTOP_Motherboard-rescue:C-device C214
 U 1 1 5DB2E5B8
 P 12425 3675
@@
 $EndComp
 $Comp
-L device:C C239
+L HILTOP_Motherboard-rescue:C-device C239
 U 1 1 5DB2E654
 P 12650 3675
