File: HILTOP_motherboard/RS485.sch (KiCad schematic (older format))
At the start: 58 parts, among them U13 CME0505S3C, U15 ISO3080, U16 ISO3080, U17 CME0505S3C, U18 USB6B1, U19 USB6B1, U20 USB6B1, U21 USB6B1, U43 MAX3107, U44 MAX3107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

Commit message: changed silkscreen to revD and updated sheet information
Parts:
- U13, U17: symbol Devtank:CME0303S3C -> HILTOP_Motherboard-rescue:CME0303S3C-Devtank
- U43, U44: symbol Devtank:MAX3107 -> HILTOP_Motherboard-rescue:MAX3107-Devtank
Changed lines of the file:
@@
 Sheet 11 12
 Title "HILTOP Motherboard"
-Date "2020-04-28"
-Rev "Rev C"
+Date "2021-02-17"
+Rev "Rev D"
 Comp "Devtank Ltd"
-Comment1 ""
+Comment1 "Part No: 304-001"
 Comment2 ""
 Comment3 ""
@@
 $EndComp
 $Comp
-L Devtank:GND_ISO3 #PWR0192
+L HILTOP_Motherboard-rescue:GND_ISO3-Devtank #PWR0192
 U 1 1 589A9068
 P 9175 2475
@@
 $EndComp
 $Comp
-L Devtank:GND_ISO3 #PWR0189
+L HILTOP_Motherboard-rescue:GND_ISO3-Devtank #PWR0189
 U 1 1 589A906B
 P 8875 3625
@@
 $EndComp
 $Comp
-L Devtank:GND_ISO4 #PWR0191
+L HILTOP_Motherboard-rescue:GND_ISO4-Devtank #PWR0191
 U 1 1 589A907C
 P 8875 6075
@@
 $EndComp
 $Comp
-L Devtank:GND_ISO4 #PWR0197
+L HILTOP_Motherboard-rescue:GND_ISO4-Devtank #PWR0197
 U 1 1 589A907D
 P 10600 8175
@@
 $EndComp
 $Comp
-L Devtank:GND_ISO4 #PWR0193
+L HILTOP_Motherboard-rescue:GND_ISO4-Devtank #PWR0193
 U 1 1 593AA526
 P 9175 4925
@@
 $EndComp
 $Comp
-L Devtank:GND_ISO3 #PWR0181
+L HILTOP_Motherboard-rescue:GND_ISO3-Devtank #PWR0181
 U 1 1 589A9056
 P 6050 8175
@@
 	9400 3375 9750 3375
 $Comp
-L Devtank:GND_ISO3 #PWR0194
+L HILTOP_Motherboard-rescue:GND_ISO3-Devtank #PWR0194
 U 1 1 5AE948B9
 P 9675 3625
@@
 	9350 5825 9750 5825
 $Comp
-L Devtank:GND_ISO4 #PWR0195
+L HILTOP_Motherboard-rescue:GND_ISO4-Devtank #PWR0195
 U 1 1 5AE9578A
 P 9675 6075
@@
 Connection ~ 3300 8000
 $Comp
-L Devtank:CME0303S3C U13
+L HILTOP_Motherboard-rescue:CME0303S3C-Devtank U13
 U 1 1 589A9055
 P 4275 7850
@@
 	5025 7700 5025 7525
 $Comp
-L Devtank:+5V_ISO3 #PWR0188
+L HILTOP_Motherboard-rescue:+5V_ISO3-Devtank #PWR0188
 U 1 1 5AEA3286
 P 8875 1925
@@
 $EndComp
 $Comp
-L Devtank:+5V_ISO4 #PWR0190
+L HILTOP_Motherboard-rescue:+5V_ISO4-Devtank #PWR0190
 U 1 1 5AEA32BE
 P 8875 4375
@@
 $EndComp
 $Comp
-L Devtank:+5V_ISO3 #PWR0180
+L HILTOP_Motherboard-rescue:+5V_ISO3-Devtank #PWR0180
 U 1 1 5AEA5482
 P 6050 7350
@@
 Connection ~ 10275 8000
 $Comp
-L Devtank:CME0303S3C U17
+L HILTOP_Motherboard-rescue:CME0303S3C-Devtank U17
 U 1 1 5AEA893F
 P 8850 7850
@@
 Connection ~ 10600 7525
 $Comp
-L Devtank:+5V_ISO4 #PWR0196
+L HILTOP_Motherboard-rescue:+5V_ISO4-Devtank #PWR0196
 U 1 1 5AEA8C4F
 P 10600 7350
@@
 	7025 3625 7025 3475
 $Comp
-L Devtank:+5V_ISO3 #PWR0201
+L HILTOP_Motherboard-rescue:+5V_ISO3-Devtank #PWR0201
 U 1 1 5AED924B
 P 10825 2400
@@
 	10750 2925 10550 2925
 $Comp
-L Devtank:GND_ISO3 #PWR0198
+L HILTOP_Motherboard-rescue:GND_ISO3-Devtank #PWR0198
 U 1 1 5AED9511
 P 10750 3625
@@
 	10550 5075 10650 5075
 $Comp
-L Devtank:+5V_ISO4 #PWR0200
+L HILTOP_Motherboard-rescue:+5V_ISO4-Devtank #PWR0200
 U 1 1 5AEDB949
 P 10775 4850
@@
 	10775 5075 10775 4850
 $Comp
-L Devtank:GND_ISO4 #PWR0199
+L HILTOP_Motherboard-rescue:GND_ISO4-Devtank #PWR0199
 U 1 1 5AEDBBAE
 P 10750 6075
@@
 	10750 5925 10750 6075
 $Comp
-L Devtank:MAX3107 U43
+L HILTOP_Motherboard-rescue:MAX3107-Devtank U43
 U 1 1 5C52F3AC
 P 4775 2575
@@
 	7025 6075 7025 5925
 $Comp
-L Devtank:MAX3107 U44
+L HILTOP_Motherboard-rescue:MAX3107-Devtank U44
 U 1 1 5C8947B0
 P 4775 5025
@@
 	12650 3375 12900 3375
 $Comp
-L Devtank:GND_ISO3 #PWR0458
+L HILTOP_Motherboard-rescue:GND_ISO3-Devtank #PWR0458
 U 1 1 5D943A37
 P 11975 4000
@@
 Parts in dashed box to be placed\nnear output connector.
 $Comp
-L Devtank:GND_ISO4 #PWR0459
+L HILTOP_Motherboard-rescue:GND_ISO4-Devtank #PWR0459
 U 1 1 5ED00EC9
 P 11975 6475
