File: HILTOP_motherboard/AdjPower.sch (KiCad schematic (older format))
At the start: 92 parts, among them Q1 Si7148DP-T1-E3, Q2 Si7148DP-T1-E3, Q4 2N7002, U10 TLC271, U11 ADS1015, U12 MCP4725, U8 LM5118, U9 INA250A3

Commit message: changed silkscreen to revD and updated sheet information
Parts:
- Q1, Q2: symbol Devtank:Q_NMOS_DS_POWERPAK -> HILTOP_Motherboard-rescue:Q_NMOS_DS_POWERPAK-Devtank
- RL1: symbol Devtank:SPST-NO -> HILTOP_Motherboard-rescue:SPST-NO-Devtank
- U10: symbol Devtank:TLC271 -> HILTOP_Motherboard-rescue:TLC271-Devtank
- U11: symbol Devtank:ADS1015 -> HILTOP_Motherboard-rescue:ADS1015-Devtank
- U12: symbol Devtank:MCP4725 -> HILTOP_Motherboard-rescue:MCP4725-Devtank
- U8: symbol Devtank:LM5118 -> HILTOP_Motherboard-rescue:LM5118-Devtank
- U9: symbol Devtank:INA250 -> HILTOP_Motherboard-rescue:INA250-Devtank
Changed lines of the file:
@@
 Sheet 5 12
 Title "HILTOP Motherboard"
-Date "2020-04-28"
-Rev "Rev C"
+Date "2021-02-17"
+Rev "Rev D"
 Comp "Devtank Ltd"
-Comment1 ""
+Comment1 "Part No: 304-001"
 Comment2 ""
 Comment3 ""
@@
 PWR_ENABLE
 $Comp
-L Devtank:LM5118 U8
+L HILTOP_Motherboard-rescue:LM5118-Devtank U8
 U 1 1 58E08D87
 P 4650 4300
@@
 $EndComp
 $Comp
-L Devtank:ADS1015 U11
+L HILTOP_Motherboard-rescue:ADS1015-Devtank U11
 U 1 1 58DFE046
 P 14400 5100
@@
 $EndComp
 $Comp
-L Devtank:MCP4725 U12
+L HILTOP_Motherboard-rescue:MCP4725-Devtank U12
 U 1 1 58DFEBB8
 P 13950 7800
@@
 VADJ_GND
 $Comp
-L Devtank:TLC271 U10
+L HILTOP_Motherboard-rescue:TLC271-Devtank U10
 U 1 1 58EA7C27
 P 8650 8850
@@
 $EndComp
 $Comp
-L Devtank:SPST-NO RL1
+L HILTOP_Motherboard-rescue:SPST-NO-Devtank RL1
 U 1 1 58FEC418
 P 12550 4250
@@
 $EndComp
 $Comp
-L Devtank:INA250 U9
+L HILTOP_Motherboard-rescue:INA250-Devtank U9
 U 1 1 58FFB89A
 P 10700 4550
@@
 $EndComp
 $Comp
-L Devtank:-5V #PWR0324
+L HILTOP_Motherboard-rescue:-5V-Devtank #PWR0324
 U 1 1 5904EE57
 P 8700 9600
@@
 $EndComp
 $Comp
-L Devtank:Q_NMOS_DS_POWERPAK Q1
+L HILTOP_Motherboard-rescue:Q_NMOS_DS_POWERPAK-Devtank Q1
 U 1 1 593D8AB2
 P 6800 3100
@@
 $EndComp
 $Comp
-L Devtank:Q_NMOS_DS_POWERPAK Q2
+L HILTOP_Motherboard-rescue:Q_NMOS_DS_POWERPAK-Devtank Q2
 U 1 1 593D9A34
 P 7350 5000
