File: HILTOP_motherboard/PWM_Fans.sch (KiCad schematic (older format))
At the start: 14 parts, among them Q5 ZXMN6A07F, Q6 ZXMN6A07F, U42 FDC6330L

Commit message: BOM nearly complete!
Parts:
- removed R210, R213: 100K, Resistor_SMD:R_0603_1608Metric, symbol device:R
- removed R211: DNP, Resistor_SMD:R_0603_1608Metric, symbol device:R
- removed R212, R214: 1K, Resistor_SMD:R_0603_1608Metric, symbol device:R
- removed U42: FDC6330L, Devtank_PCB_Lib:SuperSOT-6, symbol Devtank:FDC6324L
- added C237, C238: DNF, Capacitor_SMD:C_0603_1608Metric, symbol device:C
- added Q7: ZXMN6A07F, Package_TO_SOT_SMD:SOT-23, symbol device:Q_NMOS_GSD
- added Q8: SSM3J328R, Package_TO_SOT_SMD:SOT-23, symbol device:Q_PMOS_GSD
- added R159, R184, R185: 10K, Resistor_SMD:R_0603_1608Metric, symbol device:R
- Q5, Q6: Devtank (none) -> 170-002
Connections:
- net labels removed: +3V3
- wire segments 49 -> 51
Changed lines of the file:
@@
 $Descr A4 11693 8268
 encoding utf-8
-Sheet 12 12
+Sheet 11 12
 Title ""
 Date ""
@@
 Text HLabel 4425 2450 0    60   Input ~ 0
 PWW_CTRL
-Text HLabel 1550 4275 0    60   Input ~ 0
+Text HLabel 2175 6350 0    60   Input ~ 0
 FAN_PWR
 Text HLabel 7750 2150 2    60   Output ~ 0
@@
 F 2 "Package_TO_SOT_SMD:SOT-23" H 6400 2550 50  0001 C CNN
 F 3 "" H 6200 2450 50  0001 C CNN
+F 4 "170-002" H 6200 2450 50  0001 C CNN "Devtank"
 	1    6200 2450
 	1    0    0    -1
@@
 F 2 "Package_TO_SOT_SMD:SOT-23" H 6400 4425 50  0001 C CNN
 F 3 "" H 6200 4325 50  0001 C CNN
+F 4 "170-002" H 6200 4325 50  0001 C CNN "Devtank"
 	1    6200 4325
 	1    0    0    -1
@@
 	4900 2450 4425 2450
 Connection ~ 4900 2450
-$Comp
-L Devtank:FDC6324L U42
-U 1 1 5C2BEFC6
-P 3975 6100
-F 0 "U42" H 3450 6575 50  0000 C CNN
-F 1 "FDC6330L" H 4400 6575 50  0000 C CNN
-F 2 "Devtank_PCB_Lib:SuperSOT-6" H 3925 6050 50  0001 C CNN
-F 3 "" H 3075 6500 50  0000 C CNN
-	1    3975 6100
-	1    0    0    -1
-$EndComp
-$Comp
-L device:R R213
-U 1 1 5C2BF311
-P 2800 6100
-F 0 "R213" H 2675 6150 50  0000 C CNN
-F 1 "100K" H 2650 6050 50  0000 C CNN
-F 2 "Resistor_SMD:R_0603_1608Metric" V 2730 6100 50  0001 C CNN
-F 3 "" H 2800 6100 50  0000 C CNN
-F 4 "101-015" H 2800 6100 60  0001 C CNN "Devtank"
-	1    2800 6100
-	1    0    0    -1
-$EndComp
-$Comp
-L power:+12V #PWR0416
-U 1 1 5C2BF5F6
-P 2225 5500
-F 0 "#PWR0416" H 2225 5350 50  0001 C CNN
-F 1 "+12V" H 2240 5673 50  0000 C CNN
-F 2 "" H 2225 5500 50  0001 C CNN
-F 3 "" H 2225 5500 50  0001 C CNN
-	1    2225 5500
-	1    0    0    -1
-$EndComp
-Wire Wire Line
-	2800 5850 2800 5950
-Wire Wire Line
-	2800 6250 2800 6350
-Wire Wire Line
-	2800 6350 3275 6350
-Wire Wire Line
-	3275 5850 2800 5850
-Connection ~ 2800 5850
-Wire Wire Line
-	2225 5850 2225 5500
-Text HLabel 5900 5850 2    60   Output ~ 0
+Text HLabel 4200 5150 2    60   Output ~ 0
 12V_SW_LOAD
-Wire Wire Line
-	4675 5850 4925 5850
-Wire Wire Line
-	4675 6100 4925 6100
-Wire Wire Line
-	4925 6100 4925 5850
-Connection ~ 4925 5850
-Wire Wire Line
-	4925 5850 5900 5850
-$Comp
-L device:R R214
-U 1 1 5C2C1540
-P 5100 6350
-F 0 "R214" V 5000 6200 50  0000 C CNN
-F 1 "1K" V 5000 6475 50  0000 C CNN
-F 2 "Resistor_SMD:R_0603_1608Metric" V 5030 6350 50  0001 C CNN
-F 3 "" H 5100 6350 50  0000 C CNN
-F 4 "101-012" V 5100 6350 60  0001 C CNN "Devtank"
-	1    5100 6350
-	0    1    1    0
-$EndComp
-Wire Wire Line
-	4950 6350 4675 6350
-$Comp
-L power:GND #PWR0417
-U 1 1 5C2C1D1E
-P 5500 6450
-F 0 "#PWR0417" H 5500 6200 50  0001 C CNN
-F 1 "GND" H 5500 6300 50  0000 C CNN
-F 2 "" H 5500 6450 50  0001 C CNN
-F 3 "" H 5500 6450 50  0001 C CNN
-	1    5500 6450
-	1    0    0    -1
-$EndComp
-Wire Wire Line
-	5500 6450 5500 6350
-Wire Wire Line
-	5500 6350 5250 6350
-$Comp
-L device:R R210
-U 1 1 5C2C5AC7
-P 1825 4500
-F 0 "R210" H 1700 4550 50  0000 C CNN
-F 1 "100K" H 1675 4450 50  0000 C CNN
-F 2 "Resistor_SMD:R_0603_1608Metric" V 1755 4500 50  0001 C CNN
-F 3 "" H 1825 4500 50  0000 C CNN
-F 4 "101-015" H 1825 4500 60  0001 C CNN "Devtank"
-	1    1825 4500
-	1    0    0    -1
-$EndComp
-$Comp
-L power:GND #PWR0414
-U 1 1 5C2C5C95
-P 1825 4750
-F 0 "#PWR0414" H 1825 4500 50  0001 C CNN
-F 1 "GND" H 1825 4600 50  0000 C CNN
-F 2 "" H 1825 4750 50  0001 C CNN
-F 3 "" H 1825 4750 50  0001 C CNN
-	1    1825 4750
-	1    0    0    -1
-$EndComp
-Wire Wire Line
-	1825 4750 1825 4650
-$Comp
-L device:R R211
-U 1 1 5C2C648B
-P 1950 4050
-F 0 "R211" H 1825 4100 50  0000 C CNN
-F 1 "DNP" H 1800 4000 50  0000 C CNN
-F 2 "Resistor_SMD:R_0603_1608Metric" V 1880 4050 50  0001 C CNN
-F 3 "" H 1950 4050 50  0000 C CNN
-	1    1950 4050
-	1    0    0    -1
-$EndComp
-$Comp
-L power:+3V3 #PWR0415
-U 1 1 5C2C65B8
-P 1950 3700
-F 0 "#PWR0415" H 1950 3550 50  0001 C CNN
-F 1 "+3V3" H 1965 3873 50  0000 C CNN
-F 2 "" H 1950 3700 50  0001 C CNN
-F 3 "" H 1950 3700 50  0001 C CNN
-	1    1950 3700
-	1    0    0    -1
-$EndComp
-$Comp
-L device:R R212
-U 1 1 5C2C76CA
-P 2400 4275
-F 0 "R212" V 2300 4125 50  0000 C CNN
-F 1 "1K" V 2300 4400 50  0000 C CNN
-F 2 "Resistor_SMD:R_0603_1608Metric" V 2330 4275 50  0001 C CNN
-F 3 "" H 2400 4275 50  0000 C CNN
-F 4 "101-012" V 2400 4275 60  0001 C CNN "Devtank"
-	1    2400 4275
-	0    1    1    0
-$EndComp
-Wire Wire Line
-	1950 3700 1950 3900
-Wire Wire Line
-	2250 4275 1950 4275
-Wire Wire Line
-	1950 4200 1950 4275
-Connection ~ 1950 4275
-Wire Wire Line
-	1950 4275 1825 4275
-Wire Wire Line
-	1825 4350 1825 4275
-Connection ~ 1825 4275
-Wire Wire Line
-	1825 4275 1550 4275
-Wire Wire Line
-	2550 4275 3000 4275
-Wire Wire Line
-	3000 4275 3000 6100
-Wire Wire Line
-	3000 6100 3275 6100
-Wire Wire Line
-	2225 5850 2800 5850
+$Comp
+L power:GND #PWR0281
+U 1 1 5C6F6F0B
+P 3175 6825
+F 0 "#PWR0281" H 3175 6575 50  0001 C CNN
+F 1 "GND" H 3175 6675 50  0000 C CNN
+F 2 "" H 3175 6825 50  0001 C CNN
+F 3 "" H 3175 6825 50  0001 C CNN
+	1    3175 6825
+	1    0    0    -1
+$EndComp
+$Comp
+L device:Q_NMOS_GSD Q7
+U 1 1 5C6F6F19
+P 3075 6350
+F 0 "Q7" H 3275 6400 50  0000 L CNN
+F 1 "ZXMN6A07F" H 3275 6300 50  0000 L CNN
+F 2 "Package_TO_SOT_SMD:SOT-23" H 3275 6450 50  0001 C CNN
+F 3 "" H 3075 6350 50  0001 C CNN
+F 4 "170-002" H 3075 6350 50  0001 C CNN "Devtank"
+	1    3075 6350
+	1    0    0    -1
+$EndComp
+$Comp
+L device:R R159
+U 1 1 5C6F6F21
+P 2750 6550
+F 0 "R159" H 2625 6600 50  0000 C CNN
+F 1 "10K" H 2625 6500 50  0000 C CNN
+F 2 "Resistor_SMD:R_0603_1608Metric" V 2680 6550 50  0001 C CNN
+F 3 "" H 2750 6550 50  0000 C CNN
+F 4 "101-010" H 2750 6550 60  0001 C CNN "Devtank"
+	1    2750 6550
+	1    0    0    -1
+$EndComp
+Wire Wire Line
+	3175 6550 3175 6750
+Wire Wire Line
+	2750 6400 2750 6350
+Wire Wire Line
+	2750 6750 3175 6750
+Connection ~ 3175 6750
+Wire Wire Line
+	2750 6750 2750 6700
+Connection ~ 2750 6350
+Wire Wire Line
+	3175 6750 3175 6825
+Wire Wire Line
+	2750 6350 2875 6350
+$Comp
+L device:Q_PMOS_GSD Q8
+U 1 1 5C6F7F86
+P 3775 5250
+F 0 "Q8" V 4118 5250 50  0000 C CNN
+F 1 "SSM3J328R" V 4027 5250 50  0000 C CNN
+F 2 "Package_TO_SOT_SMD:SOT-23" H 3975 5350 50  0001 C CNN
+F 3 "" H 3775 5250 50  0001 C CNN
+F 4 "173-003" V 3775 5250 50  0001 C CNN "Devtank"
+	1    3775 5250
+	0    1    -1   0
+$EndComp
+$Comp
+L device:R R184
+U 1 1 5C6F9478
+P 3175 5400
+F 0 "R184" H 3050 5450 50  0000 C CNN
+F 1 "10K" H 3050 5350 50  0000 C CNN
+F 2 "Resistor_SMD:R_0603_1608Metric" V 3105 5400 50  0001 C CNN
+F 3 "" H 3175 5400 50  0000 C CNN
+F 4 "101-010" H 3175 5400 60  0001 C CNN "Devtank"
+	1    3175 5400
+	1    0    0    -1
+$EndComp
+$Comp
+L device:R R185
+U 1 1 5C6F9600
+P 3175 5900
+F 0 "R185" H 3050 5950 50  0000 C CNN
+F 1 "10K" H 3050 5850 50  0000 C CNN
+F 2 "Resistor_SMD:R_0603_1608Metric" V 3105 5900 50  0001 C CNN
+F 3 "" H 3175 5900 50  0000 C CNN
+F 4 "101-010" H 3175 5900 60  0001 C CNN "Devtank"
+	1    3175 5900
+	1    0    0    -1
+$EndComp
+Wire Wire Line
+	2800 5150 2800 4975
+$Comp
+L power:+12V #PWR0280
+U 1 1 5C6FA6A6
+P 2800 4975
+F 0 "#PWR0280" H 2800 4825 50  0001 C CNN
+F 1 "+12V" H 2815 5148 50  0000 C CNN
+F 2 "" H 2800 4975 50  0001 C CNN
+F 3 "" H 2800 4975 50  0001 C CNN
+	1    2800 4975
+	1    0    0    -1
+$EndComp
+Wire Wire Line
+	4200 5150 4125 5150
+Wire Wire Line
+	3775 5450 3775 5650
+Wire Wire Line
+	3775 5650 3400 5650
+Wire Wire Line
+	3175 5650 3175 5750
+Wire Wire Line
+	3175 5250 3175 5150
+Connection ~ 3175 5150
+Wire Wire Line
+	3175 5150 2800 5150
+Wire Wire Line
+	3175 5550 3175 5650
+Connection ~ 3175 5650
+Wire Wire Line
+	3175 6050 3175 6150
+Wire Wire Line
+	2175 6350 2750 6350
+$Comp
+L device:C C237
+U 1 1 5C708943
+P 3400 5400
+F 0 "C237" H 3515 5446 50  0000 L CNN
+F 1 "DNF" H 3515 5355 50  0000 L CNN
+F 2 "Capacitor_SMD:C_0603_1608Metric" H 3438 5250 50  0001 C CNN
+F 3 "" H 3400 5400 50  0001 C CNN
+	1    3400 5400
+	1    0    0    -1
+$EndComp
+Wire Wire Line
+	3175 5150 3400 5150
+$Comp
+L device:C C238
+U 1 1 5C70A734
+P 4125 5400
+F 0 "C238" H 4010 5354 50  0000 R CNN
+F 1 "DNF" H 4010 5445 50  0000 R CNN
+F 2 "Capacitor_SMD:C_0603_1608Metric" H 4163 5250 50  0001 C CNN
+F 3 "" H 4125 5400 50  0001 C CNN
+	1    4125 5400
+	-1   0    0    1
+$EndComp
+Wire Wire Line
+	4125 5250 4125 5150
+Connection ~ 4125 5150
+Wire Wire Line
+	4125 5150 3975 5150
+Wire Wire Line
+	4125 5550 4125 5650
+Wire Wire Line
+	4125 5650 3775 5650
+Connection ~ 3775 5650
+Wire Wire Line
+	3400 5550 3400 5650
+Connection ~ 3400 5650
+Wire Wire Line
+	3400 5650 3175 5650
+Wire Wire Line
+	3400 5250 3400 5150
+Connection ~ 3400 5150
+Wire Wire Line
+	3400 5150 3575 5150
 $EndSCHEMATC

Commit message: Rev C - pre-release
Parts:
- C237, C238: symbol device:C -> HILTOP_Motherboard-rescue:C-device
- Q5, Q6, Q7: symbol device:Q_NMOS_GSD -> HILTOP_Motherboard-rescue:Q_NMOS_GSD-device
- Q8: symbol device:Q_PMOS_GSD -> HILTOP_Motherboard-rescue:Q_PMOS_GSD-device
- R159, R184, R185, R215, R216, R217, R218, R219, R220: symbol device:R -> HILTOP_Motherboard-rescue:R-device
Changed lines of the file:
@@
 $Descr A4 11693 8268
 encoding utf-8
-Sheet 11 12
+Sheet 10 12
 Title "HILTOP Motherboard"
 Date "2019-07-03"
@@
 	6300 2000 6300 2150
 $Comp
-L device:R R215
+L HILTOP_Motherboard-rescue:R-device R215
 U 1 1 5F1521D2
 P 5600 2450
@@
 $EndComp
 $Comp
-L device:Q_NMOS_GSD Q?
+L HILTOP_Motherboard-rescue:Q_NMOS_GSD-device Q?
 U 1 1 5F1521D9
 P 6200 2450
@@
 $EndComp
 $Comp
-L device:R R?
+L HILTOP_Motherboard-rescue:R-device R?
 U 1 1 5F1521E1
 P 5875 2650
@@
 	6300 3900 6300 4050
 $Comp
-L device:R R216
+L HILTOP_Motherboard-rescue:R-device R216
 U 1 1 5F152488
 P 5600 4325
@@
 $EndComp
 $Comp
-L device:Q_NMOS_GSD Q6
+L HILTOP_Motherboard-rescue:Q_NMOS_GSD-device Q6
 U 1 1 5F15248F
 P 6200 4325
@@
 $EndComp
 $Comp
-L device:R R218
+L HILTOP_Motherboard-rescue:R-device R218
 U 1 1 5F152497
 P 5875 4525
@@
 	4900 4325 5450 4325
 $Comp
-L device:R R?
+L HILTOP_Motherboard-rescue:R-device R?
 U 1 1 5F152601
 P 6300 1850
@@
 $EndComp
 $Comp
-L device:R R?
+L HILTOP_Motherboard-rescue:R-device R?
 U 1 1 5F1526AA
 P 6300 3750
@@
 $EndComp
 $Comp
-L device:Q_NMOS_GSD Q7
+L HILTOP_Motherboard-rescue:Q_NMOS_GSD-device Q7
 U 1 1 5C6F6F19
 P 3075 6350
@@
 $EndComp
 $Comp
-L device:R R159
+L HILTOP_Motherboard-rescue:R-device R159
 U 1 1 5C6F6F21
 P 2750 6550
@@
 	2750 6350 2875 6350
 $Comp
-L device:Q_PMOS_GSD Q8
+L HILTOP_Motherboard-rescue:Q_PMOS_GSD-device Q8
 U 1 1 5C6F7F86
 P 3775 5250
@@
 $EndComp
 $Comp
-L device:R R184
+L HILTOP_Motherboard-rescue:R-device R184
 U 1 1 5C6F9478
 P 3175 5400
@@
 $EndComp
 $Comp
-L device:R R185
+L HILTOP_Motherboard-rescue:R-device R185
 U 1 1 5C6F9600
 P 3175 5900
@@
 	2175 6350 2750 6350
 $Comp
-L device:C C237
+L HILTOP_Motherboard-rescue:C-device C237
 U 1 1 5C708943
 P 3400 5400
@@
 	3175 5150 3400 5150
 $Comp
-L device:C C238
+L HILTOP_Motherboard-rescue:C-device C238
 U 1 1 5C70A734
 P 4125 5400
