File: HILTOP_motherboard/SATA_Bridge.sch (KiCad schematic (older format))
At the start: 60 parts, among them J25 DEBUG, U37 TUSB9261, U38 AT25DN512CSSHF-B, Y7 40MHz Crystal

Commit message: finished new tracking for RS485 signals and general house keeping
Parts:
- removed D84: STPS1L30, Diode_SMD:D_SMB, symbol device:D
- added C59: DNF, Capacitor_SMD:C_0402_1005Metric, symbol device:C
- added R186: 100K, Resistor_SMD:R_0603_1608Metric, symbol device:R
- added R187: 0R, Resistor_SMD:R_0805_2012Metric, symbol device:R
- added R94: DNF, Resistor_SMD:R_0603_1608Metric, symbol device:R
Connections:
- net labels added: ~RESET
- wire segments 267 -> 275
- no-connect marks 15 -> 14
Changed lines of the file:
@@
 Sheet 8 12
 Title "HILTOP Motherboard"
-Date "2019-01-10"
-Rev "Issue 1"
+Date "2019-07-03"
+Rev "Rev B"
 Comp "Devtank Ltd"
 Comment1 ""
@@
 L power:+1V2 #PWR0402
 U 1 1 5A99EB0C
-P 7500 7700
-F 0 "#PWR0402" H 7500 7550 50  0001 C CNN
-F 1 "+1V2" H 7500 7840 50  0000 C CNN
-F 2 "" H 7500 7700 50  0000 C CNN
-F 3 "" H 7500 7700 50  0000 C CNN
-	1    7500 7700
+P 7650 7700
+F 0 "#PWR0402" H 7650 7550 50  0001 C CNN
+F 1 "+1V2" H 7650 7840 50  0000 C CNN
+F 2 "" H 7650 7700 50  0000 C CNN
+F 3 "" H 7650 7700 50  0000 C CNN
+	1    7650 7700
 	1    0    0    -1
 $EndComp
@@
 	6050 9500 6050 9800
 Wire Wire Line
-	7500 8000 7500 7700
+	7650 8000 7650 7700
 Connection ~ 6175 8000
 Wire Wire Line
@@
 Connection ~ 6225 1675
 $Comp
-L device:D D84
-U 1 1 5B3E1777
-P 7250 8000
-F 0 "D84" H 7250 8100 50  0000 C CNN
-F 1 "STPS1L30" H 7250 7900 50  0000 C CNN
-F 2 "Diode_SMD:D_SMB" H 7250 8000 50  0001 C CNN
-F 3 "" H 7250 8000 50  0001 C CNN
-F 4 "133-001" H 7250 8000 50  0001 C CNN "Devtank"
-	1    7250 8000
-	1    0    0    -1
-$EndComp
-$Comp
 L device:R R224
 U 1 1 5B3E2C11
@@
 	7100 8000 6875 8000
 Wire Wire Line
-	7400 8000 7500 8000
+	7400 8000 7650 8000
 $Comp
 L Devtank:+1V1_SATA #PWR0397
@@
 NoConn ~ 4100 4400
 NoConn ~ 4100 4500
-NoConn ~ 4100 5575
 NoConn ~ 4900 6250
 NoConn ~ 5200 6250
@@
 Text Label 3600 2850 0    60   ~ 0
 RX_P
+$Comp
+L device:R R187
+U 1 1 5D2A03C4
+P 7250 8000
+F 0 "R187" V 7150 7950 50  0000 C CNN
+F 1 "0R" V 7350 7950 50  0000 C CNN
+F 2 "Resistor_SMD:R_0805_2012Metric" V 7180 8000 50  0001 C CNN
+F 3 "" H 7250 8000 50  0000 C CNN
+F 4 "101-005" V 7250 8000 60  0001 C CNN "Devtank"
+	1    7250 8000
+	0    1    1    0
+$EndComp
+$Comp
+L power:+3V3 #PWR?
+U 1 1 5D506DAF
+P 2800 6450
+AR Path="/589A1B39/5D506DAF" Ref="#PWR?"  Part="1"
+AR Path="/5A951BF0/5D506DAF" Ref="#PWR0456"  Part="1"
+F 0 "#PWR0456" H 2800 6300 50  0001 C CNN
+F 1 "+3V3" H 2800 6590 50  0000 C CNN
+F 2 "" H 2800 6450 50  0000 C CNN
+F 3 "" H 2800 6450 50  0000 C CNN
+	1    2800 6450
+	1    0    0    -1
+$EndComp
+$Comp
+L device:R R?
+U 1 1 5D506DB6
+P 2800 6750
+AR Path="/589A1B39/5D506DB6" Ref="R?"  Part="1"
+AR Path="/5A951BF0/5D506DB6" Ref="R186"  Part="1"
+F 0 "R186" H 2950 6700 50  0000 C CNN
+F 1 "100K" H 2950 6800 50  0000 C CNN
+F 2 "Resistor_SMD:R_0603_1608Metric" V 2730 6750 50  0001 C CNN
+F 3 "" H 2800 6750 50  0000 C CNN
+F 4 "101-015" H 2800 6750 60  0001 C CNN "Devtank"
+	1    2800 6750
+	-1   0    0    1
+$EndComp
+$Comp
+L device:C C?
+U 1 1 5D506DBE
+P 2800 7200
+AR Path="/589A1B39/5D506DBE" Ref="C?"  Part="1"
+AR Path="/5A951BF0/5D506DBE" Ref="C59"  Part="1"
+F 0 "C59" H 2825 7300 50  0000 L CNN
+F 1 "DNF" H 2825 7100 50  0000 L CNN
+F 2 "Capacitor_SMD:C_0402_1005Metric" H 2838 7050 50  0001 C CNN
+F 3 "" H 2800 7200 50  0000 C CNN
+F 4 "105-019" H 2800 7200 60  0001 C CNN "Devtank"
+	1    2800 7200
+	1    0    0    -1
+$EndComp
+$Comp
+L power:GND #PWR?
+U 1 1 5D506DC5
+P 2800 7350
+AR Path="/589A1B39/5D506DC5" Ref="#PWR?"  Part="1"
+AR Path="/5A951BF0/5D506DC5" Ref="#PWR0457"  Part="1"
+F 0 "#PWR0457" H 2800 7100 50  0001 C CNN
+F 1 "GND" H 2800 7200 50  0000 C CNN
+F 2 "" H 2800 7350 50  0000 C CNN
+F 3 "" H 2800 7350 50  0000 C CNN
+	1    2800 7350
+	1    0    0    -1
+$EndComp
+Text HLabel 1800 7000 0    60   Input ~ 0
+~RESET
+$Comp
+L device:R R?
+U 1 1 5D506DCD
+P 2300 7000
+AR Path="/589A1B39/5D506DCD" Ref="R?"  Part="1"
+AR Path="/5A951BF0/5D506DCD" Ref="R94"  Part="1"
+F 0 "R94" V 2200 6900 50  0000 C CNN
+F 1 "DNF" V 2200 7100 50  0000 C CNN
+F 2 "Resistor_SMD:R_0603_1608Metric" V 2230 7000 50  0001 C CNN
+F 3 "" H 2300 7000 50  0000 C CNN
+F 4 "101-005" V 2300 7000 60  0001 C CNN "Devtank"
+	1    2300 7000
+	0    1    1    0
+$EndComp
+Connection ~ 2800 7000
+Wire Wire Line
+	2800 6900 2800 7000
+Wire Wire Line
+	2450 7000 2800 7000
+Wire Wire Line
+	2150 7000 1800 7000
+Wire Wire Line
+	2800 7000 2800 7050
+Wire Wire Line
+	2800 7000 4050 7000
+Wire Wire Line
+	2800 6450 2800 6600
+Wire Wire Line
+	4050 7000 4050 5575
+Wire Wire Line
+	4050 5575 4100 5575
 $EndSCHEMATC

Commit message: Rev C - pre-release
Parts:
- C195, C196, C197, C198, C199, C200, C201, C203, C204, C205, C206, C207, C208, C209, C210, C211, C212, C213, C215, C216, C218, C221, C222, C223, C59: symbol device:C -> HILTOP_Motherboard-rescue:C-device
- D85, D86, D87, D88, D89, D90, D91, D92: symbol device:LED -> HILTOP_Motherboard-rescue:LED-device
- FB11, FB7, FB9: symbol device:L -> HILTOP_Motherboard-rescue:L-device
- J25: symbol Connector:Conn_01x03 -> HILTOP_Motherboard-rescue:Conn_01x03-Connector
- R177, R187, R224, R225, R226, R227, R228, R229, R230, R231, R232, R233, R234, R235, R236, R237, R238, R239, R240, R241, R242: symbol device:R -> HILTOP_Motherboard-rescue:R-device
- R186: value 100K -> DNF; symbol device:R -> HILTOP_Motherboard-rescue:R-device; Devtank 101-015 -> (none)
- R94: value DNF -> 0R; symbol device:R -> HILTOP_Motherboard-rescue:R-device
- U38: symbol memory:AT25_EEPROM -> HILTOP_Motherboard-rescue:AT25_EEPROM-memory
- Y7: symbol device:Crystal_GND24 -> HILTOP_Motherboard-rescue:Crystal_GND24-device
Changed lines of the file:
@@
 $Descr A3 16535 11693
 encoding utf-8
-Sheet 8 12
+Sheet 7 12
 Title "HILTOP Motherboard"
 Date "2019-07-03"
@@
 CAP_SATARX_P
 $Comp
-L device:C C197
+L HILTOP_Motherboard-rescue:C-device C197
 U 1 1 5A95CF3D
 P 2950 2175
@@
 $EndComp
 $Comp
-L device:C C198
+L HILTOP_Motherboard-rescue:C-device C198
 U 1 1 5A95D01D
 P 2950 2400
@@
 $EndComp
 $Comp
-L device:C C199
+L HILTOP_Motherboard-rescue:C-device C199
 U 1 1 5A95D06F
 P 2950 2625
@@
 $EndComp
 $Comp
-L device:C C200
+L HILTOP_Motherboard-rescue:C-device C200
 U 1 1 5A95D0AA
 P 2950 2850
@@
 $EndComp
 $Comp
-L device:L FB7
+L HILTOP_Motherboard-rescue:L-device FB7
 U 1 1 5A99EB19
 P 6400 9800
@@
 $EndComp
 $Comp
-L device:L FB9
+L HILTOP_Motherboard-rescue:L-device FB9
 U 1 1 5A99EB21
 P 6525 8000
@@
 $EndComp
 $Comp
-L device:L FB11
+L HILTOP_Motherboard-rescue:L-device FB11
 U 1 1 5A99EB29
 P 9500 9800
@@
 $EndComp
 $Comp
-L device:C C215
+L HILTOP_Motherboard-rescue:C-device C215
 U 1 1 5A99EB49
 P 6800 10100
@@
 $EndComp
 $Comp
-L device:C C223
+L HILTOP_Motherboard-rescue:C-device C223
 U 1 1 5A99EB59
 P 9150 10100
@@
 $EndComp
 $Comp
-L device:C C216
+L HILTOP_Motherboard-rescue:C-device C216
 U 1 1 5A9A1DD9
 P 7100 10100
@@
 $EndComp
 $Comp
-L device:C C218
+L HILTOP_Motherboard-rescue:C-device C218
 U 1 1 5A9A1E63
 P 7400 10100
@@
 $EndComp
 $Comp
-L device:C C221
+L HILTOP_Motherboard-rescue:C-device C221
 U 1 1 5A9A1FCA
 P 8025 10100
@@
 $EndComp
 $Comp
-L device:C C222
+L HILTOP_Motherboard-rescue:C-device C222
 U 1 1 5A9A276A
 P 8825 10100
@@
 $EndComp
 $Comp
-L device:C C205
+L HILTOP_Motherboard-rescue:C-device C205
 U 1 1 5A9A572F
 P 4100 8250
@@
 $EndComp
 $Comp
-L device:C C207
+L HILTOP_Motherboard-rescue:C-device C207
 U 1 1 5A9A5736
 P 4450 8250
@@
 $EndComp
 $Comp
-L device:C C209
+L HILTOP_Motherboard-rescue:C-device C209
 U 1 1 5A9A573D
 P 4800 8250
@@
 $EndComp
 $Comp
-L device:C C211
+L HILTOP_Motherboard-rescue:C-device C211
 U 1 1 5A9A5744
 P 5150 8250
@@
 $EndComp
 $Comp
-L device:C C212
+L HILTOP_Motherboard-rescue:C-device C212
 U 1 1 5A9A574B
 P 5500 8250
@@
 $EndComp
 $Comp
-L device:C C213
+L HILTOP_Motherboard-rescue:C-device C213
 U 1 1 5A9A5752
 P 5850 8250
@@
 $EndComp
 $Comp
-L device:C C203
+L HILTOP_Motherboard-rescue:C-device C203
 U 1 1 5A9A6E91
 P 3750 8250
@@
 $EndComp
 $Comp
-L device:C C201
+L HILTOP_Motherboard-rescue:C-device C201
 U 1 1 5A9A7062
 P 3000 8250
@@
 $EndComp
 $Comp
-L device:C C196
+L HILTOP_Motherboard-rescue:C-device C196
 U 1 1 5A9A819C
 P 2650 8250
@@
 $EndComp
 $Comp
-L device:C C195
+L HILTOP_Motherboard-rescue:C-device C195
 U 1 1 5A9A8344
 P 2300 8250
@@
 $EndComp
 $Comp
-L memory:AT25_EEPROM U38
+L HILTOP_Motherboard-rescue:AT25_EEPROM-memory U38
 U 1 1 5B3A146D
 P 10375 3275
@@
 $EndComp
 $Comp
-L device:R R228
+L HILTOP_Motherboard-rescue:R-device R228
 U 1 1 5B3ADA3E
 P 8525 2600
@@
 $EndComp
 $Comp
-L device:R R232
+L HILTOP_Motherboard-rescue:R-device R232
 U 1 1 5B3ADA46
 P 9950 4050
@@
 	8875 2850 7975 2850
 $Comp
-L device:R R229
+L HILTOP_Motherboard-rescue:R-device R229
 U 1 1 5B3ADF8F
 P 8525 3150
@@
 	11100 3375 11100 4050
 $Comp
-L device:R R231
+L HILTOP_Motherboard-rescue:R-device R231
 U 1 1 5B3B1094
 P 9675 2775
@@
 $EndComp
 $Comp
-L device:R R230
+L HILTOP_Motherboard-rescue:R-device R230
 U 1 1 5B3B1FBC
 P 9375 2775
@@
 	10375 2575 10375 2725
 $Comp
-L device:C C208
+L HILTOP_Motherboard-rescue:C-device C208
 U 1 1 5B3B2741
 P 10700 2725
@@
 	9175 4750 7975 4750
 $Comp
-L device:R R233
+L HILTOP_Motherboard-rescue:R-device R233
 U 1 1 5B3B5F80
 P 10275 4775
@@
 $EndComp
 $Comp
-L device:R R234
+L HILTOP_Motherboard-rescue:R-device R234
 U 1 1 5B3B66C6
 P 10775 4450
@@
 Connection ~ 6225 1675
 $Comp
-L device:R R224
+L HILTOP_Motherboard-rescue:R-device R224
 U 1 1 5B3E2C11
 P 3300 5450
@@
 $EndComp
 $Comp
-L device:R R226
+L HILTOP_Motherboard-rescue:R-device R226
 U 1 1 5B3E3634
 P 3300 5650
@@
 $EndComp
 $Comp
-L device:R R225
+L HILTOP_Motherboard-rescue:R-device R225
 U 1 1 5B3E3AC9
 P 3300 5550
@@
 $EndComp
 $Comp
-L device:R R227
+L HILTOP_Motherboard-rescue:R-device R227
 U 1 1 5B3E4135
 P 3300 5750
@@
 Connection ~ 2875 5750
 $Comp
-L device:Crystal_GND24 Y7
+L HILTOP_Motherboard-rescue:Crystal_GND24-device Y7
 U 1 1 5B3F6674
 P 1725 5125
@@
 $EndComp
 $Comp
-L device:C C206
+L HILTOP_Motherboard-rescue:C-device C206
 U 1 1 5B3F667C
 P 2075 5375
@@
 $EndComp
 $Comp
-L device:C C204
+L HILTOP_Motherboard-rescue:C-device C204
 U 1 1 5B3F668A
 P 1375 5375
@@
 Connection ~ 1725 5375
 $Comp
-L device:R R177
+L HILTOP_Motherboard-rescue:R-device R177
 U 1 1 5B3F94D1
 P 2075 5925
@@
 	6050 6250 6050 6600
 $Comp
-L Connector:Conn_01x03 J25
+L HILTOP_Motherboard-rescue:Conn_01x03-Connector J25
 U 1 1 5B3FF3CC
 P 2675 3950
@@
 GPIO_7
 $Comp
-L device:R R235
+L HILTOP_Motherboard-rescue:R-device R235
 U 1 1 5B4184B9
 P 11425 6625
@@
 $EndComp
 $Comp
-L device:LED D85
+L HILTOP_Motherboard-rescue:LED-device D85
 U 1 1 5B4184C0
 P 10625 6625
@@
 $EndComp
 $Comp
-L device:R R236
+L HILTOP_Motherboard-rescue:R-device R236
 U 1 1 5B418C9B
 P 11425 6825
@@
 $EndComp
 $Comp
-L device:LED D86
+L HILTOP_Motherboard-rescue:LED-device D86
 U 1 1 5B418CA1
 P 10625 6825
@@
 $EndComp
 $Comp
-L device:R R237
+L HILTOP_Motherboard-rescue:R-device R237
 U 1 1 5B418E2B
 P 11425 7025
@@
 $EndComp
 $Comp
-L device:LED D87
+L HILTOP_Motherboard-rescue:LED-device D87
 U 1 1 5B418E32
 P 10625 7025
@@
 $EndComp
 $Comp
-L device:R R238
+L HILTOP_Motherboard-rescue:R-device R238
 U 1 1 5B418FF6
 P 11425 7225
@@
 $EndComp
 $Comp
-L device:LED D88
+L HILTOP_Motherboard-rescue:LED-device D88
 U 1 1 5B418FFD
 P 10625 7225
@@
 $EndComp
 $Comp
-L device:R R239
+L HILTOP_Motherboard-rescue:R-device R239
 U 1 1 5B419124
 P 11425 7425
@@
 $EndComp
 $Comp
-L device:LED D89
+L HILTOP_Motherboard-rescue:LED-device D89
 U 1 1 5B41912B
 P 10625 7425
@@
 $EndComp
 $Comp
-L device:R R240
+L HILTOP_Motherboard-rescue:R-device R240
 U 1 1 5B419280
 P 11425 7625
@@
 $EndComp
 $Comp
-L device:LED D90
+L HILTOP_Motherboard-rescue:LED-device D90
 U 1 1 5B419287
 P 10625 7625
@@
 $EndComp
 $Comp
-L device:R R241
+L HILTOP_Motherboard-rescue:R-device R241
 U 1 1 5B419FCE
 P 11425 7825
@@
 $EndComp
 $Comp
-L device:LED D91
+L HILTOP_Motherboard-rescue:LED-device D91
 U 1 1 5B419FD5
 P 10625 7825
@@
 $EndComp
 $Comp
-L device:R R242
+L HILTOP_Motherboard-rescue:R-device R242
 U 1 1 5B41A0FE
 P 11425 8025
@@
 $EndComp
 $Comp
-L device:LED D92
+L HILTOP_Motherboard-rescue:LED-device D92
 U 1 1 5B41A105
 P 10625 8025
@@
 	12075 7825 12075 8025
 $Comp
-L device:C C210
+L HILTOP_Motherboard-rescue:C-device C210
 U 1 1 5C849D3C
 P 6875 8275
@@
 RX_P
 $Comp
-L device:R R187
+L HILTOP_Motherboard-rescue:R-device R187
 U 1 1 5D2A03C4
 P 7250 8000
@@
 $EndComp
 $Comp
-L device:R R?
+L HILTOP_Motherboard-rescue:R-device R?
 U 1 1 5D506DB6
 P 2800 6750
@@
 AR Path="/5A951BF0/5D506DB6" Ref="R186"  Part="1"
 F 0 "R186" H 2950 6700 50  0000 C CNN
-F 1 "100K" H 2950 6800 50  0000 C CNN
+F 1 "DNF" H 2950 6800 50  0000 C CNN
 F 2 "Resistor_SMD:R_0603_1608Metric" V 2730 6750 50  0001 C CNN
 F 3 "" H 2800 6750 50  0000 C CNN
-F 4 "101-015" H 2800 6750 60  0001 C CNN "Devtank"
 	1    2800 6750
 	-1   0    0    1
 $EndComp
 $Comp
-L device:C C?
+L HILTOP_Motherboard-rescue:C-device C?
 U 1 1 5D506DBE
 P 2800 7200
@@
 ~RESET
 $Comp
-L device:R R?
+L HILTOP_Motherboard-rescue:R-device R?
 U 1 1 5D506DCD
 P 2300 7000
@@
 AR Path="/5A951BF0/5D506DCD" Ref="R94"  Part="1"
 F 0 "R94" V 2200 6900 50  0000 C CNN
-F 1 "DNF" V 2200 7100 50  0000 C CNN
+F 1 "0R" V 2200 7100 50  0000 C CNN
 F 2 "Resistor_SMD:R_0603_1608Metric" V 2230 7000 50  0001 C CNN
 F 3 "" H 2300 7000 50  0000 C CNN

Commit message: changed silkscreen to revD and updated sheet information
Parts:
- U37: symbol Devtank:TUSB9261 -> HILTOP_Motherboard-rescue:TUSB9261-Devtank
Changed lines of the file:
@@
 Sheet 7 12
 Title "HILTOP Motherboard"
-Date "2020-04-28"
-Rev "Rev C"
+Date "2021-02-17"
+Rev "Rev D"
 Comp "Devtank Ltd"
-Comment1 ""
+Comment1 "Part No: 304-001"
 Comment2 ""
 Comment3 ""
@@
 $EndComp
 $Comp
-L Devtank:+3V3_SATA_A #PWR0404
+L HILTOP_Motherboard-rescue:+3V3_SATA_A-Devtank #PWR0404
 U 1 1 5A99FBDC
 P 9150 9500
@@
 $EndComp
 $Comp
-L Devtank:+3V3_SATA_D #PWR0399
+L HILTOP_Motherboard-rescue:+3V3_SATA_D-Devtank #PWR0399
 U 1 1 5A9A0239
 P 6800 9500
@@
 Connection ~ 2650 8000
 $Comp
-L Devtank:TUSB9261 U37
+L HILTOP_Motherboard-rescue:TUSB9261-Devtank U37
 U 1 1 5B3A08F6
 P 6050 4400
@@
 	11175 4450 10925 4450
 $Comp
-L Devtank:+3V3_SATA_A #PWR0401
+L HILTOP_Motherboard-rescue:+3V3_SATA_A-Devtank #PWR0401
 U 1 1 5B3C4638
 P 7175 1550
@@
 $EndComp
 $Comp
-L Devtank:+3V3_SATA_D #PWR0396
+L HILTOP_Motherboard-rescue:+3V3_SATA_D-Devtank #PWR0396
 U 1 1 5B3C4AA8
 P 6125 1550
@@
 Connection ~ 3725 5650
 $Comp
-L Devtank:+3V3_SATA_D #PWR0389
+L HILTOP_Motherboard-rescue:+3V3_SATA_D-Devtank #PWR0389
 U 1 1 5B3E4F01
 P 2775 5300
@@
 	7400 8000 7650 8000
 $Comp
-L Devtank:+1V1_SATA #PWR0397
+L HILTOP_Motherboard-rescue:+1V1_SATA-Devtank #PWR0397
 U 1 1 5B404D47
 P 6175 7700
@@
 $EndComp
 $Comp
-L Devtank:+1V1_SATA #PWR0392
+L HILTOP_Motherboard-rescue:+1V1_SATA-Devtank #PWR0392
 U 1 1 5B406E18
 P 4825 1550
